File: etb-9201.kicad_sch (KiCad schematic)
At the start: 5 parts, among them U11 TLE9201SG

Commit message: fome-mc: implement integrated motorcycle ECU schematics, 474-part PCB, BOM/CPL, DESIGN.md, and VALIDATION.md
Parts:
- renumbered C28 to C201, C29 to C202, R48 to R210, U11 to U201
Changed lines of the file:
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@@
   (symbol (lib_id "tle9201_2:TLE9201SG") (at 73.025 43.18 0)
     (in_bom yes) (on_board yes)
-    (property "Reference" "U11" (id 0) (at 72.39 27.305 0))
+    (property "Reference" "U201" (id 0) (at 72.39 27.305 0))
     (property "Value" "TLE9201SG" (id 1) (at 72.39 29.6164 0))
     (property "Footprint" "Package_SO:Infineon_PG-DSO-12-9" (id 2) (at 69.215 41.91 0)
@@
   (symbol (lib_id "Device:C_Small") (at 88.9 28.575 0)
     (in_bom yes) (on_board yes)
-    (property "Reference" "C28" (id 0) (at 91.2368 27.4066 0)
+    (property "Reference" "C201" (id 0) (at 91.2368 27.4066 0)
       (effects (font (size 1.27 1.27)) (justify left))
     )
@@
   (symbol (lib_id "Device:C_Small") (at 88.9 40.005 0)
     (in_bom yes) (on_board yes)
-    (property "Reference" "C29" (id 0) (at 91.2368 38.8366 0)
+    (property "Reference" "C202" (id 0) (at 91.2368 38.8366 0)
       (effects (font (size 1.27 1.27)) (justify left))
     )
@@
   (symbol (lib_id "Device:R") (at 44.45 36.83 270)
     (in_bom yes) (on_board yes)
-    (property "Reference" "R48" (id 0) (at 44.45 39.37 90))
+    (property "Reference" "R210" (id 0) (at 44.45 39.37 90))
     (property "Value" "10k" (id 1) (at 44.45 36.83 90))
     (property "Footprint" "Resistor_SMD:R_0402_1005Metric" (id 2) (at 44.45 35.052 90)
