File: Keep_Alive.kicad_sch (KiCad schematic)
At the start: 7 parts, among them IC1 PSM712-LF-T7, U41 MIC5205-3.3YM5

Commit message: Remove all legacy Atlas-clone files/references and standardize on fome-mc
Other:
- title: Atlas-clone -> fome-mc
Changed lines of the file:
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@@
 	(paper "A4")
 	(title_block
-		(title "Atlas-clone")
+		(title "fome-mc")
 		(date "2024-11-14")
 		(rev "v1.0-atlas-h7")
@@
 		)
 		(instances
-			(project "Atlas-clone"
+			(project "fome-mc"
 				(path "/3b9c5ffd-e59b-402d-8c5e-052f7ca643a4/46495fed-359e-4c30-808a-9217af090de7"
 					(reference "IC1")
@@
 		)
 		(instances
-			(project "Atlas-clone"
+			(project "fome-mc"
 				(path "/3b9c5ffd-e59b-402d-8c5e-052f7ca643a4/46495fed-359e-4c30-808a-9217af090de7"
 					(reference "#PWR0258")
@@
 		)
 		(instances
-			(project "Atlas-clone"
+			(project "fome-mc"
 				(path "/3b9c5ffd-e59b-402d-8c5e-052f7ca643a4/46495fed-359e-4c30-808a-9217af090de7"
 					(reference "U41")
@@
 		)
 		(instances
-			(project "Atlas-clone"
+			(project "fome-mc"
 				(path "/3b9c5ffd-e59b-402d-8c5e-052f7ca643a4/46495fed-359e-4c30-808a-9217af090de7"
 					(reference "#PWR0260")
@@
 		)
 		(instances
-			(project "Atlas-clone"
+			(project "fome-mc"
 				(path "/3b9c5ffd-e59b-402d-8c5e-052f7ca643a4/46495fed-359e-4c30-808a-9217af090de7"
 					(reference "#PWR0257")
@@
 		)
 		(instances
-			(project "Atlas-clone"
+			(project "fome-mc"
 				(path "/3b9c5ffd-e59b-402d-8c5e-052f7ca643a4/46495fed-359e-4c30-808a-9217af090de7"
 					(reference "C90")
@@
 		)
 		(instances
-			(project "Atlas-clone"
+			(project "fome-mc"
 				(path "/3b9c5ffd-e59b-402d-8c5e-052f7ca643a4/46495fed-359e-4c30-808a-9217af090de7"
 					(reference "D17")
@@
 		)
 		(instances
-			(project "Atlas-clone"
+			(project "fome-mc"
 				(path "/3b9c5ffd-e59b-402d-8c5e-052f7ca643a4/46495fed-359e-4c30-808a-9217af090de7"
 					(reference "#PWR0259")
@@
 		)
 		(instances
-			(project "Atlas-clone"
+			(project "fome-mc"
 				(path "/3b9c5ffd-e59b-402d-8c5e-052f7ca643a4/46495fed-359e-4c30-808a-9217af090de7"
 					(reference "R107")
@@
 		)
 		(instances
-			(project "Atlas-clone"
+			(project "fome-mc"
 				(path "/3b9c5ffd-e59b-402d-8c5e-052f7ca643a4/46495fed-359e-4c30-808a-9217af090de7"
 					(reference "C89")
@@
 		)
 		(instances
-			(project "Atlas-clone"
+			(project "fome-mc"
 				(path "/3b9c5ffd-e59b-402d-8c5e-052f7ca643a4/46495fed-359e-4c30-808a-9217af090de7"
 					(reference "D16")
@@
 		)
 		(instances
-			(project "Atlas-clone"
+			(project "fome-mc"
 				(path "/3b9c5ffd-e59b-402d-8c5e-052f7ca643a4/46495fed-359e-4c30-808a-9217af090de7"
 					(reference "#FLG01401")
