File: highside_quad.kicad_sch (KiCad schematic)
At the start: 14 parts, among them U40 BTS716G

Commit message: Remove all legacy Atlas-clone files/references and standardize on fome-mc
Other:
- title: Atlas-clone -> fome-mc
Changed lines of the file:
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@@
 	(paper "A4")
 	(title_block
-		(title "Atlas-clone")
+		(title "fome-mc")
 		(date "2024-11-14")
 		(rev "v1.0-atlas-h7")
@@
 		)
 		(instances
-			(project "Atlas-clone"
+			(project "fome-mc"
 				(path "/3b9c5ffd-e59b-402d-8c5e-052f7ca643a4/00000000-0000-0000-0000-00005dd5b2e0"
 					(reference "RN11")
@@
 		)
 		(instances
-			(project "Atlas-clone"
+			(project "fome-mc"
 				(path "/3b9c5ffd-e59b-402d-8c5e-052f7ca643a4/00000000-0000-0000-0000-00005dd5b2e0"
 					(reference "C85")
@@
 		)
 		(instances
-			(project "Atlas-clone"
+			(project "fome-mc"
 				(path "/3b9c5ffd-e59b-402d-8c5e-052f7ca643a4/00000000-0000-0000-0000-00005dd5b2e0"
 					(reference "C86")
@@
 		)
 		(instances
-			(project "Atlas-clone"
+			(project "fome-mc"
 				(path "/3b9c5ffd-e59b-402d-8c5e-052f7ca643a4/00000000-0000-0000-0000-00005dd5b2e0"
 					(reference "#PWR0248")
@@
 		)
 		(instances
-			(project "Atlas-clone"
+			(project "fome-mc"
 				(path "/3b9c5ffd-e59b-402d-8c5e-052f7ca643a4/00000000-0000-0000-0000-00005dd5b2e0"
 					(reference "#PWR0250")
@@
 		)
 		(instances
-			(project "Atlas-clone"
+			(project "fome-mc"
 				(path "/3b9c5ffd-e59b-402d-8c5e-052f7ca643a4/00000000-0000-0000-0000-00005dd5b2e0"
 					(reference "R102")
@@
 		)
 		(instances
-			(project "Atlas-clone"
+			(project "fome-mc"
 				(path "/3b9c5ffd-e59b-402d-8c5e-052f7ca643a4/00000000-0000-0000-0000-00005dd5b2e0"
 					(reference "R99")
@@
 		)
 		(instances
-			(project "Atlas-clone"
+			(project "fome-mc"
 				(path "/3b9c5ffd-e59b-402d-8c5e-052f7ca643a4/00000000-0000-0000-0000-00005dd5b2e0"
 					(reference "#PWR0245")
@@
 		)
 		(instances
-			(project "Atlas-clone"
+			(project "fome-mc"
 				(path "/3b9c5ffd-e59b-402d-8c5e-052f7ca643a4/00000000-0000-0000-0000-00005dd5b2e0"
 					(reference "#PWR0247")
@@
 		)
 		(instances
-			(project "Atlas-clone"
+			(project "fome-mc"
 				(path "/3b9c5ffd-e59b-402d-8c5e-052f7ca643a4/00000000-0000-0000-0000-00005dd5b2e0"
 					(reference "#PWR0252")
@@
 		)
 		(instances
-			(project "Atlas-clone"
+			(project "fome-mc"
 				(path "/3b9c5ffd-e59b-402d-8c5e-052f7ca643a4/00000000-0000-0000-0000-00005dd5b2e0"
 					(reference "R101")
@@
 		)
 		(instances
-			(project "Atlas-clone"
+			(project "fome-mc"
 				(path "/3b9c5ffd-e59b-402d-8c5e-052f7ca643a4/00000000-0000-0000-0000-00005dd5b2e0"
 					(reference "R100")
@@
 		)
 		(instances
-			(project "Atlas-clone"
+			(project "fome-mc"
 				(path "/3b9c5ffd-e59b-402d-8c5e-052f7ca643a4/00000000-0000-0000-0000-00005dd5b2e0"
 					(reference "#PWR0246")
@@
 		)
 		(instances
-			(project "Atlas-clone"
+			(project "fome-mc"
 				(path "/3b9c5ffd-e59b-402d-8c5e-052f7ca643a4/00000000-0000-0000-0000-00005dd5b2e0"
 					(reference "R103")
@@
 		)
 		(instances
-			(project "Atlas-clone"
+			(project "fome-mc"
 				(path "/3b9c5ffd-e59b-402d-8c5e-052f7ca643a4/00000000-0000-0000-0000-00005dd5b2e0"
 					(reference "#PWR0249")
@@
 		)
 		(instances
-			(project "Atlas-clone"
+			(project "fome-mc"
 				(path "/3b9c5ffd-e59b-402d-8c5e-052f7ca643a4/00000000-0000-0000-0000-00005dd5b2e0"
 					(reference "R104")
@@
 		)
 		(instances
-			(project "Atlas-clone"
+			(project "fome-mc"
 				(path "/3b9c5ffd-e59b-402d-8c5e-052f7ca643a4/00000000-0000-0000-0000-00005dd5b2e0"
 					(reference "#PWR0251")
@@
 		)
 		(instances
-			(project "Atlas-clone"
+			(project "fome-mc"
 				(path "/3b9c5ffd-e59b-402d-8c5e-052f7ca643a4/00000000-0000-0000-0000-00005dd5b2e0"
 					(reference "#PWR0255")
@@
 		)
 		(instances
-			(project "Atlas-clone"
+			(project "fome-mc"
 				(path "/3b9c5ffd-e59b-402d-8c5e-052f7ca643a4/00000000-0000-0000-0000-00005dd5b2e0"
 					(reference "R106")
@@
 		)
 		(instances
-			(project "Atlas-clone"
+			(project "fome-mc"
 				(path "/3b9c5ffd-e59b-402d-8c5e-052f7ca643a4/00000000-0000-0000-0000-00005dd5b2e0"
 					(reference "U40")
@@
 		)
 		(instances
-			(project "Atlas-clone"
+			(project "fome-mc"
 				(path "/3b9c5ffd-e59b-402d-8c5e-052f7ca643a4/00000000-0000-0000-0000-00005dd5b2e0"
 					(reference "C88")
@@
 		)
 		(instances
-			(project "Atlas-clone"
+			(project "fome-mc"
 				(path "/3b9c5ffd-e59b-402d-8c5e-052f7ca643a4/00000000-0000-0000-0000-00005dd5b2e0"
 					(reference "R105")
@@
 		)
 		(instances
-			(project "Atlas-clone"
+			(project "fome-mc"
 				(path "/3b9c5ffd-e59b-402d-8c5e-052f7ca643a4/00000000-0000-0000-0000-00005dd5b2e0"
 					(reference "#PWR0256")
@@
 		)
 		(instances
-			(project "Atlas-clone"
+			(project "fome-mc"
 				(path "/3b9c5ffd-e59b-402d-8c5e-052f7ca643a4/00000000-0000-0000-0000-00005dd5b2e0"
 					(reference "#PWR0254")
@@
 		)
 		(instances
-			(project "Atlas-clone"
+			(project "fome-mc"
 				(path "/3b9c5ffd-e59b-402d-8c5e-052f7ca643a4/00000000-0000-0000-0000-00005dd5b2e0"
 					(reference "C87")
@@
 		)
 		(instances
-			(project "Atlas-clone"
+			(project "fome-mc"
 				(path "/3b9c5ffd-e59b-402d-8c5e-052f7ca643a4/00000000-0000-0000-0000-00005dd5b2e0"
 					(reference "#PWR0253")
