File: knock.kicad_sch (KiCad schematic)
At the start: 24 parts, among them U7 MCP6004

Commit message: Remove all legacy Atlas-clone files/references and standardize on fome-mc
Other:
- title: Atlas-clone -> fome-mc
Changed lines of the file:
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@@
 	(paper "A4")
 	(title_block
-		(title "Atlas-clone")
+		(title "fome-mc")
 		(date "2024-11-14")
 		(rev "v1.0-atlas-h7")
@@
 		)
 		(instances
-			(project "Atlas-clone"
+			(project "fome-mc"
 				(path "/3b9c5ffd-e59b-402d-8c5e-052f7ca643a4/00000000-0000-0000-0000-00005e814213"
 					(reference "U7")
@@
 		)
 		(instances
-			(project "Atlas-clone"
+			(project "fome-mc"
 				(path "/3b9c5ffd-e59b-402d-8c5e-052f7ca643a4/00000000-0000-0000-0000-00005e814213"
 					(reference "U7")
@@
 		)
 		(instances
-			(project "Atlas-clone"
+			(project "fome-mc"
 				(path "/3b9c5ffd-e59b-402d-8c5e-052f7ca643a4/00000000-0000-0000-0000-00005e814213"
 					(reference "U7")
@@
 		)
 		(instances
-			(project "Atlas-clone"
+			(project "fome-mc"
 				(path "/3b9c5ffd-e59b-402d-8c5e-052f7ca643a4/00000000-0000-0000-0000-00005e814213"
 					(reference "U7")
@@
 		)
 		(instances
-			(project "Atlas-clone"
+			(project "fome-mc"
 				(path "/3b9c5ffd-e59b-402d-8c5e-052f7ca643a4/00000000-0000-0000-0000-00005e814213"
 					(reference "U7")
@@
 		)
 		(instances
-			(project "Atlas-clone"
+			(project "fome-mc"
 				(path "/3b9c5ffd-e59b-402d-8c5e-052f7ca643a4/00000000-0000-0000-0000-00005e814213"
 					(reference "#PWR060")
@@
 		)
 		(instances
-			(project "Atlas-clone"
+			(project "fome-mc"
 				(path "/3b9c5ffd-e59b-402d-8c5e-052f7ca643a4/00000000-0000-0000-0000-00005e814213"
 					(reference "#PWR059")
@@
 		)
 		(instances
-			(project "Atlas-clone"
+			(project "fome-mc"
 				(path "/3b9c5ffd-e59b-402d-8c5e-052f7ca643a4/00000000-0000-0000-0000-00005e814213"
 					(reference "R11")
@@
 		)
 		(instances
-			(project "Atlas-clone"
+			(project "fome-mc"
 				(path "/3b9c5ffd-e59b-402d-8c5e-052f7ca643a4/00000000-0000-0000-0000-00005e814213"
 					(reference "R12")
@@
 		)
 		(instances
-			(project "Atlas-clone"
+			(project "fome-mc"
 				(path "/3b9c5ffd-e59b-402d-8c5e-052f7ca643a4/00000000-0000-0000-0000-00005e814213"
 					(reference "R17")
@@
 		)
 		(instances
-			(project "Atlas-clone"
+			(project "fome-mc"
 				(path "/3b9c5ffd-e59b-402d-8c5e-052f7ca643a4/00000000-0000-0000-0000-00005e814213"
 					(reference "R19")
@@
 		)
 		(instances
-			(project "Atlas-clone"
+			(project "fome-mc"
 				(path "/3b9c5ffd-e59b-402d-8c5e-052f7ca643a4/00000000-0000-0000-0000-00005e814213"
 					(reference "R21")
@@
 		)
 		(instances
-			(project "Atlas-clone"
+			(project "fome-mc"
 				(path "/3b9c5ffd-e59b-402d-8c5e-052f7ca643a4/00000000-0000-0000-0000-00005e814213"
 					(reference "#PWR054")
@@
 		)
 		(instances
-			(project "Atlas-clone"
+			(project "fome-mc"
 				(path "/3b9c5ffd-e59b-402d-8c5e-052f7ca643a4/00000000-0000-0000-0000-00005e814213"
 					(reference "#PWR053")
@@
 		)
 		(instances
-			(project "Atlas-clone"
+			(project "fome-mc"
 				(path "/3b9c5ffd-e59b-402d-8c5e-052f7ca643a4/00000000-0000-0000-0000-00005e814213"
 					(reference "C18")
@@
 		)
 		(instances
-			(project "Atlas-clone"
+			(project "fome-mc"
 				(path "/3b9c5ffd-e59b-402d-8c5e-052f7ca643a4/00000000-0000-0000-0000-00005e814213"
 					(reference "C22")
@@
 		)
 		(instances
-			(project "Atlas-clone"
+			(project "fome-mc"
 				(path "/3b9c5ffd-e59b-402d-8c5e-052f7ca643a4/00000000-0000-0000-0000-00005e814213"
 					(reference "C20")
@@
 		)
 		(instances
-			(project "Atlas-clone"
+			(project "fome-mc"
 				(path "/3b9c5ffd-e59b-402d-8c5e-052f7ca643a4/00000000-0000-0000-0000-00005e814213"
 					(reference "#PWR055")
@@
 		)
 		(instances
-			(project "Atlas-clone"
+			(project "fome-mc"
 				(path "/3b9c5ffd-e59b-402d-8c5e-052f7ca643a4/00000000-0000-0000-0000-00005e814213"
 					(reference "#PWR057")
@@
 		)
 		(instances
-			(project "Atlas-clone"
+			(project "fome-mc"
 				(path "/3b9c5ffd-e59b-402d-8c5e-052f7ca643a4/00000000-0000-0000-0000-00005e814213"
 					(reference "R18")
@@
 		)
 		(instances
-			(project "Atlas-clone"
+			(project "fome-mc"
 				(path "/3b9c5ffd-e59b-402d-8c5e-052f7ca643a4/00000000-0000-0000-0000-00005e814213"
 					(reference "R20")
@@
 		)
 		(instances
-			(project "Atlas-clone"
+			(project "fome-mc"
 				(path "/3b9c5ffd-e59b-402d-8c5e-052f7ca643a4/00000000-0000-0000-0000-00005e814213"
 					(reference "R22")
@@
 		)
 		(instances
-			(project "Atlas-clone"
+			(project "fome-mc"
 				(path "/3b9c5ffd-e59b-402d-8c5e-052f7ca643a4/00000000-0000-0000-0000-00005e814213"
 					(reference "C19")
@@
 		)
 		(instances
-			(project "Atlas-clone"
+			(project "fome-mc"
 				(path "/3b9c5ffd-e59b-402d-8c5e-052f7ca643a4/00000000-0000-0000-0000-00005e814213"
 					(reference "C23")
@@
 		)
 		(instances
-			(project "Atlas-clone"
+			(project "fome-mc"
 				(path "/3b9c5ffd-e59b-402d-8c5e-052f7ca643a4/00000000-0000-0000-0000-00005e814213"
 					(reference "C21")
@@
 		)
 		(instances
-			(project "Atlas-clone"
+			(project "fome-mc"
 				(path "/3b9c5ffd-e59b-402d-8c5e-052f7ca643a4/00000000-0000-0000-0000-00005e814213"
 					(reference "#PWR056")
@@
 		)
 		(instances
-			(project "Atlas-clone"
+			(project "fome-mc"
 				(path "/3b9c5ffd-e59b-402d-8c5e-052f7ca643a4/00000000-0000-0000-0000-00005e814213"
 					(reference "#PWR058")
@@
 		)
 		(instances
-			(project "Atlas-clone"
+			(project "fome-mc"
 				(path "/3b9c5ffd-e59b-402d-8c5e-052f7ca643a4/00000000-0000-0000-0000-00005e814213"
 					(reference "R13")
@@
 		)
 		(instances
-			(project "Atlas-clone"
+			(project "fome-mc"
 				(path "/3b9c5ffd-e59b-402d-8c5e-052f7ca643a4/00000000-0000-0000-0000-00005e814213"
 					(reference "R15")
@@
 		)
 		(instances
-			(project "Atlas-clone"
+			(project "fome-mc"
 				(path "/3b9c5ffd-e59b-402d-8c5e-052f7ca643a4/00000000-0000-0000-0000-00005e814213"
 					(reference "C16")
@@
 		)
 		(instances
-			(project "Atlas-clone"
+			(project "fome-mc"
 				(path "/3b9c5ffd-e59b-402d-8c5e-052f7ca643a4/00000000-0000-0000-0000-00005e814213"
 					(reference "C15")
@@
 		)
 		(instances
-			(project "Atlas-clone"
+			(project "fome-mc"
 				(path "/3b9c5ffd-e59b-402d-8c5e-052f7ca643a4/00000000-0000-0000-0000-00005e814213"
 					(reference "#PWR052")
@@
 		)
 		(instances
-			(project "Atlas-clone"
+			(project "fome-mc"
 				(path "/3b9c5ffd-e59b-402d-8c5e-052f7ca643a4/00000000-0000-0000-0000-00005e814213"
 					(reference "R16")
@@
 		)
 		(instances
-			(project "Atlas-clone"
+			(project "fome-mc"
 				(path "/3b9c5ffd-e59b-402d-8c5e-052f7ca643a4/00000000-0000-0000-0000-00005e814213"
 					(reference "R14")
@@
 		)
 		(instances
-			(project "Atlas-clone"
+			(project "fome-mc"
 				(path "/3b9c5ffd-e59b-402d-8c5e-052f7ca643a4/00000000-0000-0000-0000-00005e814213"
 					(reference "C17")
@@
 		)
 		(instances
-			(project "Atlas-clone"
+			(project "fome-mc"
 				(path "/3b9c5ffd-e59b-402d-8c5e-052f7ca643a4/00000000-0000-0000-0000-00005e814213"
 					(reference "JP1")
@@
 		)
 		(instances
-			(project "Atlas-clone"
+			(project "fome-mc"
 				(path "/3b9c5ffd-e59b-402d-8c5e-052f7ca643a4/00000000-0000-0000-0000-00005e814213"
 					(reference "JP2")
