File: lowside_quad.kicad_sch (KiCad schematic)
At the start: 4 parts, among them U1001 VNLD5090, U1002 VNLD5090

Commit message: Remove all legacy Atlas-clone files/references and standardize on fome-mc
Other:
- title: Atlas-clone -> fome-mc
Changed lines of the file:
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@@
 	(paper "A4")
 	(title_block
-		(title "Atlas-clone")
+		(title "fome-mc")
 		(date "2024-11-14")
 		(rev "v1.0-atlas-h7")
@@
 		)
 		(instances
-			(project "Atlas-clone"
+			(project "fome-mc"
 				(path "/3b9c5ffd-e59b-402d-8c5e-052f7ca643a4/00000000-0000-0000-0000-00005d98a146"
 					(reference "RN6")
@@
 		)
 		(instances
-			(project "Atlas-clone"
+			(project "fome-mc"
 				(path "/3b9c5ffd-e59b-402d-8c5e-052f7ca643a4/00000000-0000-0000-0000-00005d98a146"
 					(reference "RN5")
@@
 		)
 		(instances
-			(project "Atlas-clone"
+			(project "fome-mc"
 				(path "/3b9c5ffd-e59b-402d-8c5e-052f7ca643a4/00000000-0000-0000-0000-00005d98a146"
 					(reference "#PWR0221")
@@
 		)
 		(instances
-			(project "Atlas-clone"
+			(project "fome-mc"
 				(path "/3b9c5ffd-e59b-402d-8c5e-052f7ca643a4/00000000-0000-0000-0000-00005d98a146"
 					(reference "#PWR0222")
@@
 		)
 		(instances
-			(project "Atlas-clone"
+			(project "fome-mc"
 				(path "/3b9c5ffd-e59b-402d-8c5e-052f7ca643a4/00000000-0000-0000-0000-00005d98a146"
 					(reference "#PWR0223")
@@
 		)
 		(instances
-			(project "Atlas-clone"
+			(project "fome-mc"
 				(path "/3b9c5ffd-e59b-402d-8c5e-052f7ca643a4/00000000-0000-0000-0000-00005d98a146"
 					(reference "#PWR0224")
@@
 		)
 		(instances
-			(project "Atlas-clone"
+			(project "fome-mc"
 				(path "/3b9c5ffd-e59b-402d-8c5e-052f7ca643a4/00000000-0000-0000-0000-00005d98a146"
 					(reference "#PWR01001")
@@
 		)
 		(instances
-			(project "Atlas-clone"
+			(project "fome-mc"
 				(path "/3b9c5ffd-e59b-402d-8c5e-052f7ca643a4/00000000-0000-0000-0000-00005d98a146"
 					(reference "#PWR01002")
@@
 		)
 		(instances
-			(project "Atlas-clone"
+			(project "fome-mc"
 				(path "/3b9c5ffd-e59b-402d-8c5e-052f7ca643a4/00000000-0000-0000-0000-00005d98a146"
 					(reference "#PWR01003")
@@
 		)
 		(instances
-			(project "Atlas-clone"
+			(project "fome-mc"
 				(path "/3b9c5ffd-e59b-402d-8c5e-052f7ca643a4/00000000-0000-0000-0000-00005d98a146"
 					(reference "#PWR01004")
@@
 		)
 		(instances
-			(project "Atlas-clone"
+			(project "fome-mc"
 				(path "/3b9c5ffd-e59b-402d-8c5e-052f7ca643a4/00000000-0000-0000-0000-00005d98a146"
 					(reference "U1001")
@@
 		)
 		(instances
-			(project "Atlas-clone"
+			(project "fome-mc"
 				(path "/3b9c5ffd-e59b-402d-8c5e-052f7ca643a4/00000000-0000-0000-0000-00005d98a146"
 					(reference "U1002")
