File: mcu.kicad_sch (KiCad schematic)
At the start: 75 parts, among them J10 Micro_SD_Card, J11 Conn_01x06, J12 Conn_01x02, J13 USB_B, J14 USB_B, J15 Conn_01x01, J16 Conn_01x01, J8 Conn_02x05_Odd_Even, J9 Conn_01x06, SW1 SW_Push, SW2 SW_Push, U23 REF3333, U24 LPS25HB, U26 STM32H753ZIT6, U27 USBLC6-2SC6, U28 S3225SMD32.768KOSC, Y1 8MHz

Commit message: fome-mc: implement integrated motorcycle ECU schematics, 474-part PCB, BOM/CPL, DESIGN.md, and VALIDATION.md
Parts:
- U25: renamed from J10; value Micro_SD_Card -> XTSD04GLGEAG; footprint Connector_Card:microSD_HC_Wuerth_693072010801 -> ampseal:LGA-8_6x8mm_P1.25mm; LCSC C164170 -> C558840; PN 47219-2001 -> XTSD04GLGEAG
- U28: footprint Oscillator:Oscillator_SMD_SeikoEpson_SG8002LB-4Pin_3.2x2.5mm -> Package_TO_SOT_SMD:SOT-23-5
Connections:
- net SD_CS is gone; now on net SD_D3: U25.2 (DAT3/CD)
- net SD_MISO is gone; now on net SD_D0: U25.7 (DAT0)
- net SD_MOSI is gone; now on net SD_CMD: U25.3 (CMD)
- net SD_SCK is gone; now on net SD_CLK: U25.5 (CLK)
- net WBO1_NRST: now reaches U26.1 (PE2)
- net WBO1_BOOT0: now reaches U26.2 (PE3)
- net WBO2_NRST: now reaches U26.3 (PE4)
- net WBO2_BOOT0: now reaches U26.4 (PE5)
- no-connect marks 22 -> 18
Changed lines of the file:
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@@
 		)
 	)
-	(label "SD_SCK"
+	(label "SD_CLK"
 		(at 286.385 174.625 180)
 		(fields_autoplaced yes)
@@
 		)
 	)
-	(label "SD_MOSI"
+	(label "SD_CMD"
 		(at 286.385 169.545 180)
 		(fields_autoplaced yes)
@@
 		)
 	)
-	(label "SD_CS"
+	(label "SD_D3"
 		(at 286.385 167.005 180)
 		(fields_autoplaced yes)
@@
 		)
 	)
-	(label "SD_MISO"
+	(label "SD_D0"
 		(at 286.385 179.705 180)
 		(fields_autoplaced yes)
@@
 		(on_board yes)
 		(dnp no)
-		(property "Reference" "J10"
+		(property "Reference" "U25"
 			(at 313.69 153.8732 0)
 			(effects
@@
 			)
 		)
-		(property "Value" "Micro_SD_Card"
+		(property "Value" "XTSD04GLGEAG"
 			(at 313.69 156.1846 0)
 			(effects
@@
 			)
 		)
-		(property "Footprint" "Connector_Card:microSD_HC_Wuerth_693072010801"
+		(property "Footprint" "ampseal:LGA-8_6x8mm_P1.25mm"
 			(at 344.17 164.465 0)
 			(effects
@@
 			)
 		)
-		(property "Datasheet" "http://katalog.we-online.de/em/datasheet/693072010801.pdf"
+		(property "Datasheet" "https://datasheet.lcsc.com/lcsc/2005251034_XTX-XTSD04GLGEAG_C558840.pdf"
 			(at 314.96 172.085 0)
 			(effects
@@
 			)
 		)
-		(property "Description" ""
+		(property "Description" "4Gbit (512MB) Soldered Pottable SD NAND Flash LGA-8 6x8mm"
 			(at 314.96 172.085 0)
 			(effects
@@
 			)
 		)
-		(property "LCSC" "C164170"
+		(property "LCSC" "C558840"
 			(at 314.96 172.085 0)
 			(effects
@@
 			)
 		)
-		(property "PN" "47219-2001"
+		(property "PN" "XTSD04GLGEAG"
 			(at 314.96 172.085 0)
 			(effects
@@
 			(project "Atlas-clone"
 				(path "/3b9c5ffd-e59b-402d-8c5e-052f7ca643a4/00000000-0000-0000-0000-00005d99e6ee"
-					(reference "J10")
+					(reference "U25")
+					(unit 1)
+				)
+			)
+			(project "fome-mc"
+				(path "/3b9c5ffd-e59b-402d-8c5e-052f7ca643a4/00000000-0000-0000-0000-00005d99e6ee"
+					(reference "U25")
 					(unit 1)
 				)
@@
 		)
 	)
-	(no_connect
-		(at 104.14 192.405)
+	(hierarchical_label "WBO1_NRST"
+		(shape output)
+		(at 104.14 192.405 180)
+		(effects
+			(font
+				(size 1.27 1.27)
+			)
+			(justify right)
+		)
 	)
-	(no_connect
-		(at 104.14 194.945)
+	(hierarchical_label "WBO1_BOOT0"
+		(shape output)
+		(at 104.14 194.945 180)
+		(effects
+			(font
+				(size 1.27 1.27)
+			)
+			(justify right)
+		)
 	)
-	(no_connect
-		(at 104.14 197.485)
+	(hierarchical_label "WBO2_NRST"
+		(shape output)
+		(at 104.14 197.485 180)
+		(effects
+			(font
+				(size 1.27 1.27)
+			)
+			(justify right)
+		)
 	)
-	(no_connect
-		(at 104.14 200.025)
+	(hierarchical_label "WBO2_BOOT0"
+		(shape output)
+		(at 104.14 200.025 180)
+		(effects
+			(font
+				(size 1.27 1.27)
+			)
+			(justify right)
+		)
 	)
 	(no_connect
@@
 			(effects (font (size 1.27 1.27)))
 		)
-		(property "Footprint" "Oscillator:Oscillator_SMD_SeikoEpson_SG8002LB-4Pin_3.2x2.5mm"
+		(property "Footprint" "Package_TO_SOT_SMD:SOT-23-5"
 			(at 235.0 34.29 0)
 			(effects (font (size 1.27 1.27)) (hide yes))
@@
 		)
 	)
+	(hierarchical_label "BOOT0"
+		(shape input)
+		(at 104.14 83.185 180)
+		(effects
+			(font
+				(size 1.27 1.27)
+			)
+			(justify right)
+		)
+	)

Commit message: Remove all legacy Atlas-clone files/references and standardize on fome-mc
Other:
- title: Atlas-clone -> fome-mc
