File: psu.kicad_sch (KiCad schematic)
At the start: 42 parts, among them U1 TLS115D0E, U2 TLS115D0E, U3 LMR14020, U4 MCP2551-I-SN, U46 LM2733XMFX/NOPB, U5 MCP2551-I-SN, U6 AMS1117-3.3

Commit message: Remove all legacy Atlas-clone files/references and standardize on fome-mc
Other:
- title: Atlas-clone -> fome-mc
