File: quad_analog.kicad_sch (KiCad schematic)
At the start: 20 parts, among them U17 MCP6004, U18 SRV05-4

Commit message: Remove all legacy Atlas-clone files/references and standardize on fome-mc
Other:
- title: Atlas-clone -> fome-mc
Changed lines of the file:
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@@
 	(paper "A4")
 	(title_block
-		(title "Atlas-clone")
+		(title "fome-mc")
 		(date "2024-11-14")
 		(rev "v1.0-atlas-h7")
@@
 		)
 		(instances
-			(project "Atlas-clone"
+			(project "fome-mc"
 				(path "/3b9c5ffd-e59b-402d-8c5e-052f7ca643a4/00000000-0000-0000-0000-00005d9a3845"
 					(reference "U17")
@@
 		)
 		(instances
-			(project "Atlas-clone"
+			(project "fome-mc"
 				(path "/3b9c5ffd-e59b-402d-8c5e-052f7ca643a4/00000000-0000-0000-0000-00005d9a3845"
 					(reference "U17")
@@
 		)
 		(instances
-			(project "Atlas-clone"
+			(project "fome-mc"
 				(path "/3b9c5ffd-e59b-402d-8c5e-052f7ca643a4/00000000-0000-0000-0000-00005d9a3845"
 					(reference "U17")
@@
 		)
 		(instances
-			(project "Atlas-clone"
+			(project "fome-mc"
 				(path "/3b9c5ffd-e59b-402d-8c5e-052f7ca643a4/00000000-0000-0000-0000-00005d9a3845"
 					(reference "U17")
@@
 		)
 		(instances
-			(project "Atlas-clone"
+			(project "fome-mc"
 				(path "/3b9c5ffd-e59b-402d-8c5e-052f7ca643a4/00000000-0000-0000-0000-00005d9a3845"
 					(reference "R52")
@@
 		)
 		(instances
-			(project "Atlas-clone"
+			(project "fome-mc"
 				(path "/3b9c5ffd-e59b-402d-8c5e-052f7ca643a4/00000000-0000-0000-0000-00005d9a3845"
 					(reference "R53")
@@
 		)
 		(instances
-			(project "Atlas-clone"
+			(project "fome-mc"
 				(path "/3b9c5ffd-e59b-402d-8c5e-052f7ca643a4/00000000-0000-0000-0000-00005d9a3845"
 					(reference "R54")
@@
 		)
 		(instances
-			(project "Atlas-clone"
+			(project "fome-mc"
 				(path "/3b9c5ffd-e59b-402d-8c5e-052f7ca643a4/00000000-0000-0000-0000-00005d9a3845"
 					(reference "#PWR0105")
@@
 		)
 		(instances
-			(project "Atlas-clone"
+			(project "fome-mc"
 				(path "/3b9c5ffd-e59b-402d-8c5e-052f7ca643a4/00000000-0000-0000-0000-00005d9a3845"
 					(reference "#PWR0106")
@@
 		)
 		(instances
-			(project "Atlas-clone"
+			(project "fome-mc"
 				(path "/3b9c5ffd-e59b-402d-8c5e-052f7ca643a4/00000000-0000-0000-0000-00005d9a3845"
 					(reference "#PWR0107")
@@
 		)
 		(instances
-			(project "Atlas-clone"
+			(project "fome-mc"
 				(path "/3b9c5ffd-e59b-402d-8c5e-052f7ca643a4/00000000-0000-0000-0000-00005d9a3845"
 					(reference "#PWR0108")
@@
 		)
 		(instances
-			(project "Atlas-clone"
+			(project "fome-mc"
 				(path "/3b9c5ffd-e59b-402d-8c5e-052f7ca643a4/00000000-0000-0000-0000-00005d9a3845"
 					(reference "#PWR0109")
@@
 		)
 		(instances
-			(project "Atlas-clone"
+			(project "fome-mc"
 				(path "/3b9c5ffd-e59b-402d-8c5e-052f7ca643a4/00000000-0000-0000-0000-00005d9a3845"
 					(reference "#PWR0110")
@@
 		)
 		(instances
-			(project "Atlas-clone"
+			(project "fome-mc"
 				(path "/3b9c5ffd-e59b-402d-8c5e-052f7ca643a4/00000000-0000-0000-0000-00005d9a3845"
 					(reference "U17")
@@
 		)
 		(instances
-			(project "Atlas-clone"
+			(project "fome-mc"
 				(path "/3b9c5ffd-e59b-402d-8c5e-052f7ca643a4/00000000-0000-0000-0000-00005d9a3845"
 					(reference "RN2")
@@
 		)
 		(instances
-			(project "Atlas-clone"
+			(project "fome-mc"
 				(path "/3b9c5ffd-e59b-402d-8c5e-052f7ca643a4/00000000-0000-0000-0000-00005d9a3845"
 					(reference "R51")
@@
 		)
 		(instances
-			(project "Atlas-clone"
+			(project "fome-mc"
 				(path "/3b9c5ffd-e59b-402d-8c5e-052f7ca643a4/00000000-0000-0000-0000-00005d9a3845"
 					(reference "C46")
@@
 		)
 		(instances
-			(project "Atlas-clone"
+			(project "fome-mc"
 				(path "/3b9c5ffd-e59b-402d-8c5e-052f7ca643a4/00000000-0000-0000-0000-00005d9a3845"
 					(reference "#PWR0104")
@@
 		)
 		(instances
-			(project "Atlas-clone"
+			(project "fome-mc"
 				(path "/3b9c5ffd-e59b-402d-8c5e-052f7ca643a4/00000000-0000-0000-0000-00005d9a3845"
 					(reference "#PWR0111")
@@
 		)
 		(instances
-			(project "Atlas-clone"
+			(project "fome-mc"
 				(path "/3b9c5ffd-e59b-402d-8c5e-052f7ca643a4/00000000-0000-0000-0000-00005d9a3845"
 					(reference "#PWR0112")
@@
 		)
 		(instances
-			(project "Atlas-clone"
+			(project "fome-mc"
 				(path "/3b9c5ffd-e59b-402d-8c5e-052f7ca643a4/00000000-0000-0000-0000-00005d9a3845"
 					(reference "#PWR0115")
@@
 		)
 		(instances
-			(project "Atlas-clone"
+			(project "fome-mc"
 				(path "/3b9c5ffd-e59b-402d-8c5e-052f7ca643a4/00000000-0000-0000-0000-00005d9a3845"
 					(reference "#PWR0103")
@@
 		)
 		(instances
-			(project "Atlas-clone"
+			(project "fome-mc"
 				(path "/3b9c5ffd-e59b-402d-8c5e-052f7ca643a4/00000000-0000-0000-0000-00005d9a3845"
 					(reference "R55")
@@
 		)
 		(instances
-			(project "Atlas-clone"
+			(project "fome-mc"
 				(path "/3b9c5ffd-e59b-402d-8c5e-052f7ca643a4/00000000-0000-0000-0000-00005d9a3845"
 					(reference "R56")
@@
 		)
 		(instances
-			(project "Atlas-clone"
+			(project "fome-mc"
 				(path "/3b9c5ffd-e59b-402d-8c5e-052f7ca643a4/00000000-0000-0000-0000-00005d9a3845"
 					(reference "R57")
@@
 		)
 		(instances
-			(project "Atlas-clone"
+			(project "fome-mc"
 				(path "/3b9c5ffd-e59b-402d-8c5e-052f7ca643a4/00000000-0000-0000-0000-00005d9a3845"
 					(reference "R58")
@@
 		)
 		(instances
-			(project "Atlas-clone"
+			(project "fome-mc"
 				(path "/3b9c5ffd-e59b-402d-8c5e-052f7ca643a4/00000000-0000-0000-0000-00005d9a3845"
 					(reference "R59")
@@
 		)
 		(instances
-			(project "Atlas-clone"
+			(project "fome-mc"
 				(path "/3b9c5ffd-e59b-402d-8c5e-052f7ca643a4/00000000-0000-0000-0000-00005d9a3845"
 					(reference "R60")
@@
 		)
 		(instances
-			(project "Atlas-clone"
+			(project "fome-mc"
 				(path "/3b9c5ffd-e59b-402d-8c5e-052f7ca643a4/00000000-0000-0000-0000-00005d9a3845"
 					(reference "R61")
@@
 		)
 		(instances
-			(project "Atlas-clone"
+			(project "fome-mc"
 				(path "/3b9c5ffd-e59b-402d-8c5e-052f7ca643a4/00000000-0000-0000-0000-00005d9a3845"
 					(reference "R62")
@@
 		)
 		(instances
-			(project "Atlas-clone"
+			(project "fome-mc"
 				(path "/3b9c5ffd-e59b-402d-8c5e-052f7ca643a4/00000000-0000-0000-0000-00005d9a3845"
 					(reference "C47")
@@
 		)
 		(instances
-			(project "Atlas-clone"
+			(project "fome-mc"
 				(path "/3b9c5ffd-e59b-402d-8c5e-052f7ca643a4/00000000-0000-0000-0000-00005d9a3845"
 					(reference "C48")
@@
 		)
 		(instances
-			(project "Atlas-clone"
+			(project "fome-mc"
 				(path "/3b9c5ffd-e59b-402d-8c5e-052f7ca643a4/00000000-0000-0000-0000-00005d9a3845"
 					(reference "C49")
@@
 		)
 		(instances
-			(project "Atlas-clone"
+			(project "fome-mc"
 				(path "/3b9c5ffd-e59b-402d-8c5e-052f7ca643a4/00000000-0000-0000-0000-00005d9a3845"
 					(reference "C50")
@@
 		)
 		(instances
-			(project "Atlas-clone"
+			(project "fome-mc"
 				(path "/3b9c5ffd-e59b-402d-8c5e-052f7ca643a4/00000000-0000-0000-0000-00005d9a3845"
 					(reference "U18")
@@
 		)
 		(instances
-			(project "Atlas-clone"
+			(project "fome-mc"
 				(path "/3b9c5ffd-e59b-402d-8c5e-052f7ca643a4/00000000-0000-0000-0000-00005d9a3845"
 					(reference "#PWR0114")
@@
 		)
 		(instances
-			(project "Atlas-clone"
+			(project "fome-mc"
 				(path "/3b9c5ffd-e59b-402d-8c5e-052f7ca643a4/00000000-0000-0000-0000-00005d9a3845"
 					(reference "#PWR0113")
