File: triggers.kicad_sch (KiCad schematic)
At the start: 39 parts, among them U10 SN74LVC2G17DB, U11 SRV05-4, U12 SRV05-4, U13 SRV05-4, U14 SN74LVC2G17DB, U8 SN74LVC2G17DB, U9 SN74LVC2G17DB

Commit message: Remove all legacy Atlas-clone files/references and standardize on fome-mc
Other:
- title: Atlas-clone -> fome-mc
