File: fome-mc.kicad_pcb (KiCad board)
At the start: 4 copper layers, 162 x 115 mm, 474 parts, among them IC1 PSM712-LF-T7, J1 TE_776163-1, J11 Conn_01x06, J12 Conn_01x02, J13 USB_B, J14 USB_B, J15 Conn_01x01, J16 Conn_01x01, J2 TE_776163-2, J8 Conn_02x05_Odd_Even, J9 Conn_01x06, Q201 FGD3040G2-F085, Q202 FGD3040G2-F085, Q203 FGD3040G2-F085, Q204 FGD3040G2-F085, Q301 VND14NV04, Q401 VND14NV04, SW1 SW_Push, SW2 SW_Push, U1 TLS115D0E, U10 SN74LVC2G17DB, U1001 VNLD5090, U1002 VNLD5090, U11 SRV05-4, U1101 VNLD5090, U1102 VNLD5090, U12 SRV05-4, U1201 VNLD5090, U1202 VNLD5090, U13 SRV05-4, U14 SN74LVC2G17DB, U15 MCP6004, U16 SRV05-4, U17 MCP6004, U18 SRV05-4, U19 MCP6004, U2 TLS115D0E, U20 SRV05-4, U201 TLE9201SG, U202 DRV8825PWPR, U203 TLE9201SG, U21 MCP6004, U22 SRV05-4, U23 REF3333, U24 LPS25HB, U25 CSNP32GCR01-AOW, U26 STM32H753ZIT6, U27 USBLC6-2SC6, U28 S3225SMD32.768KOSC, U3 LMR14020, U301 MCP6004, U302 STM32F042K6Tx, U303 REF3033, U305 AD8628, U307 TJA1051T-3, U309 XC6206P332MR, U4 MCP2551-I-SN, U40 BTS716G, U401 MCP6004, U402 STM32F042K6Tx, U403 REF3033, U405 AD8628, U407 TJA1051T-3, U409 XC6206P332MR, U41 MIC5205-3.3YM5, U42 MIC4427, U43 MIC4427, U44 MIC4427, U45 MIC4427, U46 LM2733XMFX/NOPB, U5 MCP2551-I-SN, U6 AMS1117-3.3, U7 MCP6004, U8 SN74LVC2G17DB, U9 SN74LVC2G17DB, Y1 8MHz

Commit message: Re-integrate ATWINC1500-MR210UB Wi-Fi on SPI4 and remap WBO1/2 reset/boot pins (FOMEMC-2)
Parts:
- added U29: ATWINC1500-MR210UB, ampseal:ATWINC1500-MR210UB, F.Cu at (40.0, 134.0)
- R122: value 68k -> 10k
- moved R122 126.9 mm to (40.0, 120.0)
- moved C106 126.5 mm to (44.0, 120.0)
Connections:
- C106 pad 1: Net-(U28-GND) -> (no net)
- C106 pad 2: unconnected-(C106-Pad2) -> (no net)
- R122 pad 1: Net-(U46-OUT) -> (no net)
- R122 pad 2: unconnected-(R122-Pad2) -> (no net)
