File: sheets/wbo1.kicad_sch (KiCad schematic)
At the start: 58 parts, among them Q301 VND14NV04, U301 MCP6004, U302 STM32F042K6Tx, U303 REF3033, U305 AD8628, U307 TJA1051T-3, U309 XC6206P332MR

Commit message: Remediate power supply, main relay keep-alive, and schematic ERC to 0 errors
Connections:
- net +3V3 is gone; now on net +3V3_WBO1: U307.5 (VIO)
- net VDDA renamed VDDA_WBO1

Commit message: Complete FOMEMC-11, FOMEMC-12, and FOMEMC-16: sync 492 PCB footprints, restore min_resolved_spokes=2 (0 starved thermals), enable teardrops, enforce >=1.2mm IGBT collector clearance, widen /IGN1..4_COIL, add WBO heater copper zones, and refresh CPL/BOM/renders
Connections:
- no-connect marks 8 -> 7
Changed lines of the file:
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@@
-	)
-	(no_connect
-		(at 269.875 38.1)
 	)
 	(no_connect

Commit message: Remediate FOMEMC-17..20: 50V X7R PSU caps & 42V INJ clamp DNP, U29 DS70005304F footprint + 1P3V bypass, HV_IGN 0.50mm clearance + U25 decoupling, and 0 ERC violations
Connections:
- net SEL_2: no longer names the net of U302.18 (PA8)
- net SWCLK: no longer names the net of U302.24 (PA14)
- net SWDIO: no longer names the net of U302.23 (PA13)
- no-connect marks 7 -> 10
