File: sheets/etb-9201.kicad_sch (KiCad schematic)
At the start: 5 parts, among them U201 TLE9201SG

Commit message: Remediate power supply, main relay keep-alive, and schematic ERC to 0 errors
Parts:
- C1201: value 10u -> 2.2u; LCSC C13585 -> C90787; LCSC_ext 0 -> (none); PN (none) -> GCJ31CR71H225KA12L
Changed lines of the file:
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@@
       (effects (font (size 1.27 1.27)) (justify left))
     )
-    (property "Value" "10u" (id 1) (at 59.436 27.813 0)
+    (property "Value" "2.2u" (id 1) (at 59.436 27.813 0)
       (effects (font (size 1.27 1.27)) (justify left))
     )
@@
       (effects (font (size 1.27 1.27)) hide)
     )
-    (property "LCSC" "C13585" (id 4) (at 56.515 26.67 0)
+    (property "LCSC" "C90787" (id 4) (at 56.515 26.67 0)
       (effects (font (size 1.27 1.27)) hide)
     )
-    (property "LCSC_ext" "0" (id 5) (at 56.515 26.67 0)
+    (property "PN" "GCJ31CR71H225KA12L" (id 5) (at 56.515 26.67 0)
       (effects (font (size 1.27 1.27)) hide)
     )
@@
       (effects (font (size 1.27 1.27)) hide)
     )
-    (property "Value" "+3.3V" (id 1) (at 87.7062 54.991 90)
+    (property "Value" "+3V3" (id 1) (at 87.7062 54.991 90)
       (effects (font (size 1.27 1.27)) (justify left))
     )
@@
       (effects (font (size 1.27 1.27)) hide)
     )
-    (property "Value" "+3.3V" (id 1) (at 37.3888 36.449 90)
+    (property "Value" "+3V3" (id 1) (at 37.3888 36.449 90)
       (effects (font (size 1.27 1.27)) (justify left))
     )

Commit message: Remediate FOMEMC-22..27: sheet contracts, doc/BOM/netlist parity, 494-part BOM/CPL, Mode A2 VR + C38/C39, wide WBO heater buses, and 4x M4 holes with 0 DRC warnings
Parts:
- C201, C202: LCSC C57112 -> C344025
Changed lines of the file:
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@@
       (effects (font (size 1.27 1.27)) hide)
     )
-    (property "LCSC" "C57112" (id 5) (at 88.9 28.575 0)
+    (property "LCSC" "C344025" (id 5) (at 88.9 28.575 0)
       (effects (font (size 1.27 1.27)) hide)
     )
@@
       (effects (font (size 1.27 1.27)) hide)
     )
-    (property "LCSC" "C57112" (id 5) (at 88.9 40.005 0)
+    (property "LCSC" "C344025" (id 5) (at 88.9 40.005 0)
       (effects (font (size 1.27 1.27)) hide)
     )
