File: sheets/highside_quad.kicad_sch (KiCad schematic)
At the start: 14 parts, among them U40 BTS716G

Commit message: Remediate FOMEMC-22..27: sheet contracts, doc/BOM/netlist parity, 494-part BOM/CPL, Mode A2 VR + C38/C39, wide WBO heater buses, and 4x M4 holes with 0 DRC warnings
Parts:
- C85, C86, C87, C88: LCSC C57112 -> C344025
Changed lines of the file:
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@@
 			)
 		)
-		(property "LCSC" "C57112"
+		(property "LCSC" "C344025"
 			(at 101.6 47.625 0)
 			(effects
@@
 			)
 		)
-		(property "LCSC" "C57112"
+		(property "LCSC" "C344025"
 			(at 101.6 74.295 0)
 			(effects
@@
 			)
 		)
-		(property "LCSC" "C57112"
+		(property "LCSC" "C344025"
 			(at 101.6 132.715 0)
 			(effects
@@
 			)
 		)
-		(property "LCSC" "C57112"
+		(property "LCSC" "C344025"
 			(at 101.6 103.505 0)
 			(effects
