File: sheets/ign4.kicad_sch (KiCad schematic)
At the start: 16 parts, among them U42 MIC4427, U43 MIC4427

Commit message: Remediate FOMEMC-22..27: sheet contracts, doc/BOM/netlist parity, 494-part BOM/CPL, Mode A2 VR + C38/C39, wide WBO heater buses, and 4x M4 holes with 0 DRC warnings
Parts:
- C91, C92: LCSC C14663 -> C161115
- C93, C94, C95, C96: LCSC C57112 -> C344025
Changed lines of the file:
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@@
 			)
 		)
-		(property "LCSC" "C14663"
+		(property "LCSC" "C161115"
 			(at 81.28 73.025 0)
 			(effects
@@
 			)
 		)
-		(property "LCSC" "C14663"
+		(property "LCSC" "C161115"
 			(at 81.28 34.29 0)
 			(effects
@@
 			)
 		)
-		(property "LCSC" "C57112"
+		(property "LCSC" "C344025"
 			(at 99.695 55.245 0)
 			(effects
@@
 			)
 		)
-		(property "LCSC" "C57112"
+		(property "LCSC" "C344025"
 			(at 99.695 38.735 0)
 			(effects
@@
 			)
 		)
-		(property "LCSC" "C57112"
+		(property "LCSC" "C344025"
 			(at 99.695 76.835 0)
 			(effects
@@
 			)
 		)
-		(property "LCSC" "C57112"
+		(property "LCSC" "C344025"
 			(at 99.695 93.345 0)
 			(effects
