File: sheets/knock.kicad_sch (KiCad schematic)
At the start: 24 parts, among them U7 MCP6004

Commit message: Remediate FOMEMC-22..27: sheet contracts, doc/BOM/netlist parity, 494-part BOM/CPL, Mode A2 VR + C38/C39, wide WBO heater buses, and 4x M4 holes with 0 DRC warnings
Parts:
- C15: LCSC C57112 -> C344025
- JP1, JP2: now not fitted; now left out of the parts list
Changed lines of the file:
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@@
 			)
 		)
-		(property "LCSC" "C57112"
+		(property "LCSC" "C344025"
 			(at 26.67 100.965 0)
 			(effects
@@
 		(unit 1)
 		(exclude_from_sim no)
-		(in_bom yes)
-		(on_board yes)
-		(dnp no)
+		(in_bom no)
+		(on_board yes)
+		(dnp yes)
 		(property "Reference" "JP1"
 			(at 46.99 38.735 0)
@@
 		(unit 1)
 		(exclude_from_sim no)
-		(in_bom yes)
-		(on_board yes)
-		(dnp no)
+		(in_bom no)
+		(on_board yes)
+		(dnp yes)
 		(property "Reference" "JP2"
 			(at 46.99 75.565 0)
