File: sheets/psu.kicad_sch (KiCad schematic)
At the start: 42 parts, among them U1 TLS115D0E, U2 TLS115D0E, U3 LMR14020, U4 MCP2551-I-SN, U46 LM2733XMFX/NOPB, U5 MCP2551-I-SN, U6 AMS1117-3.3

Commit message: Remediate power supply, main relay keep-alive, and schematic ERC to 0 errors
Parts:
- removed C107: 4.7u, Capacitor_SMD:C_0603_1608Metric, symbol Device:C_Small
- removed D18, D2: D_Schottky, Diode_SMD:D_SMA, symbol Device:D_Schottky
- removed L3: 10u, sunlord-MWSA0503:MWSA0503, symbol Device:L
- removed R122: 68k, Resistor_SMD:R_0402_1005Metric, symbol Device:R_Small
- removed R123: 10k, Resistor_SMD:R_0402_1005Metric, symbol Device:R_Small
- removed U46: LM2733XMFX/NOPB, Package_TO_SOT_SMD:SOT-23-5, symbol Regulator_Linear:MIC5205-3.3YM5
- added C108: 100n, Capacitor_SMD:C_0603_1608Metric, symbol Device:C
- added D19: BZT52C12, Diode_SMD:D_SOD-123, symbol Device:D_Zener
- added Q1: AO4485, Package_SO:SOIC-8_3.9x4.9mm_P1.27mm, symbol Transistor_FET:IRF7404
- added R124: 47k, Resistor_SMD:R_0603_1608Metric, symbol Device:R
- C12: footprint Capacitor_SMD:C_1206_3216Metric -> Capacitor_SMD:C_0603_1608Metric; LCSC C13585 -> C161115; PN (none) -> GCJ188R71H104KA12D
- D1: value SM15T33CA -> SMCJ33A; symbol Device:D_TVS -> Device:D_Zener; LCSC C151281 -> C224049; PN SM15T33CA -> SMCJ33A
- U3: value LMR14020 -> LMR16020PDDAR; LCSC C187824 -> C190006; PN LMR14020 -> LMR16020PDDAR
- U6: value AMS1117-3.3 -> TLV75733PDBVR; footprint Package_TO_SOT_SMD:SOT-223-3_TabPin2 -> Package_TO_SOT_SMD:SOT-23-5; symbol Regulator_Linear:AMS1117-3.3 -> Regulator_Linear:TLV75733PDBV; LCSC C6186 -> C485517; LCSC_ext 0 -> (none); PN (none) -> TLV75733PDBVR
Connections:
- net +3V3: now also U6.5 (OUT); no longer U4.5 (Vref), U5.5 (Vref), U6.2 (VO)
- net +5V: now also U6.1 (IN)
- net 12V_RAW: now also C108.1, Q1.5 (D), Q1.6 (D), Q1.7 (D), Q1.8 (D)
- net 12v_PROT: now also D19.1 (K), Q1.1 (S), Q1.2 (S), Q1.3 (S)
- net GND: now also U6.2 (GND), C108.2, R124.2; no longer U6.1 (GND)
- new net: D19.2 (A), Q1.4 (G), R124.1
- no-connect marks 0 -> 3

Commit message: Add D210 BZT52C6V8 BOOT0 threshold Zener, R217/R218/D211 PA9 VBUS sense divider/clamp, and SMCJ24A TVS protection on 12V_RAW and 12V_MR (FOMEMC-7)
Parts:
- D1: value SMCJ33A -> SMCJ24A; LCSC C224049 -> C224045; PN SMCJ33A -> SMCJ24A
Changed lines of the file:
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@@
 			)
 		)
-		(property "Value" "SMCJ33A"
+		(property "Value" "SMCJ24A"
 			(at 33.7566 35.433 90)
 			(effects
@@
 			)
 		)
-		(property "Description" "1500W 33V Unidirectional SMC TVS Diode (53.3V max clamp)"
+		(property "Description" "1500W 24V Unidirectional SMC TVS Diode (38.9V max clamp)"
 			(at 31.75 34.29 0)
 			(effects
@@
 			)
 		)
-		(property "PN" "SMCJ33A"
+		(property "PN" "SMCJ24A"
 			(at 31.75 34.29 0)
 			(effects
@@
 			)
 		)
-		(property "LCSC" "C224049"
+		(property "LCSC" "C224045"
 			(at 31.75 34.29 0)
 			(effects

Commit message: Complete FOMEMC-11, FOMEMC-12, and FOMEMC-16: sync 492 PCB footprints, restore min_resolved_spokes=2 (0 starved thermals), enable teardrops, enforce >=1.2mm IGBT collector clearance, widen /IGN1..4_COIL, add WBO heater copper zones, and refresh CPL/BOM/renders
Parts:
- C12: LCSC C161115 -> C96446; PN GCJ188R71H104KA12D -> CL10A106MA8NRNC
Changed lines of the file:
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@@
 			)
 		)
-		(property "Description" "100nF 50V X7R 0603 Soft-Terminated (Flex-Term) AEC-Q200 MLCC"
+		(property "Description" "10uF 25V X5R 0603 MLCC"
 			(at 186.055 35.56 0)
 			(effects
@@
 			)
 		)
-		(property "PN" "GCJ188R71H104KA12D"
+		(property "PN" "CL10A106MA8NRNC"
 			(at 186.055 35.56 0)
 			(effects
@@
 			)
 		)
-		(property "LCSC" "C161115"
+		(property "LCSC" "C96446"
 			(at 186.055 35.56 0)
 			(effects

Commit message: Remediate FOMEMC-17..20: 50V X7R PSU caps & 42V INJ clamp DNP, U29 DS70005304F footprint + 1P3V bypass, HV_IGN 0.50mm clearance + U25 decoupling, and 0 ERC violations
Parts:
- C10: LCSC C14663 -> C161115
- C2, C5, C7: footprint Capacitor_SMD:C_0603_1608Metric -> Capacitor_SMD:C_0805_2012Metric; LCSC C15849 -> C354368
- C4: footprint Capacitor_SMD:C_0603_1608Metric -> Capacitor_SMD:C_1210_3225Metric; LCSC C19666 -> C417122
- C8: LCSC C57112 -> C344025
Connections:
- net 12v_PROT renamed 12V_PROT
Changed lines of the file:
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@@
 		)
 	)
-	(label "12v_PROT"
+	(label "12V_PROT"
 		(at 20.32 72.39 0)
 		(fields_autoplaced yes)
@@
 		)
 	)
-	(label "12v_PROT"
+	(label "12V_PROT"
 		(at 72.39 29.21 0)
 		(fields_autoplaced yes)
@@
 		)
 	)
-	(label "12v_PROT"
+	(label "12V_PROT"
 		(at 93.345 72.39 0)
 		(fields_autoplaced yes)
@@
 		)
 	)
-	(hierarchical_label "12v_PROT"
+	(hierarchical_label "12V_PROT"
 		(shape output)
 		(at 71.755 31.115 270)
@@
 			)
 		)
-		(property "Footprint" "Capacitor_SMD:C_0603_1608Metric"
+		(property "Footprint" "Capacitor_SMD:C_0805_2012Metric"
 			(at 109.5502 39.37 0)
 			(effects
@@
 			)
 		)
-		(property "Description" ""
+		(property "Description" "1uF 50V X7R 0805 Murata GCJ21BR71H105KA01L Soft-Terminated AEC-Q200"
 			(at 108.585 35.56 0)
 			(effects
@@
 			)
 		)
-		(property "LCSC" "C15849"
+		(property "LCSC" "C354368"
 			(at 108.585 35.56 0)
 			(effects
@@
 			)
 		)
-		(property "Footprint" "Capacitor_SMD:C_0603_1608Metric"
+		(property "Footprint" "Capacitor_SMD:C_1210_3225Metric"
 			(at 88.5952 46.355 0)
 			(effects
@@
 			)
 		)
-		(property "Description" ""
+		(property "Description" "4.7uF 50V X7R 1210 Murata GCJ32ER71H475KA12L Soft-Terminated AEC-Q200"
 			(at 87.63 42.545 0)
 			(effects
@@
 			)
 		)
-		(property "LCSC" "C19666"
+		(property "LCSC" "C417122"
 			(at 87.63 42.545 0)
 			(effects
@@
 			)
 		)
-		(property "Footprint" "Capacitor_SMD:C_0603_1608Metric"
+		(property "Footprint" "Capacitor_SMD:C_0805_2012Metric"
 			(at 21.2852 85.09 0)
 			(effects
@@
 			)
 		)
-		(property "Description" ""
+		(property "Description" "1uF 50V X7R 0805 Murata GCJ21BR71H105KA01L Soft-Terminated AEC-Q200"
 			(at 20.32 81.28 0)
 			(effects
@@
 			)
 		)
-		(property "LCSC" "C15849"
+		(property "LCSC" "C354368"
 			(at 20.32 81.28 0)
 			(effects
@@
 			)
 		)
-		(property "Footprint" "Capacitor_SMD:C_0603_1608Metric"
+		(property "Footprint" "Capacitor_SMD:C_0805_2012Metric"
 			(at 94.3102 85.09 0)
 			(effects
@@
 			)
 		)
-		(property "Description" ""
+		(property "Description" "1uF 50V X7R 0805 Murata GCJ21BR71H105KA01L Soft-Terminated AEC-Q200"
 			(at 93.345 81.28 0)
 			(effects
@@
 			)
 		)
-		(property "LCSC" "C15849"
+		(property "LCSC" "C354368"
 			(at 93.345 81.28 0)
 			(effects
@@
 			)
 		)
-		(property "Description" ""
+		(property "Description" "100nF 50V X7R 0603 Murata GCJ188R71H104KA12D Soft-Terminated AEC-Q200"
 			(at 152.4 32.385 0)
 			(effects
@@
 			)
 		)
-		(property "LCSC" "C14663"
+		(property "LCSC" "C161115"
 			(at 152.4 32.385 0)
 			(effects
@@
 			)
 		)
-		(property "Description" ""
+		(property "Description" "10nF 50V X7R 0603 Murata GCJ188R71H103KA01D Soft-Terminated AEC-Q200"
 			(at 126.365 48.895 0)
 			(effects
@@
 			)
 		)
-		(property "LCSC" "C57112"
+		(property "LCSC" "C344025"
 			(at 126.365 48.895 0)
 			(effects

Commit message: Remediate FOMEMC-22..27: sheet contracts, doc/BOM/netlist parity, 494-part BOM/CPL, Mode A2 VR + C38/C39, wide WBO heater buses, and 4x M4 holes with 0 DRC warnings
Parts:
- R7, R8: LCSC C22787 -> C22859
Changed lines of the file:
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@@
 			)
 		)
-		(property "LCSC" "C22787"
+		(property "LCSC" "C22859"
 			(at 173.978 88.8557 0)
 			(effects
@@
 			)
 		)
-		(property "LCSC" "C22787"
+		(property "LCSC" "C22859"
 			(at 175.2592 132.663 0)
 			(effects
