File: sheets/quad_analog.kicad_sch (KiCad schematic)
At the start: 20 parts, among them U17 MCP6004, U18 SRV05-4

Commit message: Remediate FOMEMC-22..27: sheet contracts, doc/BOM/netlist parity, 494-part BOM/CPL, Mode A2 VR + C38/C39, wide WBO heater buses, and 4x M4 holes with 0 DRC warnings
Parts:
- C46: LCSC C14663 -> C161115
Changed lines of the file:
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@@
 			)
 		)
-		(property "LCSC" "C14663"
+		(property "LCSC" "C161115"
 			(at 29.845 42.545 0)
 			(effects
