File: sheets/stepper_etb.kicad_sch (KiCad schematic)
At the start: 26 parts, among them U202 DRV8825PWPR, U203 TLE9201SG

Commit message: Remediate FOMEMC-17..20: 50V X7R PSU caps & 42V INJ clamp DNP, U29 DS70005304F footprint + 1P3V bypass, HV_IGN 0.50mm clearance + U25 decoupling, and 0 ERC violations
Parts:
- D201, D202, D203, D204: now not fitted; now left out of the parts list
Other:
- note added: "D201..D204: DNP on INJ1..4 (/LS1../LS4) so U1001/U1002 VNLD5090TR-E use internal 42V active clamp for fast injector turn-off. D205..D209: Populated on LS5..LS8 & MAIN_RLY inductive relay/solenoid channels."
Changed lines of the file:
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@@
 		(instances
-			(project "fome-mc" (path "/3b9c5ffd-e59b-402d-8c5e-052f7ca643a4/a1000000-0000-4000-8000-000000000002" (reference "U203") (unit 1)))
 			(project "fome-mc" (path "/3b9c5ffd-e59b-402d-8c5e-052f7ca643a4/a1000000-0000-4000-8000-000000000002" (reference "U203") (unit 1)))
 		)
@@
 		(instances
 			(project "fome-mc" (path "/3b9c5ffd-e59b-402d-8c5e-052f7ca643a4/a1000000-0000-4000-8000-000000000002" (reference "#PWR0854") (unit 1)))
-			(project "fome-mc" (path "/3b9c5ffd-e59b-402d-8c5e-052f7ca643a4/a1000000-0000-4000-8000-000000000002" (reference "#PWR0854") (unit 1)))
 		)
 	)
@@
 		(instances
 			(project "fome-mc" (path "/3b9c5ffd-e59b-402d-8c5e-052f7ca643a4/a1000000-0000-4000-8000-000000000002" (reference "#PWR0855") (unit 1)))
-			(project "fome-mc" (path "/3b9c5ffd-e59b-402d-8c5e-052f7ca643a4/a1000000-0000-4000-8000-000000000002" (reference "#PWR0855") (unit 1)))
 		)
 	)
@@
 		(instances
 			(project "fome-mc" (path "/3b9c5ffd-e59b-402d-8c5e-052f7ca643a4/a1000000-0000-4000-8000-000000000002" (reference "#PWR0856") (unit 1)))
-			(project "fome-mc" (path "/3b9c5ffd-e59b-402d-8c5e-052f7ca643a4/a1000000-0000-4000-8000-000000000002" (reference "#PWR0856") (unit 1)))
-		)
+		)
+	)
+	(text "D201..D204: DNP on INJ1..4 (/LS1../LS4) so U1001/U1002 VNLD5090TR-E use internal 42V active clamp for fast injector turn-off.\nD205..D209: Populated on LS5..LS8 & MAIN_RLY inductive relay/solenoid channels."
+		(exclude_from_sim no)
+		(at 129.54 22.86 0)
+		(effects (font (size 1.27 1.27)) (justify left))
 	)
 	(symbol
@@
 		(unit 1)
 		(exclude_from_sim no)
-		(in_bom yes)
-		(on_board yes)
-		(dnp no)
+		(in_bom no)
+		(on_board yes)
+		(dnp yes)
 		(property "Reference" "D201" (at 139.7 27.94 0) (effects (font (size 1.27 1.27))))
 		(property "Value" "B340A-13-F" (at 139.7 33.02 0) (effects (font (size 1.27 1.27))))
@@
 		(instances
 			(project "fome-mc" (path "/3b9c5ffd-e59b-402d-8c5e-052f7ca643a4/a1000000-0000-4000-8000-000000000002" (reference "D201") (unit 1)))
-			(project "fome-mc" (path "/3b9c5ffd-e59b-402d-8c5e-052f7ca643a4/a1000000-0000-4000-8000-000000000002" (reference "D201") (unit 1)))
 		)
 	)
@@
 		(unit 1)
 		(exclude_from_sim no)
-		(in_bom yes)
-		(on_board yes)
-		(dnp no)
+		(in_bom no)
+		(on_board yes)
+		(dnp yes)
 		(property "Reference" "D202" (at 139.7 38.1 0) (effects (font (size 1.27 1.27))))
 		(property "Value" "B340A-13-F" (at 139.7 43.18 0) (effects (font (size 1.27 1.27))))
@@
 		(instances
 			(project "fome-mc" (path "/3b9c5ffd-e59b-402d-8c5e-052f7ca643a4/a1000000-0000-4000-8000-000000000002" (reference "D202") (unit 1)))
-			(project "fome-mc" (path "/3b9c5ffd-e59b-402d-8c5e-052f7ca643a4/a1000000-0000-4000-8000-000000000002" (reference "D202") (unit 1)))
 		)
 	)
@@
 		(unit 1)
 		(exclude_from_sim no)
-		(in_bom yes)
-		(on_board yes)
-		(dnp no)
+		(in_bom no)
+		(on_board yes)
+		(dnp yes)
 		(property "Reference" "D203" (at 139.7 48.26 0) (effects (font (size 1.27 1.27))))
 		(property "Value" "B340A-13-F" (at 139.7 53.339999999999996 0) (effects (font (size 1.27 1.27))))
@@
 		(instances
 			(project "fome-mc" (path "/3b9c5ffd-e59b-402d-8c5e-052f7ca643a4/a1000000-0000-4000-8000-000000000002" (reference "D203") (unit 1)))
-			(project "fome-mc" (path "/3b9c5ffd-e59b-402d-8c5e-052f7ca643a4/a1000000-0000-4000-8000-000000000002" (reference "D203") (unit 1)))
 		)
 	)
@@
 		(unit 1)
 		(exclude_from_sim no)
-		(in_bom yes)
-		(on_board yes)
-		(dnp no)
+		(in_bom no)
+		(on_board yes)
+		(dnp yes)
 		(property "Reference" "D204" (at 139.7 58.42 0) (effects (font (size 1.27 1.27))))
 		(property "Value" "B340A-13-F" (at 139.7 63.5 0) (effects (font (size 1.27 1.27))))
@@
 		(instances
 			(project "fome-mc" (path "/3b9c5ffd-e59b-402d-8c5e-052f7ca643a4/a1000000-0000-4000-8000-000000000002" (reference "D204") (unit 1)))
-			(project "fome-mc" (path "/3b9c5ffd-e59b-402d-8c5e-052f7ca643a4/a1000000-0000-4000-8000-000000000002" (reference "D204") (unit 1)))
 		)
 	)
@@
 		(instances
 			(project "fome-mc" (path "/3b9c5ffd-e59b-402d-8c5e-052f7ca643a4/a1000000-0000-4000-8000-000000000002" (reference "D205") (unit 1)))
-			(project "fome-mc" (path "/3b9c5ffd-e59b-402d-8c5e-052f7ca643a4/a1000000-0000-4000-8000-000000000002" (reference "D205") (unit 1)))
 		)
 	)
@@
 		(instances
 			(project "fome-mc" (path "/3b9c5ffd-e59b-402d-8c5e-052f7ca643a4/a1000000-0000-4000-8000-000000000002" (reference "D206") (unit 1)))
-			(project "fome-mc" (path "/3b9c5ffd-e59b-402d-8c5e-052f7ca643a4/a1000000-0000-4000-8000-000000000002" (reference "D206") (unit 1)))
 		)
 	)
@@
 		(instances
 			(project "fome-mc" (path "/3b9c5ffd-e59b-402d-8c5e-052f7ca643a4/a1000000-0000-4000-8000-000000000002" (reference "D207") (unit 1)))
-			(project "fome-mc" (path "/3b9c5ffd-e59b-402d-8c5e-052f7ca643a4/a1000000-0000-4000-8000-000000000002" (reference "D207") (unit 1)))
 		)
 	)
@@
 		(instances
 			(project "fome-mc" (path "/3b9c5ffd-e59b-402d-8c5e-052f7ca643a4/a1000000-0000-4000-8000-000000000002" (reference "D208") (unit 1)))
-			(project "fome-mc" (path "/3b9c5ffd-e59b-402d-8c5e-052f7ca643a4/a1000000-0000-4000-8000-000000000002" (reference "D208") (unit 1)))
 		)
 	)
@@
 		(instances
 			(project "fome-mc" (path "/3b9c5ffd-e59b-402d-8c5e-052f7ca643a4/a1000000-0000-4000-8000-000000000002" (reference "R212") (unit 1)))
-			(project "fome-mc" (path "/3b9c5ffd-e59b-402d-8c5e-052f7ca643a4/a1000000-0000-4000-8000-000000000002" (reference "R212") (unit 1)))
-		)
+		)

Commit message: Remediate FOMEMC-22..27: sheet contracts, doc/BOM/netlist parity, 494-part BOM/CPL, Mode A2 VR + C38/C39, wide WBO heater buses, and 4x M4 holes with 0 DRC warnings
Parts:
- C203: LCSC C57112 -> C344025
Changed lines of the file:
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@@
 		(property "Value" "10n" (at 86.36 38.1 0) (effects (font (size 1.27 1.27))))
 		(property "Footprint" "Capacitor_SMD:C_0603_1608Metric" (at 86.36 35.56 0) (effects (font (size 1.27 1.27)) (hide yes)))
-		(property "LCSC" "C57112" (at 86.36 35.56 0) (effects (font (size 1.27 1.27)) (hide yes)))
+		(property "LCSC" "C344025" (at 86.36 35.56 0) (effects (font (size 1.27 1.27)) (hide yes)))
 		(pin "1")
 		(pin "2")
