File: sheets/triggers.kicad_sch (KiCad schematic)
At the start: 39 parts, among them U10 SN74LVC2G17DB, U11 SRV05-4, U12 SRV05-4, U13 SRV05-4, U14 SN74LVC2G17DB, U8 SN74LVC2G17DB, U9 SN74LVC2G17DB

Commit message: Add MAX9924UAUB+ (U13/U14) differential VR conditioners and switch Hall Schmitt triggers (U8/U9/U10) to +3V3 (FOMEMC-6)
Parts:
- removed U13: SRV05-4, Package_TO_SOT_SMD:SOT-23-6, symbol Power_Protection:SRV05-4
- removed U14: SN74LVC2G17DB, Package_TO_SOT_SMD:SOT-23-6, symbol 74xGxx:74LVC2G17
- added C109, C110: 100n, Capacitor_SMD:C_0402_1005Metric, symbol Device:C
- added R125, R126: 10k, Resistor_SMD:R_0402_1005Metric, symbol Device:R
- added U13, U14: MAX9924UAUB+, Package_SO:MSOP-10_3x3mm_P0.5mm, symbol Simon:MAX9924
- C36, C37: LCSC_ext 0 -> (none)
- C38, C39: value 1n -> 100n; LCSC C1588 -> C14663; LCSC_ext 0 -> (none)
- R35, R36, R37, R38: value 2.7k -> 10k; footprint Resistor_SMD:R_0603_1608Metric -> Resistor_SMD:R_0402_1005Metric; LCSC C13167 -> C25744; LCSC_ext 0 -> (none)
Connections:
- net +5V: no longer U10.5 (VCC), U10.5 (VCC), U8.5 (VCC), U8.5 (VCC), U9.5 (VCC), U9.5 (VCC)
- net 5V_SENSOR_SUPPLY: now also C109.1, C110.1, U13.10 (VCC), U13.6 (ZERO_EN), U14.10 (VCC), U14.6 (ZERO_EN); no longer R35.1, R36.1
- net GND: now also C38.1, C39.1, C109.2, C110.2, U13.5 (GND), U13.8 (EXT), U13.9 (INT_THRS), U14.5 (GND), U14.8 (EXT), U14.9 (INT_THRS); no longer C36.2, C37.2, C38.2, C39.2
- net VR1: now also R35.1; no longer C37.1, R36.2, R38.2
- net VR1_OUT: now also R125.2, U13.7 (COUT)
- net VR2: now also R37.1; no longer C36.1, R35.2, R37.2
- net VR2_OUT: now also R126.2, U14.7 (COUT)
- net VR2-: now reaches R38.1
- net VR2-: no longer C39.1
- new net: C37.1, R37.2, U14.1 (IN+)
- new net: C36.1, R35.2, U13.1 (IN+)
- new net: C36.2, R36.2, U13.2 (IN-)
- new net: C38.2, U13.4 (BIAS)
- new net: C37.2, R38.2, U14.2 (IN-)
- new net: C39.2, U14.4 (BIAS)
- new net +3V3: R125.1, R126.1, U10.5 (VCC), U10.5 (VCC), U8.5 (VCC), U8.5 (VCC), U9.5 (VCC), U9.5 (VCC)
- new net VR1-: R36.1
- no-connect marks 0 -> 2

Commit message: Remediate FOMEMC-22..27: sheet contracts, doc/BOM/netlist parity, 494-part BOM/CPL, Mode A2 VR + C38/C39, wide WBO heater buses, and 4x M4 holes with 0 DRC warnings
Parts:
- C38, C39: LCSC C14663 -> C161115
Connections:
- net 5V_SENSOR_SUPPLY: now also C38.2, C39.2; no longer U13.6 (ZERO_EN), U14.6 (ZERO_EN)
- net GND: now also U13.4 (BIAS), U13.6 (ZERO_EN), U14.4 (BIAS), U14.6 (ZERO_EN); no longer U13.8 (EXT), U14.8 (EXT)
- no-connect marks 2 -> 4
Other:
- moved on the sheet: C38, C39
