File: telemetry-pod/telemetry-pod.kicad_sch (KiCad schematic)
At the start: 0 parts

Commit message: Commit telemetry-pod v9 90x65 pilot snapshot and 2D/3D renders
- PILOT SNAPSHOT (not a release): commits the owner-approved 4-layer 90x65 mm
  placed-and-routed board (driver-preparation-v9-90x65, board SHA256
  2938ee1ee2cae459c869ee5c4c8443e66322034736fe3fcbf4b5e56377ea1cfa), schematic,
  project files, project-relative symbol/footprint libraries, and 2D/3D renders
  under telemetry-pod/renders/; will be replaced by the clean-main requalified
  board once open items land.
- agent-ee source SHA: a02c952 (main).
- Router provenance: routed with the validated fix content from the rejected
  runtime prototypes kr63 (d7ceadf) and kr64 (670f5c6); mechanism superseded by
  pinning the fork halbritt/KiCadRoutingTools (branch kicad-route-fixes based on
  v0.23.1 295f9ee1, KICADROUTE-65) and filing the two defects upstream.
- Stage-7 status: 12/18 pass + 2/18 info on raw agent-ee a02c952 (15/18 pass/info
  with AGENTEE-275 fab_package overlay); open items tracked under AGENTEE-275,
  AGENTEE-276, KICADROUTE-65, and the upstream ublox_NEO 3D model 404 gap in
  kicad-packages3D.
- fome-mc toolchain checks (make check / make verify-io PROJECT=telemetry-pod):
  - erc: PASS (design_clean=True, 0 violations)
  - drc: PASS (design_clean=True, 0 violations, 0 unconnected, 0 parity issues)
  - netlist: PASS (108 components, 116 nets)
  - analyze (kicad-happy): PASS (108 schematic components, 112 footprints,
    routing_complete=True)
  - export (KiBot 1.9.1): FAIL (exit code 22 parsing agent-ee bare-copper-probe/1
    JSON metadata on TP1..TP6 as a colon-delimited footprint string)
  - verify-io: FAIL (contracts/telemetry-pod.interface.json fails closed per
    FOMEMC-29 until AGENTEE-188 generates it)
Parts:
- added C1, C2, C8, C9: 4.7 uF/100 V, Capacitor_SMD:C_1210_3225Metric, symbol Device:C
- added C10, C3: 220 nF/100 V, Capacitor_SMD:C_0805_2012Metric, symbol Device:C
- added C100: 100n, Capacitor_SMD:C_0402_1005Metric, symbol Block_63616e_446576696365:C
- added C11, C16, C18, C20, C21, C22, C4, C44: 1 uF/16 V, Capacitor_SMD:C_0603_1608Metric, symbol Device:C
- added C12, C30, C32, C34, C36, C38, C39, C41, C42, C43, C5: 100 nF/50 V X7R, Capacitor_SMD:C_0603_1608Metric, symbol Device:C
- added C13, C14, C15, C17, C19, C6, C7: 22 uF/25 V, Capacitor_SMD:C_1210_3225Metric, symbol Device:C
- added C31, C33, C35, C37: 100 pF C0G/50 V, Capacitor_SMD:C_0603_1608Metric, symbol Device:C
- added C40: 470 pF C0G/50 V, Capacitor_SMD:C_0603_1608Metric, symbol Device:C
- added C45: 22uF, Capacitor_SMD:C_1210_3225Metric, symbol Device:C
- added C46, C48, C49, C51, C53: 100nF, Capacitor_SMD:C_0603_1608Metric, symbol Device:C
- added C47, C50, C52: 1uF, Capacitor_SMD:C_0603_1608Metric, symbol Device:C
- added D1: SMCJ24CA, Diode_SMD:D_SMC, symbol Device:D_TVS
- added D100: PESD1CAN-UX, Package_TO_SOT_SMD:SOT-323_SC-70, symbol Block_63616e_446576696365:D_TVS_x2_AAC
- added D2: BZT52C12-7-F, Diode_SMD:D_SOD-123, symbol Device:D_Zener
- added D3: PESD5V0C1BLS-QYL, PodPower:SOD882BD, symbol Device:D_TVS
- added J1: 776228-1, ampseal:ampseal-23, symbol Connector_Generic:Conn_01x23
- added J2: 732511150, Connector_Coaxial:SMA_Molex_73251-1153_EdgeMount_Horizontal, symbol Connector:Conn_Coaxial
- added L1: 15 uH, PodPower:SRP7050TA, symbol Device:L
- added L2: 6.8 uH, PodPower:SRP7050WA, symbol Device:L
- added L3: LQW18AN56NJ00D, Inductor_SMD:L_0603_1608Metric, symbol Device:L
- added Q1: DMP6023LE-13, PodPower:DMP6023LE_SOT223, symbol Transistor_FET:Q_PMOS_GDS
- added R1, R24, R25: 100 kohm, Resistor_SMD:R_0603_1608Metric, symbol Device:R
- added R10, R11, R13, R14, R16, R17, R19, R20, R22, R23, R3, R5: 10 kohm, Resistor_SMD:R_0603_1608Metric, symbol Device:R
- added R100: 120, Resistor_SMD:R_0603_1608Metric, symbol Block_63616e_446576696365:R_Small
- added R12, R15, R18, R21: 100 ohm, Resistor_SMD:R_0603_1608Metric, symbol Device:R
- added R2: 51 kohm, Resistor_SMD:R_0603_1608Metric, symbol Device:R
- added R26: 10 ohm/0.25 W, Resistor_SMD:R_1206_3216Metric, symbol Device:R
- added R27: 2 kohm, Resistor_SMD:R_0603_1608Metric, symbol Device:R
- added R28: 1 kohm, Resistor_SMD:R_0603_1608Metric, symbol Device:R
- added R29, R30, R31, R32, R33: 10k, Resistor_SMD:R_0603_1608Metric, symbol Device:R
- added R4: 22 kohm, Resistor_SMD:R_0603_1608Metric, symbol Device:R
- added R6: 47 kohm, Resistor_SMD:R_0603_1608Metric, symbol Device:R
- added R7: 1 ohm, Resistor_SMD:R_0603_1608Metric, symbol Device:R
- added TP1: POD_UART_TX, PodFeatures:PogoPad_D1.5mm, symbol PodFeatures:PogoPad
- added TP2: POD_UART_RX, PodFeatures:PogoPad_D1.5mm, symbol PodFeatures:PogoPad
- added TP3: GND, PodFeatures:PogoPad_D1.5mm, symbol PodFeatures:PogoPad
- added TP4: MCU_EN, PodFeatures:PogoPad_D1.5mm, symbol PodFeatures:PogoPad
- added TP5: MCU_BOOT, PodFeatures:PogoPad_D1.5mm, symbol PodFeatures:PogoPad
- added TP6: +3V3, PodFeatures:PogoPad_D1.5mm, symbol PodFeatures:PogoPad
- added U1: ESP32-S3-WROOM-1-N8, RF_Module:ESP32-S3-WROOM-1, symbol RF_Module:ESP32-S3-WROOM-1
- added U10: TPS2553QDBVRQ1, Package_TO_SOT_SMD:SOT-23-6, symbol PodPower:TPS2553QDBVRQ1
- added U100: TJA1051T-3, Package_SO:SOIC-8_3.9x4.9mm_P1.27mm, symbol Block_63616e_496e746572666163655f43414e5f4c494e:TJA1051T-3
- added U11: REF5050AIDR, Package_SO:SOIC-8_3.9x4.9mm_P1.27mm, symbol Reference_Voltage:REF5050AD
- added U12, U6: TPS7B4253QDDARQ1, PodPower:DDA0008J_C02, symbol PodPower:TPS7B4253QDDARQ1
- added U2: LSM6DSO32TR, Package_LGA:LGA-14_3x2.5mm_P0.5mm_LayoutBorder3x4y, symbol PodPrimarySPI:LSM6DSO32
- added U3: NEO-M9N-00B, RF_GPS:ublox_NEO, symbol RF_GPS:NEO-M9N
- added U4: MCP3204-BI/SL, Package_SO:SOIC-14_3.9x8.7mm_P1.27mm, symbol Analog_ADC:MCP3204
- added U5, U7: LMR36520ADDAR, PodPower:DDA0008B, symbol PodPower:LMR36520ADDAR
- added U8: ADA4096-4ARUZ-R7, Package_SO:TSSOP-14_4.4x5mm_P0.65mm, symbol PodPower:ADA4096-4ARUZ-R7
- added U9: OPA320AIDBVR, Package_TO_SOT_SMD:SOT-23-5, symbol PodPower:OPA320AIDBVR_VREF
Connections:
- new net +3V3: C13.1, C14.1, C15.1, C38.1, C41.1, C43.1, C44.1, C45.1, C46.1, C48.1, C49.1, C50.1, C51.1, C52.1, C53.1, L2.2, R25.2, R29.1, R30.1, R31.1, R32.1, R4.1, TP6.1 (PROBE), U1.2 (3V3), U10.1 (IN), U10.5 (ILIM), U100.5 (VIO), U2.5 (VDDIO), U2.8 (VDD), U3.2 (D_SEL), U3.22 (V_BCKP), U3.23 (VCC), U4.14 (Vdd), U8.4 (V+), U9.5 (V+)
- new net +5V_CAN: C100.1, C19.1, U100.3 (VCC), U12.1 (OUT), U12.4 (FB)
- new net ADC_AIN0: C31.1, R12.2, U4.1 (CH0)
- new net ADC_AIN1: C33.1, R15.2, U4.2 (CH1)
- new net ADC_AIN2: C35.1, R18.2, U4.3 (CH2)
- new net ADC_AIN3: C37.1, R21.2, U4.4 (CH3)
- new net ADC_CS: R32.2, U1.17 (IO9), U4.8 (~{CS}/SHDN)
- new net AFE_BUF0: R12.1, U8.1 (OUTA), U8.2 (-INA)
- new net AFE_BUF1: R15.1, U8.6 (-INB), U8.7 (OUTB)
- new net AFE_BUF2: R18.1, U8.8 (OUTC), U8.9 (-INC)
- new net AFE_BUF3: R21.1, U8.13 (-IND), U8.14 (OUTD)
- new net AFE_DIV0: C30.1, R10.2, R11.1, U8.3 (+INA)
- new net AFE_DIV1: C32.1, R13.2, R14.1, U8.5 (+INB)
- new net AFE_DIV2: C34.1, R16.2, R17.1, U8.10 (+INC)
- new net AFE_DIV3: C36.1, R19.2, R20.1, U8.12 (+IND)
- new net ANT_BIAS: C42.1, L3.1, R26.2
- new net ANT_LIMITED: R26.1, U10.6 (OUT)
- new net BOOT_3V3: C12.1, U7.7 (BOOT)
- new net BOOT_PRE: C5.1, U5.7 (BOOT)
- new net FB_3V3: R28.2, R5.1, U7.5 (FB)
- new net FB_3V3_SERIES: R28.1, R4.2
- new net FB_PRE: R27.2, R3.1, U5.5 (FB)
- new net FB_PRE_SERIES: R2.2, R27.1
- new net GND: C1.2, C10.2, C100.2, C11.2, C13.2, C14.2, C15.2, C16.2, C17.2, C18.2, C19.2, C2.2, C20.2, C21.2, C22.2, C3.2, C30.2, C31.2, C32.2, C33.2, C34.2, C35.2, C36.2, C37.2, C38.2, C39.2, C4.2, C40.2, C41.2, C42.2, C43.2, C44.2, C45.2, C46.2, C47.2, C48.2, C49.2, C50.2, C51.2, C52.2, C53.2, C6.2, C7.2, C8.2, C9.2, D1.2 (A2), D100.3 (common), D3.2 (A2), J1.10 (Pin_10), J1.13 (Pin_13), J1.16 (Pin_16), J1.4 (Pin_4), J1.7 (Pin_7), J2.2 (Ext), R1.2, R11.2, R14.2, R17.2, R20.2, R23.2, R24.2, R3.2, R33.2, R5.2, R6.2, TP3.1 (PROBE), U1.1 (GND), U1.40 (GND), U1.41 (GND), U10.2 (GND), U100.2 (GND), U100.8 (S), U11.4 (GND), U12.3 (GND), U12.6 (GND), U12.9 (EP), U2.2 (SDx), U2.3 (SCx), U2.6 (GND), U2.7 (GND), U3.10 (GND), U3.12 (GND), U3.13 (GND), U3.24 (GND), U3.7 (VDD_USB), U4.12 (AGND), U4.7 (DGND), U5.1 (PGND), U5.9 (EP), U6.3 (GND), U6.6 (GND), U6.9 (EP), U7.1 (PGND), U7.9 (EP), U8.11 (V-), U9.2 (V-)
- new net GNSS_ANT_FAULT_N: R25.1, U10.4 (FAULT)
- new net GNSS_LNA_EN: R24.1, U10.3 (EN), U3.14 (LNA_EN)
- new net GNSS_PPS: U1.7 (IO7), U3.3 (TIMEPULSE)
- new net GNSS_RX_IN: U1.10 (IO17), U3.21 (RXD/SPI_MOSI)
- new net GNSS_TX_OUT: U1.11 (IO18), U3.20 (TXD/SPI_MISO)
- new net IMU_CS: R31.2, U1.18 (IO10), U2.12 (CS)
- new net IMU_INT1: U1.6 (IO6), U2.4 (INT1)
- new net MCU_BOOT: R30.2, TP5.1 (PROBE), U1.27 (IO0)
- new net MCU_BOOT46: R33.1, U1.16 (IO46)
- new net MCU_EN: C47.1, R29.2, TP4.1 (PROBE), U1.3 (EN)
- new net POD_12V_IN: D1.1 (A1), J1.3 (Pin_3), Q1.2 (D)
- new net POD_12V_PROTECTED: C1.1, C10.1, C2.1, C3.1, C8.1, C9.1, D2.1 (K), Q1.3 (S), U5.2 (VIN), U5.3 (EN), U7.2 (VIN), U7.3 (EN)
- new net POD_5V_SENSOR: C17.1, J1.11 (Pin_11), J1.14 (Pin_14), J1.5 (Pin_5), J1.8 (Pin_8), R22.1, R6.1, U6.1 (OUT), U6.4 (FB)
- new net POD_CAN_N: D100.1 (A1), J1.2 (Pin_2), R100.2, U100.6 (CANL)
- new net POD_CAN_P: D100.2 (A2), J1.1 (Pin_1), R100.1, U100.7 (CANH)
- new net POD_FRONT_BRAKE_SIGNAL: J1.12 (Pin_12), R16.1
- new net POD_FRONT_FORK_SIGNAL: J1.6 (Pin_6), R10.1
- new net POD_GNSS_RF: D3.1 (A1), J2.1 (In), L3.2, U3.11 (RF_IN)
- new net POD_REAR_BRAKE_SIGNAL: J1.15 (Pin_15), R19.1
- new net POD_REAR_SHOCK_SIGNAL: J1.9 (Pin_9), R13.1
- new net POD_UART_RX: TP2.1 (PROBE), U1.36 (RXD0)
- new net POD_UART_TX: TP1.1 (PROBE), U1.37 (TXD0)
- new net PRE_6V3: C16.1, C18.1, C20.1, C6.1, C7.1, L1.2, R2.1, U11.2 (Vin), U12.8 (IN), U6.8 (IN)
- new net REF_CAP_NODE: C22.1, R7.2
- new net REF_DIV: C39.1, R22.2, R23.1, U9.3 (+IN)
- new net REF_NR: C21.1, U11.5 (Trim/NR)
- new net REVERSE_GATE: D2.2 (A), Q1.1 (G), R1.1
- new net SENSOR_REF_2V5: C40.1, U4.13 (Vref), U9.1 (OUT), U9.4 (-IN)
- new net SETPOINT_5V: R7.1, U11.6 (Vout), U12.5 (ADJ), U6.5 (ADJ)
- new net SPI_MISO: U1.21 (IO13), U2.1 (SDO), U4.10 (Dout)
- new net SPI_MOSI: U1.19 (IO11), U2.14 (SDA), U4.9 (Din)
- new net SPI_SCK: U1.20 (IO12), U2.13 (SCL), U4.11 (CLK)
- new net SW_3V3: C12.2, L2.1, U7.8 (SW)
- new net SW_PRE: C5.2, L1.1, U5.8 (SW)
- new net TWAI_RX: U1.5 (IO5), U100.4 (RXD)
- new net TWAI_TX: U1.4 (IO4), U100.1 (TXD)
- new net VCC_3V3: C11.1, U7.6 (VCC)
- new net VCC_PRE: C4.1, U5.6 (VCC)
- no-connect marks 0 -> 54
Other:
- note added: "3V3 regulator (U7) and 3V3 bulk"
- note added: "5V reference, sensor and CAN supplies"
- note added: "6V3 pre-regulator (U5)"
- note added: "ADC"
- note added: "CAN transceiver"
- note added: "GNSS receiver and antenna feed"
- note added: "IMU"
- note added: "MCU"
- note added: "Pod connector"
- note added: "Power entry and reverse protection"
- note added: "Sensor input dividers and buffers"
- note added: "Test points"
