File: telemetry-pod/telemetry-pod.kicad_sch (KiCad schematic)
At the start: 108 parts, among them J1 776228-1, J2 732511150, Q1 DMP6023LE-13, U1 ESP32-S3-WROOM-1-N8, U10 TPS2553QDBVRQ1, U100 TJA1051T-3, U11 REF5050AIDR, U12 TPS7B4253QDDARQ1, U2 LSM6DSO32TR, U3 NEO-M9N-00B, U4 MCP3204-BI/SL, U5 LMR36520ADDAR, U6 TPS7B4253QDDARQ1, U7 LMR36520ADDAR, U8 ADA4096-4ARUZ-R7, U9 OPA320AIDBVR

Commit message: AGENTEE-207: j6 authentic two-iteration production preparation on agent-ee 81e387ee; production schematic re-emitted as the telemetry-pod project (AGENTEE-445)
Pinned agent-ee 81e387ee (AGENTEE-197 landed, hand-fit chain 08ddaa17, emitter
field order 41e91eca). pipeline.py verifies the export blob by blob against that
commit. Everything ran in the pinned CI image (ae-ci-exec, network none).

- Plan schema: requirement_source telemetry-pod-rev3, bound to fome-mc's pinned
  Revision 3 capture (requirements/compiled), added as scope baseline sources.
  The microSD spec equals it except the POD-CD-STORAGE row (checked); its own
  selection refuses unapproved-source (kept).
- Envelope: the five generic obligations are staged under agent-ee source
  contract telemetry-pod-expanded/1 (H1-H4, J1 fixed/containment/part-identity,
  U1 fixed/containment/antenna keepout, 20 open items). The final guard keeps
  blocking on them. Enclosure and harness are open design deliverables.
- Scope: parts_subset over composition/parts.json (J1 identity witness); fab_package
  declares JP1-5 copper, TP1-6 probes and the J1 not_assembled exclusion;
  antenna-facts datasheet_facts check; fab profile relabelled to the production
  envelope's requirement id (values and citations unchanged); declared hand-fit
  citation in the assembly check; emitter captures root fixed (emit-schematic
  failed on every library with 'footprints').
- No driver-default probe plan and no compiled-only scope. Stock is graded per
  id at generation (81 ids: 80 in stock, J1 C596198 zero; none stale).
- Real dry run: prepared, max_iterations 2 (plan), routing budget 900 s /
  timeout 2100 s, placement timeout 1500 s, derived watchdog 8400 s; review
  packet carries the 4 block obligations, copper_unknown and the 174-entry
  ledger; binding-fill 305 components / 248 ratings. No campaign launched.
- AGENTEE-445: the campaign's schematic-stage steps (binding-fill,
  emit-schematic, forward-annotate) ran with stage receipt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
Parts:
- added C110, C111, C112, C114, C115, C116, C117, C125, C127, C129, C87, C90, C93, C97: 100nF 50V X7R, Capacitor_SMD:C_0603_1608Metric, symbol Device:C
- added C118, C119, C120, C121, C122, C123, C124, C86, C89, C92, C98: 1uF 50V X7R, Capacitor_SMD:C_0805_2012Metric, symbol Device:C
- added C126, C88, C91, C94: 10nF 50V C0G 10%, Capacitor_SMD:C_0603_1608Metric, symbol Device:C
- added C128: 10uF 16V X7R, Capacitor_SMD:C_1206_3216Metric, symbol Device:C
- added C54, C56, C58, C60: 100 nF/50 V X7R, Capacitor_SMD:C_0603_1608Metric, symbol Device:C
- added C55, C57, C59, C61: 100 pF C0G/50 V, Capacitor_SMD:C_0603_1608Metric, symbol Device:C
- added C62, C65, C72, C76, C78, C79, C83, C84, C85: 100nF, Capacitor_SMD:C_0603_1608Metric, symbol Device:C
- added C64: 4.7 uF/16 V X7R, Capacitor_SMD:C_0805_2012Metric, symbol Device:C
- added C71, C75, C77: 22nF, Capacitor_SMD:C_0603_1608Metric, symbol Device:C
- added C80: 1uF, Capacitor_SMD:C_0603_1608Metric, symbol Device:C
- added C81, C82: 18pF C0G, Capacitor_SMD:C_0603_1608Metric, symbol Device:C
- added C95, C96: 220pF C0G, Capacitor_SMD:C_0603_1608Metric, symbol Device:C
- added D101, D104: PESD2CANFD24V-TR, Package_TO_SOT_SMD:SOT-23, symbol PodCAN:PESD2CANFD24V_T
- added D102, D103, D105: BAV199,215, Package_TO_SOT_SMD:SOT-23, symbol PodWheel:BAV199
- added J3: DM3AT-SF-PEJM5, Connector_Card:microSD_HC_Hirose_DM3AT-SF-PEJM5, symbol Connector:Micro_SD_Card_Det_Hirose_DM3AT
- added JP1: TIRE_TERM_CLOSE_ONLY_AT_BUS_END, Jumper:SolderJumper-2_P1.3mm_Open_RoundedPad1.0x1.5mm, symbol CANJumper:SolderJumper_2_Open
- added JP2: AUX1_THERM_PULLUP_CLOSE_TO_ENABLE, Jumper:SolderJumper-2_P1.3mm_Open_RoundedPad1.0x1.5mm, symbol CANJumper:SolderJumper_2_Open
- added JP3: AUX2_THERM_PULLUP_CLOSE_TO_ENABLE, Jumper:SolderJumper-2_P1.3mm_Open_RoundedPad1.0x1.5mm, symbol CANJumper:SolderJumper_2_Open
- added JP4: AUX3_THERM_PULLUP_CLOSE_TO_ENABLE, Jumper:SolderJumper-2_P1.3mm_Open_RoundedPad1.0x1.5mm, symbol CANJumper:SolderJumper_2_Open
- added JP5: AUX4_THERM_PULLUP_CLOSE_TO_ENABLE, Jumper:SolderJumper-2_P1.3mm_Open_RoundedPad1.0x1.5mm, symbol CANJumper:SolderJumper_2_Open
- added R110, R111, R119, R120: 620 ohm, Resistor_SMD:R_2512_6332Metric, symbol Device:R
- added R112, R113, R115, R121, R122, R124, R57, R61, R63: 10 kohm 0.1%, Resistor_SMD:R_0603_1608Metric, symbol Device:R
- added R114, R123: 56 kohm 0.1%, Resistor_SMD:R_0603_1608Metric, symbol Device:R
- added R116, R125: 100 kohm 0.1%, Resistor_SMD:R_0603_1608Metric, symbol Device:R
- added R117, R126: 4.7 kohm 1%, Resistor_SMD:R_0603_1608Metric, symbol Device:R
- added R118, R127, R36, R39, R42, R45: 100 ohm, Resistor_SMD:R_0603_1608Metric, symbol Device:R
- added R128, R129, R130, R132, R133, R134, R136, R137, R138, R144, R145, R146, R148, R149, R150, R152, R153, R154, R156, R157, R158, R166, R167, R168: 499 kohm 0.1% 25ppm/C, Resistor_SMD:R_0603_1608Metric, symbol Device:R
- added R131, R135, R139, R147, R151, R155, R159, R169: 4.99 kohm 0.1% 25ppm/C, Resistor_SMD:R_0603_1608Metric, symbol Device:R
- added R160, R161: 2.2 kohm 1% 100ppm/C, Resistor_SMD:R_0603_1608Metric, symbol Device:R
- added R162, R73, R77, R81: 1.05 Mohm 0.1% 25ppm/K, Resistor_SMD:R_0805_2012Metric, symbol Device:R
- added R163: 95.3 kohm 0.1% 25ppm/K, Resistor_SMD:R_0603_1608Metric, symbol Device:R
- added R164: 287 kohm 0.1% 25ppm/K, Resistor_SMD:R_0603_1608Metric, symbol Device:R
- added R165: 44.2 kohm 0.1% 25ppm/K, Resistor_SMD:R_0603_1608Metric, symbol Device:R
- added R170, R171, R172, R173: 10 kohm 0.1% 25ppm/K, Resistor_SMD:R_0603_1608Metric, symbol Device:R
- added R174, R175: 200 ohm 1% 100ppm/K 1.5W CRCW2512-HP, Resistor_SMD:R_2512_6332Metric, symbol Device:R
- added R176, R177, R178: 499 kohm 0.1% 25ppm/K, Resistor_SMD:R_0603_1608Metric, symbol Device:R
- added R179: 4.99 kohm 0.1% 25ppm/K, Resistor_SMD:R_0603_1608Metric, symbol Device:R
- added R180: 100 kohm 1% 100ppm/K, Resistor_SMD:R_0603_1608Metric, symbol Device:R
- added R181: 1.2 kohm 0.1% 25ppm/K, Resistor_SMD:R_0603_1608Metric, symbol Device:R
- added R34, R35, R37, R38, R40, R41, R43, R44, R46, R47, R48, R49, R50, R55, R64, R65, R66, R67, R68, R69, R71, R72: 10 kohm, Resistor_SMD:R_0603_1608Metric, symbol Device:R
- added R56: 16.9 kohm 0.1%, Resistor_SMD:R_0603_1608Metric, symbol Device:R
- added R60: 30.1 kohm 0.1% 25ppm/K, Resistor_SMD:R_0603_1608Metric, symbol Device:R
- added R62: 64.9 kohm 0.1%, Resistor_SMD:R_0603_1608Metric, symbol Device:R
- added R70: 120 ohm, Resistor_SMD:R_0603_1608Metric, symbol Device:R
- added R74, R78, R82: 68.1 kohm 0.1% 25ppm/K, Resistor_SMD:R_0603_1608Metric, symbol Device:R
- added R75, R79, R83: 215 kohm 0.1% 25ppm/K, Resistor_SMD:R_0603_1608Metric, symbol Device:R
- added R76, R80: 44.2 kohm 0.1%, Resistor_SMD:R_0603_1608Metric, symbol Device:R
- added R84: 26.7 kohm 0.1%, Resistor_SMD:R_0603_1608Metric, symbol Device:R
- added U13: ADA4096-4ARUZ-R7, Package_SO:TSSOP-14_4.4x5mm_P0.65mm, symbol PodPower:ADA4096-4ARUZ-R7
- added U16, U18, U19: TPS389001DSER, PodSupervisor:DSE0006A, symbol PodSupervisor:TPS389001DSE
- added U20: MCP2518FDT-E/SL, Package_SO:SOIC-14_3.9x8.7mm_P1.27mm, symbol PodCAN:MCP2518FD_SL
- added U21: TJA1051T/3/1J, Package_SO:SOIC-8_3.9x4.9mm_P1.27mm, symbol Block_63616e_496e746572666163655f43414e5f4c494e:TJA1051T-3
- added U22: SN74LVC1G132DBVR, Package_TO_SOT_SMD:SOT-23-5, symbol PodCAN:SN74LVC1G132DBV
- added U23, U24, U25, U30: TPS26625DRCR, Package_SON:VSON-10-1EP_3x3mm_P0.5mm_EP1.65x2.4mm, symbol PodSensorPower:TPS26625_DRC
- added U26: LM2903BQDRQ1, Package_SO:SOIC-8_3.9x4.9mm_P1.27mm, symbol PodWheel:LM2903BQ_D
- added U27, U28, U29: ADS1119IPWR, Package_SO:TSSOP-16_4.4x5mm_P0.65mm, symbol PodDiagnostic:ADS1119_PW
- added U31: TL431BQDBZR, Package_TO_SOT_SMD:SOT-23, symbol PodThermistor:TL431DBZ
- added Y1: X1E0003410031 20MHz 12pF, Crystal:Crystal_SMD_SeikoEpson_FA238-4Pin_3.2x2.5mm, symbol CANClock:Crystal_GND24
- C1: AGENT_EE_Ratings {"ratings":{"Voltage":"100V"},"record_sha256":"d8e824543029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 -> {"ratings":{"Voltage":"100V"},"record_sha256":"4c6b536060ad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
- C10: AGENT_EE_Ratings {"ratings":{"Voltage":"100V"},"record_sha256":"7b14d59faaee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 -> {"ratings":{"Voltage":"100V"},"record_sha256":"e3d67639b1b7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
- C100: AGENT_EE_Ratings {"ratings":{"Voltage":"16V"},"record_sha256":"1eb663ac0c345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 -> {"ratings":{"Voltage":"16V"},"record_sha256":"363b4bea83286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
- C11: AGENT_EE_Ratings {"ratings":{"Voltage":"16V"},"record_sha256":"5e4ef14638fd6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 -> {"ratings":{"Voltage":"16V"},"record_sha256":"d5e591b7af489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
- C12: AGENT_EE_Ratings {"ratings":{"Voltage":"50V"},"record_sha256":"2c4dfb95d005e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 -> {"ratings":{"Voltage":"50V"},"record_sha256":"54ea0e5fa0cf8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
- C13: AGENT_EE_Ratings {"ratings":{"Voltage":"25V"},"record_sha256":"958f8b0776737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 -> {"ratings":{"Voltage":"25V"},"record_sha256":"39066e98edcc2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
- C14: AGENT_EE_Ratings {"ratings":{"Voltage":"25V"},"record_sha256":"1add79c44cdeb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 -> {"ratings":{"Voltage":"25V"},"record_sha256":"7d8063c1a8535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
- C15: AGENT_EE_Ratings {"ratings":{"Voltage":"25V"},"record_sha256":"5fd9fb708611d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 -> {"ratings":{"Voltage":"25V"},"record_sha256":"6fba92fddbff8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
- C16: AGENT_EE_Ratings {"ratings":{"Voltage":"16V"},"record_sha256":"0110e36915f53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 -> {"ratings":{"Voltage":"16V"},"record_sha256":"4383956ecd3de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
- C17: AGENT_EE_Ratings {"ratings":{"Voltage":"25V"},"record_sha256":"efb8b1e7e192b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 -> {"ratings":{"Voltage":"25V"},"record_sha256":"fa90cb168d0b7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
- C18: AGENT_EE_Ratings {"ratings":{"Voltage":"16V"},"record_sha256":"0317eeb5bb39b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 -> {"ratings":{"Voltage":"16V"},"record_sha256":"fddcc7f04afbc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
- C19: AGENT_EE_Ratings {"ratings":{"Voltage":"25V"},"record_sha256":"e15b8da8f9050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 -> {"ratings":{"Voltage":"25V"},"record_sha256":"d62d2fa153300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
- C2: AGENT_EE_Ratings {"ratings":{"Voltage":"100V"},"record_sha256":"55baeec9341a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 -> {"ratings":{"Voltage":"100V"},"record_sha256":"088e7de65887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
- C20: AGENT_EE_Ratings {"ratings":{"Voltage":"16V"},"record_sha256":"01f50dfce8c2f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 -> {"ratings":{"Voltage":"16V"},"record_sha256":"01f9f607641fa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
- C21: AGENT_EE_Ratings {"ratings":{"Voltage":"16V"},"record_sha256":"76e85dcb7bfdf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 -> {"ratings":{"Voltage":"16V"},"record_sha256":"0abff3aa31bde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
- C22: AGENT_EE_Ratings {"ratings":{"Voltage":"16V"},"record_sha256":"383141557dbdc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 -> {"ratings":{"Voltage":"16V"},"record_sha256":"c8fd4bac89031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
- C3: AGENT_EE_Ratings {"ratings":{"Voltage":"100V"},"record_sha256":"ca85cce41b6f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 -> {"ratings":{"Voltage":"100V"},"record_sha256":"bcbc016f6379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
- C30: AGENT_EE_Ratings {"ratings":{"Voltage":"50V"},"record_sha256":"71594f51a271f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 -> {"ratings":{"Voltage":"50V"},"record_sha256":"19e47a5d03501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
- C31: AGENT_EE_Ratings {"ratings":{"Voltage":"50V"},"record_sha256":"2ef3f037976b9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 -> {"ratings":{"Voltage":"50V"},"record_sha256":"317f9835dd65c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
- C32: AGENT_EE_Ratings {"ratings":{"Voltage":"50V"},"record_sha256":"cb0c9672c8d01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 -> {"ratings":{"Voltage":"50V"},"record_sha256":"0a353e3f3a6a3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
- C33: AGENT_EE_Ratings {"ratings":{"Voltage":"50V"},"record_sha256":"19a7e78ea3557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 -> {"ratings":{"Voltage":"50V"},"record_sha256":"2c4a582e918f7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
- C34: AGENT_EE_Ratings {"ratings":{"Voltage":"50V"},"record_sha256":"362601e2de7a3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 -> {"ratings":{"Voltage":"50V"},"record_sha256":"209298f8b84f3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
- C35: AGENT_EE_Ratings {"ratings":{"Voltage":"50V"},"record_sha256":"5820ac30d5733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 -> {"ratings":{"Voltage":"50V"},"record_sha256":"baa74297aa628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
- C36: AGENT_EE_Ratings {"ratings":{"Voltage":"50V"},"record_sha256":"cc0d133d147ac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 -> {"ratings":{"Voltage":"50V"},"record_sha256":"bcfa13ea829e1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
- C37: AGENT_EE_Ratings {"ratings":{"Voltage":"50V"},"record_sha256":"a985d6e4570ed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 -> {"ratings":{"Voltage":"50V"},"record_sha256":"542031862facf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
- C38: AGENT_EE_Ratings {"ratings":{"Voltage":"50V"},"record_sha256":"53aaf9803c252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 -> {"ratings":{"Voltage":"50V"},"record_sha256":"4b75465ada340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
- C39: AGENT_EE_Ratings {"ratings":{"Voltage":"50V"},"record_sha256":"1e047b2657a00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 -> {"ratings":{"Voltage":"50V"},"record_sha256":"2ff06bbdc5c94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
- C4: AGENT_EE_Ratings {"ratings":{"Voltage":"16V"},"record_sha256":"17e2bb53ea459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 -> {"ratings":{"Voltage":"16V"},"record_sha256":"d6a85203a3d25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
- C40: AGENT_EE_Ratings {"ratings":{"Voltage":"50V"},"record_sha256":"7a4e6d009b0da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 -> {"ratings":{"Voltage":"50V"},"record_sha256":"6ebae879771c7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
- C41: AGENT_EE_Ratings {"ratings":{"Voltage":"50V"},"record_sha256":"1e2af3f2f4a0a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 -> {"ratings":{"Voltage":"50V"},"record_sha256":"26c155009d165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
- C42: AGENT_EE_Ratings {"ratings":{"Voltage":"50V"},"record_sha256":"4880bdb033631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 -> {"ratings":{"Voltage":"50V"},"record_sha256":"c22536c34862e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
- C43: AGENT_EE_Ratings {"ratings":{"Voltage":"50V"},"record_sha256":"38587a095744d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 -> {"ratings":{"Voltage":"50V"},"record_sha256":"c231f375a7bc5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
- C44: AGENT_EE_Ratings {"ratings":{"Voltage":"16V"},"record_sha256":"32f4901df5146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 -> {"ratings":{"Voltage":"16V"},"record_sha256":"76b59d2a00dc0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
- C45: AGENT_EE_Ratings {"ratings":{"Voltage":"25V"},"record_sha256":"54689c799c8ae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 -> {"ratings":{"Voltage":"25V"},"record_sha256":"37df1f20f870b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
- C46: AGENT_EE_Ratings {"ratings":{"Voltage":"50V"},"record_sha256":"a8d8a773fd799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 -> {"ratings":{"Voltage":"50V"},"record_sha256":"ff57c35b5e76f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
- C47: value 1uF -> 10nF; AGENT_EE_Ratings {"ratings":{"Voltage":"16V"},"record_sha256":"cb4ab6fa1e85b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 -> {"ratings":{"Voltage":"50V"},"record_sha256":"3dd48a34fe608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; LCSC C76706 -> C85973; Manufacturer TDK -> Murata Electronics; PARAM_Datasheet {"schema":"agent-ee.datasheet-binding/1","sha256":"ff9b0a37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 -> {"schema":"agent-ee.datasheet-binding/1","sha256":"3f5a339e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; Partnumber CGA3E1X7R1C105KT0Y0N -> GRM1885C1H103JA01D; Voltage 16V -> 50V
- C48: AGENT_EE_Ratings {"ratings":{"Voltage":"50V"},"record_sha256":"0d841baca1e2f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 -> {"ratings":{"Voltage":"50V"},"record_sha256":"417060dae6118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
- C49: AGENT_EE_Ratings {"ratings":{"Voltage":"50V"},"record_sha256":"129ccd84e722d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 -> {"ratings":{"Voltage":"50V"},"record_sha256":"4c90a2b6150a6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
- C5: AGENT_EE_Ratings {"ratings":{"Voltage":"50V"},"record_sha256":"45081501eb06d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 -> {"ratings":{"Voltage":"50V"},"record_sha256":"2c4336efe3e49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
- C50: AGENT_EE_Ratings {"ratings":{"Voltage":"16V"},"record_sha256":"0bd6f35f3e7b4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 -> {"ratings":{"Voltage":"16V"},"record_sha256":"7a8e44554de76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
- C51: AGENT_EE_Ratings {"ratings":{"Voltage":"50V"},"record_sha256":"9d9e8e89336b5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 -> {"ratings":{"Voltage":"50V"},"record_sha256":"daef87a4efe21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
- C52: AGENT_EE_Ratings {"ratings":{"Voltage":"16V"},"record_sha256":"1fc1fe8d4f6a9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 -> {"ratings":{"Voltage":"16V"},"record_sha256":"2308760d04a79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
- C53: AGENT_EE_Ratings {"ratings":{"Voltage":"50V"},"record_sha256":"ca92cc78d323f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 -> {"ratings":{"Voltage":"50V"},"record_sha256":"177d09f70f6f0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
- C6: AGENT_EE_Ratings {"ratings":{"Voltage":"25V"},"record_sha256":"e2e19f88ef5dd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 -> {"ratings":{"Voltage":"25V"},"record_sha256":"89f7e2db9aab9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
- C7: AGENT_EE_Ratings {"ratings":{"Voltage":"25V"},"record_sha256":"7612ed9b5235a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 -> {"ratings":{"Voltage":"25V"},"record_sha256":"9b19b673bbef2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
- C8: AGENT_EE_Ratings {"ratings":{"Voltage":"100V"},"record_sha256":"5831a79856b8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 -> {"ratings":{"Voltage":"100V"},"record_sha256":"8dfcf2a1813a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
- C9: AGENT_EE_Ratings {"ratings":{"Voltage":"100V"},"record_sha256":"8fe49fc0e870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 -> {"ratings":{"Voltage":"100V"},"record_sha256":"be82461f042d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
- J1: value 776228-1 -> 1-776163-1; footprint ampseal:ampseal-23 -> PodConnector:AMPSEAL_35_1-776163-1; symbol Connector_Generic:Conn_01x23 -> Connector_Generic:Conn_01x35; LCSC C498958 -> C596198; PARAM_Datasheet {"schema":"agent-ee.datasheet-binding/1","sha256":"14bd5c3b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 -> {"schema":"agent-ee.datasheet-binding/1","sha256":"7ed1f2a5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; Partnumber 776228-1 -> 1-776163-1
- R1: AGENT_EE_Ratings {"ratings":{"Power":"100mW"},"record_sha256":"8e5e56d94703d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 -> {"ratings":{"Power":"100mW"},"record_sha256":"f9d441da3f992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
- R10: AGENT_EE_Ratings {"ratings":{"Power":"100mW"},"record_sha256":"11ebdec84da43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 -> {"ratings":{"Power":"100mW"},"record_sha256":"8a1b38a446f71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
- R100: AGENT_EE_Ratings {"ratings":{"Power":"100mW"},"record_sha256":"c85c5d64e9692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 -> {"ratings":{"Power":"100mW"},"record_sha256":"3731d3ad5bca6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
- R11: AGENT_EE_Ratings {"ratings":{"Power":"100mW"},"record_sha256":"a899abf18c77d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 -> {"ratings":{"Power":"100mW"},"record_sha256":"b7b059358127a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
- R12: AGENT_EE_Ratings {"ratings":{"Power":"100mW"},"record_sha256":"dd1cab5bd8351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 -> {"ratings":{"Power":"100mW"},"record_sha256":"1117e8c3404d0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
- R13: AGENT_EE_Ratings {"ratings":{"Power":"100mW"},"record_sha256":"e6448ba99a960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 -> {"ratings":{"Power":"100mW"},"record_sha256":"4d76dcffd0cb1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
- R14: AGENT_EE_Ratings {"ratings":{"Power":"100mW"},"record_sha256":"98f9f033c80be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 -> {"ratings":{"Power":"100mW"},"record_sha256":"7aa013bb77603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
- R15: AGENT_EE_Ratings {"ratings":{"Power":"100mW"},"record_sha256":"67d9bb3bbcb08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 -> {"ratings":{"Power":"100mW"},"record_sha256":"a9a3543670bf1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
- R16: AGENT_EE_Ratings {"ratings":{"Power":"100mW"},"record_sha256":"e9c202a141724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 -> {"ratings":{"Power":"100mW"},"record_sha256":"684be4f5738f9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
- R17: AGENT_EE_Ratings {"ratings":{"Power":"100mW"},"record_sha256":"ca4f38326f26d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 -> {"ratings":{"Power":"100mW"},"record_sha256":"bd7527a538c90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
- R18: AGENT_EE_Ratings {"ratings":{"Power":"100mW"},"record_sha256":"3d8462f0aa268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 -> {"ratings":{"Power":"100mW"},"record_sha256":"49e92ebaf6e24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
- R19: AGENT_EE_Ratings {"ratings":{"Power":"100mW"},"record_sha256":"5c50ae14e4873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 -> {"ratings":{"Power":"100mW"},"record_sha256":"108ee1a6ede06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
- R2: AGENT_EE_Ratings {"ratings":{"Power":"100mW"},"record_sha256":"bf7499cdb4e7d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 -> {"ratings":{"Power":"100mW"},"record_sha256":"53761488c2b3d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
- R20: AGENT_EE_Ratings {"ratings":{"Power":"100mW"},"record_sha256":"f7a3a47f9d09b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 -> {"ratings":{"Power":"100mW"},"record_sha256":"1a83e21e2537f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
- R21: AGENT_EE_Ratings {"ratings":{"Power":"100mW"},"record_sha256":"9cc148ffa8786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 -> {"ratings":{"Power":"100mW"},"record_sha256":"0171f39e37d4c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
- R22: AGENT_EE_Ratings {"ratings":{"Power":"100mW"},"record_sha256":"46ff70557501d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 -> {"ratings":{"Power":"100mW"},"record_sha256":"b2ffb58f25577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
- R23: AGENT_EE_Ratings {"ratings":{"Power":"100mW"},"record_sha256":"ae430b59c91e6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 -> {"ratings":{"Power":"100mW"},"record_sha256":"faa88cabb825c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
- R24: AGENT_EE_Ratings {"ratings":{"Power":"100mW"},"record_sha256":"32e8f2b6571ce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 -> {"ratings":{"Power":"100mW"},"record_sha256":"4a4fc70412c73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
- R25: AGENT_EE_Ratings {"ratings":{"Power":"100mW"},"record_sha256":"5b1a73af53c01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 -> {"ratings":{"Power":"100mW"},"record_sha256":"811ea4199bdef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
- R26: AGENT_EE_Ratings {"ratings":{"Power":"250mW"},"record_sha256":"acb21f2f654b9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 -> {"ratings":{"Power":"250mW"},"record_sha256":"c9620b7d63177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
- R27: AGENT_EE_Ratings {"ratings":{"Power":"100mW"},"record_sha256":"27f3abe7d15ab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 -> {"ratings":{"Power":"100mW"},"record_sha256":"bbb8aa373556a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
- R28: AGENT_EE_Ratings {"ratings":{"Power":"100mW"},"record_sha256":"89141b81c17e9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 -> {"ratings":{"Power":"100mW"},"record_sha256":"d6dbc193ffe90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
- R29: value 10k -> 100 kohm; AGENT_EE_Ratings {"ratings":{"Power":"100mW"},"record_sha256":"57d99da031e5d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 -> {"ratings":{"Power":"100mW"},"record_sha256":"f57a972e714bc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; LCSC C95204 -> C122538; PARAM_Datasheet {"schema":"agent-ee.datasheet-binding/1","sha256":"0a729d14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 -> {"schema":"agent-ee.datasheet-binding/1","sha256":"48b00bce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; Partnumber RT0603BRD0710KL -> RT0603BRD07100KL
- R3: AGENT_EE_Ratings {"ratings":{"Power":"100mW"},"record_sha256":"ac4eba8601047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 -> {"ratings":{"Power":"100mW"},"record_sha256":"a305bc8d22cb6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
- R30: AGENT_EE_Ratings {"ratings":{"Power":"100mW"},"record_sha256":"dedbd17430dbf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 -> {"ratings":{"Power":"100mW"},"record_sha256":"e7ed9c1f1ba54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
- R31: AGENT_EE_Ratings {"ratings":{"Power":"100mW"},"record_sha256":"d6317204b5015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 -> {"ratings":{"Power":"100mW"},"record_sha256":"4275d0e4c1c2f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
- R32: AGENT_EE_Ratings {"ratings":{"Power":"100mW"},"record_sha256":"0be694e78d2dd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 -> {"ratings":{"Power":"100mW"},"record_sha256":"78688ea21b3e1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
- R33: AGENT_EE_Ratings {"ratings":{"Power":"100mW"},"record_sha256":"134e1dad3d84d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 -> {"ratings":{"Power":"100mW"},"record_sha256":"970533bb16bc0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
- R4: AGENT_EE_Ratings {"ratings":{"Power":"100mW"},"record_sha256":"e3206e1ff5560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 -> {"ratings":{"Power":"100mW"},"record_sha256":"572e5cc2f84ba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
- R5: AGENT_EE_Ratings {"ratings":{"Power":"100mW"},"record_sha256":"ed9ec80ee3cfa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 -> {"ratings":{"Power":"100mW"},"record_sha256":"cc6fd34504a1e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
- R6: AGENT_EE_Ratings {"ratings":{"Power":"100mW"},"record_sha256":"00a6f4b1eab13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 -> {"ratings":{"Power":"100mW"},"record_sha256":"823b6b6b75110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
- R7: AGENT_EE_Ratings {"ratings":{"Power":"100mW"},"record_sha256":"3e0f9b483ffb7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 -> {"ratings":{"Power":"100mW"},"record_sha256":"b24cfb456496a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
- TP1, TP2, TP3, TP4, TP5, TP6: AGENT_EE_Probe {"footprint":"PodFeatures:PogoPad_D1.5mm","footprint_source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 -> agent-ee-probe-v1-eyJmb290cHJpbnQiOiJQb2RGZWF0dXJlczpQb2dvU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
- U4: value MCP3204-BI/SL -> MCP3208-BI/SL; footprint Package_SO:SOIC-14_3.9x8.7mm_P1.27mm -> Package_SO:SOIC-16_3.9x9.9mm_P1.27mm; symbol Analog_ADC:MCP3204 -> Analog_ADC:MCP3208; LCSC C107363 -> C2979740; PARAM_Datasheet {"schema":"agent-ee.datasheet-binding/1","sha256":"89bc1e17c35e2bb1c7b8fbf0b775b3729ce9fe4d27f7e9c052a774757afc0c20","url":"https://ww1.microchip.com/downloads/en/DeviceDoc/21298e.pdf"} -> {"schema":"agent-ee.datasheet-binding/1","sha256":"89bc1e17c35e2bb1c7b8fbf0b775b3729ce9fe4d27f7e9c052a774757afc0c20","url":"https://ww1.microchip.com/downloads/aemDocuments/documents/APID/ProductDocuments/DataSheets/21298e.pdf"}; Partnumber MCP3204-BI/SL -> MCP3208-BI/SL
Connections:
- net +3V3: now also U4.16 (Vdd), C118.1, C119.1, C120.1, C121.1, C122.1, C123.1, C62.1, C64.1, C65.1, C72.1, C76.1, C78.1, C79.1, C80.1, C84.1, C85.1, J3.4 (VDD), R114.1, R117.1, R123.1, R126.1, R136.1, R160.1, R161.1, R46.1, R47.1, R48.1, R49.1, R50.1, R55.2, R56.1, R64.1, R65.1, R66.1, R67.1, R69.1, R71.1, U13.4 (V+), U16.3 (MR), U16.4 (VDD), U18.3 (MR), U18.4 (VDD), U19.3 (MR), U19.4 (VDD), U20.14 (VDD), U21.5 (VIO), U22.5 (VCC), U27.12 (AVDD), U27.13 (DVDD), U27.3 (RESET_N), U28.1 (A0), U28.12 (AVDD), U28.13 (DVDD), U28.3 (RESET_N), U29.12 (AVDD), U29.13 (DVDD), U29.2 (A1), U29.3 (RESET_N); no longer U4.14 (Vdd)
- net +5V_CAN: now also C83.1, U21.3 (VCC)
- net ADC_CS: now also U4.10 (~{CS}/SHDN); no longer U4.8 (~{CS}/SHDN)
- net GND: now also J1.22 (Pin_22), J1.25 (Pin_25), J1.28 (Pin_28), J1.32 (Pin_32), U4.14 (AGND), U4.9 (DGND), C110.2, C111.2, C112.2, C114.2, C115.2, C116.2, C117.2, C118.2, C119.2, C120.2, C121.2, C122.2, C123.2, C124.2, C125.2, C127.2, C128.2, C129.2, C54.2, C55.2, C56.2, C57.2, C58.2, C59.2, C60.2, C61.2, C62.2, C64.2, C65.2, C71.2, C72.2, C75.2, C76.2, C77.2, C78.2, C79.2, C80.2, C81.2, C82.2, C83.2, C84.2, C85.2, C86.2, C87.2, C89.2, C90.2, C92.2, C93.2, C95.2, C96.2, C97.2, C98.2, D101.3 (CC), D104.3 (CC), J3.10 (DET_A), J3.6 (VSS), J3.SH (SHIELD), R113.2, R115.2, R122.2, R124.2, R131.2, R135.2, R139.2, R147.2, R151.2, R155.2, R159.2, R169.2, R179.2, R180.2, R35.2, R38.2, R41.2, R44.2, R57.2, R61.2, R63.2, R68.2, R72.2, U13.11 (V-), U16.2 (GND), U18.2 (GND), U19.2 (GND), U20.7 (VSS), U21.2 (GND), U22.3 (GND), U23.6 (GND), U24.6 (GND), U25.6 (GND), U26.4 (GND), U27.1 (A0), U27.2 (A1), U27.4 (DGND), U27.5 (AGND), U28.2 (A1), U28.4 (DGND), U28.5 (AGND), U29.1 (A0), U29.4 (DGND), U29.5 (AGND), U30.6 (GND), U31.3 (A), Y1.2 (G), Y1.4 (G); no longer U4.12 (AGND), U4.7 (DGND)
- net MCU_EN: now also U16.6 (RESET), U22.1 (A)
- net POD_12V_PROTECTED: now also R128.1, R62.1
- net POD_5V_SENSOR: now also C124.1, R144.1, R162.1, R60.1, U30.1 (IN)
- net PRE_6V3: now also C86.1, C89.1, C92.1, C97.1, C98.1, R132.1, R73.1, R77.1, R81.1, U23.1 (IN), U24.1 (IN), U25.1 (IN), U26.8 (VCC)
- net SENSOR_REF_2V5: now also U4.15 (Vref); no longer U4.13 (Vref)
- net SPI_MISO: now also U4.12 (Dout), U20.12 (SDO); no longer U4.10 (Dout)
- net SPI_MOSI: now also U4.11 (Din), U20.11 (SDI); no longer U4.9 (Din)
- net SPI_SCK: now also U4.13 (CLK), U20.10 (SCK); no longer U4.11 (CLK)
- net POD_AUX1_SIGNAL: now reaches J1.17 (Pin_17)
- net POD_AUX1_SIGNAL: now also JP2.2 (B), R34.1
- net POD_AUX2_SIGNAL: now reaches J1.18 (Pin_18)
- net POD_AUX2_SIGNAL: now also JP3.2 (B), R37.1
- net POD_AUX3_SIGNAL: now reaches J1.19 (Pin_19)
- net POD_AUX3_SIGNAL: now also JP4.2 (B), R40.1
- net POD_AUX4_SIGNAL: now reaches J1.20 (Pin_20)
- net POD_AUX4_SIGNAL: now also JP5.2 (B), R43.1
- net POD_5V_AUX: now reaches J1.21 (Pin_21)
- net POD_5V_AUX: now also C125.1, D105.1 (A1), R166.1, R180.1, U30.10 (OUT)
- net POD_WHEEL_FRONT_SUPPLY: now reaches J1.23 (Pin_23)
- net POD_WHEEL_FRONT_SUPPLY: now also C87.1, R110.1, R148.1, U23.10 (OUT)
- net ADC_AIN4: now reaches U4.5 (CH4)
- net ADC_AIN4: now also C55.1, R36.2
- net ADC_AIN5: now reaches U4.6 (CH5)
- net ADC_AIN5: now also C57.1, R39.2
- net POWER_FAIL_N: now reaches U1.12 (IO8)
- net POWER_FAIL_N: now also R65.2, U19.6 (RESET)
- net DIAG_I2C_SDA: now reaches U1.22 (IO14)
- net DIAG_I2C_SDA: now also R160.2, U27.15 (SDA), U28.15 (SDA), U29.15 (SDA)
- net DIAG_I2C_SCL: now reaches U1.23 (IO21)
- net DIAG_I2C_SCL: now also R161.2, U27.16 (SCL), U28.16 (SCL), U29.16 (SCL)
- net SD_DAT3: now reaches U1.24 (IO47)
- net SD_DAT3: now also J3.2 (DAT3/CD), R50.2
- net SENSOR_FAULT_N: now reaches U1.25 (IO48)
- net SENSOR_FAULT_N: now also R64.2, U18.6 (RESET)
- net SD_CD: now reaches U1.28 (IO35)
- net SD_CD: now also J3.9 (DET_B), R55.1
- net SD_CLK: now reaches U1.31 (IO38)
- net SD_CLK: now also J3.5 (CLK)
- net SD_CMD: now reaches U1.32 (IO39)
- net SD_CMD: now also J3.3 (CMD), R46.2
- net SD_DAT0: now reaches U1.33 (IO40)
- net SD_DAT0: now also J3.7 (DAT0), R47.2
- net SD_DAT1: now reaches U1.34 (IO41)
- net SD_DAT1: now also J3.8 (DAT1), R48.2
- net SD_DAT2: now reaches U1.35 (IO42)
- net SD_DAT2: now also J3.1 (DAT2), R49.2
- net WHEEL_REAR_CAPTURE: now reaches U1.38 (IO2)
- net WHEEL_REAR_CAPTURE: now also R127.2
- net WHEEL_FRONT_CAPTURE: now reaches U1.39 (IO1)
- net WHEEL_FRONT_CAPTURE: now also R118.2
- net TIRE_CAN_CS: now reaches U1.8 (IO15)
- net TIRE_CAN_CS: now also R66.2, U20.13 (nCS)
- net TIRE_CAN_INT_N: now reaches U1.9 (IO16)
- net TIRE_CAN_INT_N: now also R67.2, U20.4 (INT)
- new net ADC_AIN6: C59.1, R42.2, U4.7 (CH6)
- new net ADC_AIN7: C61.1, R45.2, U4.8 (CH7)
- new net AFE_BUF4: R36.1, U13.1 (OUTA), U13.2 (-INA)
- new net AFE_BUF5: R39.1, U13.6 (-INB), U13.7 (OUTB)
- new net AFE_BUF6: R42.1, U13.8 (OUTC), U13.9 (-INC)
- new net AFE_BUF7: R45.1, U13.13 (-IND), U13.14 (OUTD)
- new net AFE_DIV4: C54.1, R34.2, R35.1, U13.3 (+INA)
- new net AFE_DIV5: C56.1, R37.2, R38.1, U13.5 (+INB)
- new net AFE_DIV6: C58.1, R40.2, R41.1, U13.10 (+INC)
- new net AFE_DIV7: C60.1, R43.2, R44.1, U13.12 (+IND)
- new net DIAG_U27_AIN0: C110.1, R130.2, R131.1, U27.11 (AIN0)
- new net DIAG_U27_AIN0_UPPER1: R128.2, R129.1
- new net DIAG_U27_AIN0_UPPER2: R129.2, R130.1
- new net DIAG_U27_AIN1: C111.1, R134.2, R135.1, U27.10 (AIN1)
- new net DIAG_U27_AIN1_UPPER1: R132.2, R133.1
- new net DIAG_U27_AIN1_UPPER2: R133.2, R134.1
- new net DIAG_U27_AIN2: C112.1, R138.2, R139.1, U27.7 (AIN2)
- new net DIAG_U27_AIN2_UPPER1: R136.2, R137.1
- new net DIAG_U27_AIN2_UPPER2: R137.2, R138.1
- new net DIAG_U28_AIN1: C114.1, R146.2, R147.1, U28.10 (AIN1)
- new net DIAG_U28_AIN1_UPPER1: R144.2, R145.1
- new net DIAG_U28_AIN1_UPPER2: R145.2, R146.1
- new net DIAG_U28_AIN2: C127.1, R168.2, R169.1, U28.7 (AIN2)
- new net DIAG_U28_AIN2_UPPER1: R166.2, R167.1
- new net DIAG_U28_AIN2_UPPER2: R167.2, R168.1
- new net DIAG_U28_AIN3: C129.1, R178.2, R179.1, U28.6 (AIN3)
- new net DIAG_U28_AIN3_UPPER1: R176.2, R177.1
- new net DIAG_U28_AIN3_UPPER2: R177.2, R178.1
- new net DIAG_U29_AIN0: C115.1, R150.2, R151.1, U29.11 (AIN0)
- new net DIAG_U29_AIN0_UPPER1: R148.2, R149.1
- new net DIAG_U29_AIN0_UPPER2: R149.2, R150.1
- new net DIAG_U29_AIN1: C116.1, R154.2, R155.1, U29.10 (AIN1)
- new net DIAG_U29_AIN1_UPPER1: R152.2, R153.1
- new net DIAG_U29_AIN1_UPPER2: R153.2, R154.1
- new net DIAG_U29_AIN2: C117.1, R158.2, R159.1, U29.7 (AIN2)
- new net DIAG_U29_AIN2_UPPER1: R156.2, R157.1
- new net DIAG_U29_AIN2_UPPER2: R157.2, R158.1
- new net POD_TIRE_SUPPLY: C93.1, J1.31 (Pin_31), R156.1, U25.10 (OUT)
- new net POD_WHEEL_FRONT_SIGNAL: D102.3 (K1_A2), D104.1 (K1), J1.24 (Pin_24)
- new net POD_WHEEL_REAR_SIGNAL: D103.3 (K1_A2), D104.2 (K2), J1.27 (Pin_27)
- new net POD_WHEEL_REAR_SUPPLY: C90.1, J1.26 (Pin_26), R119.1, R152.1, U24.10 (OUT)
- new net SENSOR_POWER_AUX_DVDT: C126.1, U30.8 (dVdT)
- new net SENSOR_POWER_AUX_ILIM: R165.1, U30.7 (ILIM)
- new net SENSOR_POWER_AUX_OVP: R163.2, R164.1, U30.3 (OVP)
- new net SENSOR_POWER_AUX_RTN: C126.2, R164.2, R165.2, U30.11 (EP_RTN), U30.5 (RTN)
- new net SENSOR_POWER_AUX_UVLO: R162.2, R163.1, U30.2 (UVLO)
- new net SENSOR_POWER_FRONT_DVDT: C88.1, U23.8 (dVdT)
- new net SENSOR_POWER_FRONT_ILIM: R76.1, U23.7 (ILIM)
- new net SENSOR_POWER_FRONT_OVP: R74.2, R75.1, U23.3 (OVP)
- new net SENSOR_POWER_FRONT_RTN: C88.2, R75.2, R76.2, U23.11 (EP_RTN), U23.5 (RTN)
- new net SENSOR_POWER_FRONT_UVLO: R73.2, R74.1, U23.2 (UVLO)
- new net SENSOR_POWER_REAR_DVDT: C91.1, U24.8 (dVdT)
- new net SENSOR_POWER_REAR_ILIM: R80.1, U24.7 (ILIM)
- new net SENSOR_POWER_REAR_OVP: R78.2, R79.1, U24.3 (OVP)
- new net SENSOR_POWER_REAR_RTN: C91.2, R79.2, R80.2, U24.11 (EP_RTN), U24.5 (RTN)
- new net SENSOR_POWER_REAR_UVLO: R77.2, R78.1, U24.2 (UVLO)
- new net SENSOR_POWER_TIRE_DVDT: C94.1, U25.8 (dVdT)
- new net SENSOR_POWER_TIRE_ILIM: R84.1, U25.7 (ILIM)
- new net SENSOR_POWER_TIRE_OVP: R82.2, R83.1, U25.3 (OVP)
- new net SENSOR_POWER_TIRE_RTN: C94.2, R83.2, R84.2, U25.11 (EP_RTN), U25.5 (RTN)
- new net SENSOR_POWER_TIRE_UVLO: R81.2, R82.1, U25.2 (UVLO)
- new net SUP_U16_CT: C71.1, U16.5 (CT)
- new net SUP_U16_SENSE: R56.2, R57.1, U16.1 (SENSE)
- new net SUP_U18_CT: C75.1, U18.5 (CT)
- new net SUP_U18_SENSE: R181.2, R61.1, U18.1 (SENSE)
- new net SUP_U18_TOP_SERIES: R181.1, R60.2
- new net SUP_U19_CT: C77.1, U19.5 (CT)
- new net SUP_U19_SENSE: R62.2, R63.1, U19.1 (SENSE)
- new net THERM_AUX1_SELECT: JP2.1 (A), R170.2
- new net THERM_AUX2_SELECT: JP3.1 (A), R171.2
- new net THERM_AUX3_SELECT: JP4.1 (A), R172.2
- new net THERM_AUX4_SELECT: JP5.1 (A), R173.2
- new net THERM_BIAS_IN: D105.3 (K1_A2), R174.1
- new net THERM_BIAS_MID: R174.2, R175.1
- new net THERM_EXC_2V495: C128.1, R170.1, R171.1, R172.1, R173.1, R175.2, R176.1, U31.1 (K), U31.2 (REF)
- new net TIRE_CAN_GPIO1: R72.1, U20.8 (GPIO1)
- new net TIRE_CAN_H: D101.1 (K1), J1.29 (Pin_29), J1.33 (Pin_33), R70.1, U21.7 (CANH)
- new net TIRE_CAN_L: D101.2 (K2), J1.30 (Pin_30), J1.34 (Pin_34), JP1.2 (B), U21.6 (CANL)
- new net TIRE_CAN_OSC1: C81.1, U20.6 (OSC1), Y1.1
- new net TIRE_CAN_OSC2: C82.1, U20.5 (OSC2), Y1.3
- new net TIRE_CAN_RX: U20.2 (RXCAN), U21.4 (RXD)
- new net TIRE_CAN_SILENT: R71.2, U21.8 (S), U22.4 (Y)
- new net TIRE_CAN_TERM: JP1.1 (A), R70.2
- new net TIRE_CAN_TX: R69.2, U20.1 (TXCAN), U21.1 (TXD)
- new net TIRE_CAN_TX_ENABLE: R68.1, U20.9 (GPIO0_XSTBY), U22.2 (B)
- new net WHEEL_FRONT_DIODE_OUT: D102.2 (K2), R112.1
- new net WHEEL_FRONT_FILTERED: C95.1, R112.2, R113.1, U26.2 (IN1-)
- new net WHEEL_FRONT_OUT: R116.1, R117.2, R118.1, U26.1 (OUT1)
- new net WHEEL_FRONT_PULLUP: D102.1 (A1), R111.2
- new net WHEEL_FRONT_PULLUP_MID: R110.2, R111.1
- new net WHEEL_FRONT_THRESHOLD: R114.2, R115.1, R116.2, U26.3 (IN1+)
- new net WHEEL_REAR_DIODE_OUT: D103.2 (K2), R121.1
- new net WHEEL_REAR_FILTERED: C96.1, R121.2, R122.1, U26.6 (IN2-)
- new net WHEEL_REAR_OUT: R125.1, R126.2, R127.1, U26.7 (OUT2)
- new net WHEEL_REAR_PULLUP: D103.1 (A1), R120.2
- new net WHEEL_REAR_PULLUP_MID: R119.2, R120.1
- new net WHEEL_REAR_THRESHOLD: R123.2, R124.1, R125.2, U26.5 (IN2+)
- no-connect marks 54 -> 53
Other:
- note added: "Auxiliary input buffers - candidate"
- note added: "Auxiliary power and diagnostic - qualification pending"
- note added: "Dedicated tire CAN - power and validation pending"
- note added: "FRONT protected sensor power - validation pending"
- note added: "Hall input conditioning - qualification pending"
- note added: "Independent rail supervision - qualification pending"
- note added: "Optional thermistor excitation - qualification pending"
- note added: "REAR protected sensor power - validation pending"
- note added: "Rail diagnostics - qualification pending"
- note added: "TIRE protected sensor power - validation pending"
- note added: "microSD storage (owner decision 2026-10-21: eMMC dropped)"
- moved on the sheet: C1, C10, C100, C11, C12, C13, C14, C15, C16, C17, C18, C19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

Commit message: AGENTEE-484: supply decoupling repaired in the canonical source and regenerated through the production path -- +C130 (U4 1uF), C131 (U8), C132 (U9), C133 (U100 VIO) 100nF; rebinds C38/C41->U2, C43->U10, C44->U3, C18->U11 (U7 keeps 3x22uF per LMR36520 Table 8-1); U3.22 V_BCKP PENDING-510; 28/28 stages; sch cef8e4c7 / pcb 0b68a0ac (313 fp); ERC 0 old/new; correspondence 2 inherited findings only; coverage PASS 313/0/0; new retention emission-7d5b0d4d-agentee484
Co-Authored-By: Claude Opus 5.5 <noreply@anthropic.com>
Parts:
- added C130: 1 uF/16 V, Capacitor_SMD:C_0603_1608Metric, symbol Device:C
- added C131, C132, C133: 100 nF/50 V X7R, Capacitor_SMD:C_0603_1608Metric, symbol Device:C
Connections:
- net +3V3: now also C130.1, C131.1, C132.1, C133.1
- net GND: now also C130.2, C131.2, C132.2, C133.2
Other:
- moved on the sheet: C100, C11, C110, C111, C112, C114, C115, C116, C117, C118, C119, C12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

Commit message: AGENTEE-488: C133/C84 pin 2 -> /+5V_CAN (VIO-to-VCC), C18 -> C694521 22uF/25V 1210 (engineering margin); regenerated 28/28 on fresh stock; retention emission-7d5b0d4d-agentee488; ERC 0; correspondence 2 inherited only; board delta exactly 3; named-return relationships + unsatisfied-on-missing-return fix (9/9); validator PASS 313/0/0
Co-Authored-By: Claude Opus 5.5 <noreply@anthropic.com>
Parts:
- C18: value 1 uF/16 V -> 22 uF/25 V; footprint Capacitor_SMD:C_0603_1608Metric -> Capacitor_SMD:C_1210_3225Metric; AGENT_EE_Ratings {"ratings":{"Voltage":"16V"},"record_sha256":"fddcc7f04afbc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 -> {"ratings":{"Voltage":"25V"},"record_sha256":"aa2c178081be7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; LCSC C76706 -> C694521; Partnumber CGA3E1X7R1C105KT0Y0N -> CGA6P3X7R1E226MT000N; Voltage 16V -> 25V
Connections:
- net +5V_CAN: now also C133.2, C84.2
- net GND: no longer C133.2, C84.2
Other:
- moved on the sheet: C110, C111, C112, C114, C115, C116, C117, C118, C119, C120, C121, C122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

Commit message: AGENTEE-488c/491 coherent production (8ecee9c, native-admit, 15:08:50-15:23:17Z, all steps exit 0): new retention emission-7d5b0d4d-agentee491 (417 files) + --install (board fa7c2ca6, sch 21965aeb); retain --check OK; ERC 0; correspondence 2 inherited U3 findings; validator PASS 313/0/0; board delta vs cbfea9be exactly R74/R78/R82 68.1k->75k and R75/R79/R83 215k->208k (same fpid/nets), 0 geometry moves
Co-Authored-By: Claude Opus 5.5 <noreply@anthropic.com>
Parts:
- R74: value 68.1 kohm 0.1% 25ppm/K -> 75 kohm 0.1% 25ppm/K; AGENT_EE_Ratings {"ratings":{"Power":"100mW"},"record_sha256":"f85d429cf5cef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 -> {"ratings":{"Power":"100mW"},"record_sha256":"074c9fa8e5c38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; LCSC C861521 -> C723587; PARAM_Datasheet {"schema":"agent-ee.datasheet-binding/1","sha256":"ecb56be7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 -> {"schema":"agent-ee.datasheet-binding/1","sha256":"7c8e6368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; Partnumber RT0603BRD0768K1L -> RT0603BRD0775KL
- R75: value 215 kohm 0.1% 25ppm/K -> 208 kohm 0.1% 25ppm/K; AGENT_EE_Ratings {"ratings":{"Power":"100mW"},"record_sha256":"f4afd38cd05f1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 -> {"ratings":{"Power":"100mW"},"record_sha256":"2fbe1720391ae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; LCSC C861226 -> C861219; PARAM_Datasheet {"schema":"agent-ee.datasheet-binding/1","sha256":"90bf8b84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 -> {"schema":"agent-ee.datasheet-binding/1","sha256":"ffde22da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; Partnumber RT0603BRD07215KL -> RT0603BRD07208KL
- R78: value 68.1 kohm 0.1% 25ppm/K -> 75 kohm 0.1% 25ppm/K; AGENT_EE_Ratings {"ratings":{"Power":"100mW"},"record_sha256":"87f1559a646a8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 -> {"ratings":{"Power":"100mW"},"record_sha256":"54e4b72a6bae6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; LCSC C861521 -> C723587; PARAM_Datasheet {"schema":"agent-ee.datasheet-binding/1","sha256":"ecb56be7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 -> {"schema":"agent-ee.datasheet-binding/1","sha256":"7c8e6368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; Partnumber RT0603BRD0768K1L -> RT0603BRD0775KL
- R79: value 215 kohm 0.1% 25ppm/K -> 208 kohm 0.1% 25ppm/K; AGENT_EE_Ratings {"ratings":{"Power":"100mW"},"record_sha256":"754e6e6e872a4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 -> {"ratings":{"Power":"100mW"},"record_sha256":"848c30f3880c4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; LCSC C861226 -> C861219; PARAM_Datasheet {"schema":"agent-ee.datasheet-binding/1","sha256":"90bf8b84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 -> {"schema":"agent-ee.datasheet-binding/1","sha256":"ffde22da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; Partnumber RT0603BRD07215KL -> RT0603BRD07208KL
- R82: value 68.1 kohm 0.1% 25ppm/K -> 75 kohm 0.1% 25ppm/K; AGENT_EE_Ratings {"ratings":{"Power":"100mW"},"record_sha256":"1b02f57df8fec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 -> {"ratings":{"Power":"100mW"},"record_sha256":"120e6a88316fa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; LCSC C861521 -> C723587; PARAM_Datasheet {"schema":"agent-ee.datasheet-binding/1","sha256":"ecb56be7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 -> {"schema":"agent-ee.datasheet-binding/1","sha256":"7c8e6368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; Partnumber RT0603BRD0768K1L -> RT0603BRD0775KL
- R83: value 215 kohm 0.1% 25ppm/K -> 208 kohm 0.1% 25ppm/K; AGENT_EE_Ratings {"ratings":{"Power":"100mW"},"record_sha256":"f208474cfb6bf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 -> {"ratings":{"Power":"100mW"},"record_sha256":"a2854aaec2b15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; LCSC C861226 -> C861219; PARAM_Datasheet {"schema":"agent-ee.datasheet-binding/1","sha256":"90bf8b84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 -> {"schema":"agent-ee.datasheet-binding/1","sha256":"ffde22da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; Partnumber RT0603BRD07215KL -> RT0603BRD07208KL
Other:
- moved on the sheet: C110, C111, C112, C114, C115, C116, C117, C118, C119, C120, C121, C122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
