File: telemetry-pod/telemetry-pod.kicad_pcb (KiCad board)
At the start: 4 copper layers, 90 x 65 mm, 112 parts, among them J1 776228-1, J2 732511150, Q1 DMP6023LE-13, U1 ESP32-S3-WROOM-1-N8, U10 TPS2553QDBVRQ1, U100 TJA1051T-3, U11 REF5050AIDR, U12 TPS7B4253QDDARQ1, U2 LSM6DSO32TR, U3 NEO-M9N-00B, U4 MCP3204-BI/SL, U5 LMR36520ADDAR, U6 TPS7B4253QDDARQ1, U7 LMR36520ADDAR, U8 ADA4096-4ARUZ-R7, U9 OPA320AIDBVR

Commit message: AGENTEE-207: j6 authentic two-iteration production preparation on agent-ee 81e387ee; production schematic re-emitted as the telemetry-pod project (AGENTEE-445)
Pinned agent-ee 81e387ee (AGENTEE-197 landed, hand-fit chain 08ddaa17, emitter
field order 41e91eca). pipeline.py verifies the export blob by blob against that
commit. Everything ran in the pinned CI image (ae-ci-exec, network none).

- Plan schema: requirement_source telemetry-pod-rev3, bound to fome-mc's pinned
  Revision 3 capture (requirements/compiled), added as scope baseline sources.
  The microSD spec equals it except the POD-CD-STORAGE row (checked); its own
  selection refuses unapproved-source (kept).
- Envelope: the five generic obligations are staged under agent-ee source
  contract telemetry-pod-expanded/1 (H1-H4, J1 fixed/containment/part-identity,
  U1 fixed/containment/antenna keepout, 20 open items). The final guard keeps
  blocking on them. Enclosure and harness are open design deliverables.
- Scope: parts_subset over composition/parts.json (J1 identity witness); fab_package
  declares JP1-5 copper, TP1-6 probes and the J1 not_assembled exclusion;
  antenna-facts datasheet_facts check; fab profile relabelled to the production
  envelope's requirement id (values and citations unchanged); declared hand-fit
  citation in the assembly check; emitter captures root fixed (emit-schematic
  failed on every library with 'footprints').
- No driver-default probe plan and no compiled-only scope. Stock is graded per
  id at generation (81 ids: 80 in stock, J1 C596198 zero; none stale).
- Real dry run: prepared, max_iterations 2 (plan), routing budget 900 s /
  timeout 2100 s, placement timeout 1500 s, derived watchdog 8400 s; review
  packet carries the 4 block obligations, copper_unknown and the 174-entry
  ledger; binding-fill 305 components / 248 ratings. No campaign launched.
- AGENTEE-445: the campaign's schematic-stage steps (binding-fill,
  emit-schematic, forward-annotate) ran with stage receipt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
Parts:
- added C110: 100nF 50V X7R, Capacitor_SMD:C_0603_1608Metric, F.Cu at (95.2, 351.8)
- added C111: 100nF 50V X7R, Capacitor_SMD:C_0603_1608Metric, F.Cu at (95.2, 355.6)
- added C112: 100nF 50V X7R, Capacitor_SMD:C_0603_1608Metric, F.Cu at (95.2, 359.4)
- added C114: 100nF 50V X7R, Capacitor_SMD:C_0603_1608Metric, F.Cu at (95.2, 363.2)
- added C115: 100nF 50V X7R, Capacitor_SMD:C_0603_1608Metric, F.Cu at (95.2, 367.0)
- added C116: 100nF 50V X7R, Capacitor_SMD:C_0603_1608Metric, F.Cu at (95.2, 370.8)
- added C117: 100nF 50V X7R, Capacitor_SMD:C_0603_1608Metric, F.Cu at (95.2, 374.6)
- added C118: 1uF 50V X7R, Capacitor_SMD:C_0805_2012Metric, F.Cu at (95.2, 378.5)
- added C119: 1uF 50V X7R, Capacitor_SMD:C_0805_2012Metric, F.Cu at (95.2, 383.5)
- added C120: 1uF 50V X7R, Capacitor_SMD:C_0805_2012Metric, F.Cu at (95.2, 388.6)
- added C121: 1uF 50V X7R, Capacitor_SMD:C_0805_2012Metric, F.Cu at (95.2, 393.7)
- added C122: 1uF 50V X7R, Capacitor_SMD:C_0805_2012Metric, F.Cu at (95.2, 398.8)
- added C123: 1uF 50V X7R, Capacitor_SMD:C_0805_2012Metric, F.Cu at (95.2, 403.9)
- added C124: 1uF 50V X7R, Capacitor_SMD:C_0805_2012Metric, F.Cu at (95.2, 408.9)
- added C125: 100nF 50V X7R, Capacitor_SMD:C_0603_1608Metric, F.Cu at (95.2, 412.8)
- added C126: 10nF 50V C0G 10%, Capacitor_SMD:C_0603_1608Metric, F.Cu at (95.2, 416.6)
- added C127: 100nF 50V X7R, Capacitor_SMD:C_0603_1608Metric, F.Cu at (95.2, 420.4)
- added C128: 10uF 16V X7R, Capacitor_SMD:C_1206_3216Metric, F.Cu at (95.2, 425.4)
- added C129: 100nF 50V X7R, Capacitor_SMD:C_0603_1608Metric, F.Cu at (95.2, 430.5)
- added C54: 100 nF/50 V X7R, Capacitor_SMD:C_0603_1608Metric, F.Cu at (95.2, 207.0)
- added C55: 100 pF C0G/50 V, Capacitor_SMD:C_0603_1608Metric, F.Cu at (95.2, 210.8)
- added C56: 100 nF/50 V X7R, Capacitor_SMD:C_0603_1608Metric, F.Cu at (95.2, 214.6)
- added C57: 100 pF C0G/50 V, Capacitor_SMD:C_0603_1608Metric, F.Cu at (95.2, 218.4)
- added C58: 100 nF/50 V X7R, Capacitor_SMD:C_0603_1608Metric, F.Cu at (95.2, 222.2)
- added C59: 100 pF C0G/50 V, Capacitor_SMD:C_0603_1608Metric, F.Cu at (95.2, 226.1)
- added C60: 100 nF/50 V X7R, Capacitor_SMD:C_0603_1608Metric, F.Cu at (95.2, 229.9)
- added C61: 100 pF C0G/50 V, Capacitor_SMD:C_0603_1608Metric, F.Cu at (95.2, 233.7)
- added C62: 100nF, Capacitor_SMD:C_0603_1608Metric, F.Cu at (95.2, 237.5)
- added C64: 4.7 uF/16 V X7R, Capacitor_SMD:C_0805_2012Metric, F.Cu at (95.2, 241.3)
- added C65: 100nF, Capacitor_SMD:C_0603_1608Metric, F.Cu at (95.2, 245.1)
- added C71: 22nF, Capacitor_SMD:C_0603_1608Metric, F.Cu at (95.2, 248.9)
- added C72: 100nF, Capacitor_SMD:C_0603_1608Metric, F.Cu at (95.2, 252.7)
- added C75: 22nF, Capacitor_SMD:C_0603_1608Metric, F.Cu at (95.2, 256.5)
- added C76: 100nF, Capacitor_SMD:C_0603_1608Metric, F.Cu at (95.2, 260.4)
- added C77: 22nF, Capacitor_SMD:C_0603_1608Metric, F.Cu at (95.2, 264.2)
- added C78: 100nF, Capacitor_SMD:C_0603_1608Metric, F.Cu at (95.2, 268.0)
- added C79: 100nF, Capacitor_SMD:C_0603_1608Metric, F.Cu at (95.2, 271.8)
- added C80: 1uF, Capacitor_SMD:C_0603_1608Metric, F.Cu at (95.2, 275.6)
- added C81: 18pF C0G, Capacitor_SMD:C_0603_1608Metric, F.Cu at (95.2, 279.4)
- added C82: 18pF C0G, Capacitor_SMD:C_0603_1608Metric, F.Cu at (95.2, 283.2)
- added C83: 100nF, Capacitor_SMD:C_0603_1608Metric, F.Cu at (95.2, 287.0)
- added C84: 100nF, Capacitor_SMD:C_0603_1608Metric, F.Cu at (95.2, 290.8)
- added C85: 100nF, Capacitor_SMD:C_0603_1608Metric, F.Cu at (95.2, 294.6)
- added C86: 1uF 50V X7R, Capacitor_SMD:C_0805_2012Metric, F.Cu at (95.2, 298.4)
- added C87: 100nF 50V X7R, Capacitor_SMD:C_0603_1608Metric, F.Cu at (95.2, 302.3)
- added C88: 10nF 50V C0G 10%, Capacitor_SMD:C_0603_1608Metric, F.Cu at (95.2, 306.1)
- added C89: 1uF 50V X7R, Capacitor_SMD:C_0805_2012Metric, F.Cu at (95.2, 309.9)
- added C90: 100nF 50V X7R, Capacitor_SMD:C_0603_1608Metric, F.Cu at (95.2, 313.7)
- added C91: 10nF 50V C0G 10%, Capacitor_SMD:C_0603_1608Metric, F.Cu at (95.2, 317.5)
- added C92: 1uF 50V X7R, Capacitor_SMD:C_0805_2012Metric, F.Cu at (95.2, 321.3)
- added C93: 100nF 50V X7R, Capacitor_SMD:C_0603_1608Metric, F.Cu at (95.2, 325.1)
- added C94: 10nF 50V C0G 10%, Capacitor_SMD:C_0603_1608Metric, F.Cu at (95.2, 328.9)
- added C95: 220pF C0G, Capacitor_SMD:C_0603_1608Metric, F.Cu at (95.2, 332.7)
- added C96: 220pF C0G, Capacitor_SMD:C_0603_1608Metric, F.Cu at (95.2, 336.6)
- added C97: 100nF 50V X7R, Capacitor_SMD:C_0603_1608Metric, F.Cu at (95.2, 340.4)
- added C98: 1uF 50V X7R, Capacitor_SMD:C_0805_2012Metric, F.Cu at (95.2, 344.2)
- added D101: PESD2CANFD24V-TR, Package_TO_SOT_SMD:SOT-23, F.Cu at (95.2, 453.4)
- added D102: BAV199,215, Package_TO_SOT_SMD:SOT-23, F.Cu at (95.2, 458.5)
- added D103: BAV199,215, Package_TO_SOT_SMD:SOT-23, F.Cu at (95.2, 463.6)
- added D104: PESD2CANFD24V-TR, Package_TO_SOT_SMD:SOT-23, F.Cu at (95.2, 468.6)
- added D105: BAV199,215, Package_TO_SOT_SMD:SOT-23, F.Cu at (95.2, 473.7)
- added J3: DM3AT-SF-PEJM5, Connector_Card:microSD_HC_Hirose_DM3AT-SF-PEJM5, B.Cu at (8.90, 32.0)
- added JP1: TIRE_TERM_CLOSE_ONLY_AT_BUS_END, Jumper:SolderJumper-2_P1.3mm_Open_RoundedPad1.0x1.5mm, F.Cu at (95.2, 478.8)
- added JP2: AUX1_THERM_PULLUP_CLOSE_TO_ENABLE, Jumper:SolderJumper-2_P1.3mm_Open_RoundedPad1.0x1.5mm, F.Cu at (95.2, 483.9)
- added JP3: AUX2_THERM_PULLUP_CLOSE_TO_ENABLE, Jumper:SolderJumper-2_P1.3mm_Open_RoundedPad1.0x1.5mm, F.Cu at (95.2, 488.9)
- added JP4: AUX3_THERM_PULLUP_CLOSE_TO_ENABLE, Jumper:SolderJumper-2_P1.3mm_Open_RoundedPad1.0x1.5mm, F.Cu at (95.2, 494.0)
- added JP5: AUX4_THERM_PULLUP_CLOSE_TO_ENABLE, Jumper:SolderJumper-2_P1.3mm_Open_RoundedPad1.0x1.5mm, F.Cu at (95.2, 499.1)
- added R110: 620 ohm, Resistor_SMD:R_2512_6332Metric, F.Cu at (95.2, 828.0)
- added R111: 620 ohm, Resistor_SMD:R_2512_6332Metric, F.Cu at (95.2, 834.4)
- added R112: 10 kohm 0.1%, Resistor_SMD:R_0603_1608Metric, F.Cu at (95.2, 839.5)
- added R113: 10 kohm 0.1%, Resistor_SMD:R_0603_1608Metric, F.Cu at (95.2, 843.3)
- added R114: 56 kohm 0.1%, Resistor_SMD:R_0603_1608Metric, F.Cu at (95.2, 847.1)
- added R115: 10 kohm 0.1%, Resistor_SMD:R_0603_1608Metric, F.Cu at (95.2, 850.9)
- added R116: 100 kohm 0.1%, Resistor_SMD:R_0603_1608Metric, F.Cu at (95.2, 854.7)
- added R117: 4.7 kohm 1%, Resistor_SMD:R_0603_1608Metric, F.Cu at (95.2, 858.5)
- added R118: 100 ohm, Resistor_SMD:R_0603_1608Metric, F.Cu at (95.2, 862.3)
- added R119: 620 ohm, Resistor_SMD:R_2512_6332Metric, F.Cu at (95.2, 867.4)
- added R120: 620 ohm, Resistor_SMD:R_2512_6332Metric, F.Cu at (95.2, 873.8)
- added R121: 10 kohm 0.1%, Resistor_SMD:R_0603_1608Metric, F.Cu at (95.2, 878.8)
- added R122: 10 kohm 0.1%, Resistor_SMD:R_0603_1608Metric, F.Cu at (95.2, 882.6)
- added R123: 56 kohm 0.1%, Resistor_SMD:R_0603_1608Metric, F.Cu at (95.2, 886.5)
- added R124: 10 kohm 0.1%, Resistor_SMD:R_0603_1608Metric, F.Cu at (95.2, 890.3)
- added R125: 100 kohm 0.1%, Resistor_SMD:R_0603_1608Metric, F.Cu at (95.2, 894.1)
- added R126: 4.7 kohm 1%, Resistor_SMD:R_0603_1608Metric, F.Cu at (95.2, 897.9)
- added R127: 100 ohm, Resistor_SMD:R_0603_1608Metric, F.Cu at (95.2, 901.7)
- added R128: 499 kohm 0.1% 25ppm/C, Resistor_SMD:R_0603_1608Metric, F.Cu at (95.2, 905.5)
- added R129: 499 kohm 0.1% 25ppm/C, Resistor_SMD:R_0603_1608Metric, F.Cu at (95.2, 909.3)
- added R130: 499 kohm 0.1% 25ppm/C, Resistor_SMD:R_0603_1608Metric, F.Cu at (95.2, 913.1)
- added R131: 4.99 kohm 0.1% 25ppm/C, Resistor_SMD:R_0603_1608Metric, F.Cu at (95.2, 916.9)
- added R132: 499 kohm 0.1% 25ppm/C, Resistor_SMD:R_0603_1608Metric, F.Cu at (95.2, 920.8)
- added R133: 499 kohm 0.1% 25ppm/C, Resistor_SMD:R_0603_1608Metric, F.Cu at (95.2, 924.6)
- added R134: 499 kohm 0.1% 25ppm/C, Resistor_SMD:R_0603_1608Metric, F.Cu at (95.2, 928.4)
- added R135: 4.99 kohm 0.1% 25ppm/C, Resistor_SMD:R_0603_1608Metric, F.Cu at (95.2, 932.2)
- added R136: 499 kohm 0.1% 25ppm/C, Resistor_SMD:R_0603_1608Metric, F.Cu at (95.2, 936.0)
- added R137: 499 kohm 0.1% 25ppm/C, Resistor_SMD:R_0603_1608Metric, F.Cu at (95.2, 939.8)
- added R138: 499 kohm 0.1% 25ppm/C, Resistor_SMD:R_0603_1608Metric, F.Cu at (95.2, 943.6)
- added R139: 4.99 kohm 0.1% 25ppm/C, Resistor_SMD:R_0603_1608Metric, F.Cu at (95.2, 947.4)
- added R144: 499 kohm 0.1% 25ppm/C, Resistor_SMD:R_0603_1608Metric, F.Cu at (95.2, 951.2)
- added R145: 499 kohm 0.1% 25ppm/C, Resistor_SMD:R_0603_1608Metric, F.Cu at (95.2, 955.0)
- added R146: 499 kohm 0.1% 25ppm/C, Resistor_SMD:R_0603_1608Metric, F.Cu at (95.2, 958.9)
- added R147: 4.99 kohm 0.1% 25ppm/C, Resistor_SMD:R_0603_1608Metric, F.Cu at (95.2, 962.7)
- added R148: 499 kohm 0.1% 25ppm/C, Resistor_SMD:R_0603_1608Metric, F.Cu at (95.2, 966.5)
- added R149: 499 kohm 0.1% 25ppm/C, Resistor_SMD:R_0603_1608Metric, F.Cu at (95.2, 970.3)
- added R150: 499 kohm 0.1% 25ppm/C, Resistor_SMD:R_0603_1608Metric, F.Cu at (95.2, 974.1)
- added R151: 4.99 kohm 0.1% 25ppm/C, Resistor_SMD:R_0603_1608Metric, F.Cu at (95.2, 977.9)
- added R152: 499 kohm 0.1% 25ppm/C, Resistor_SMD:R_0603_1608Metric, F.Cu at (95.2, 981.7)
- added R153: 499 kohm 0.1% 25ppm/C, Resistor_SMD:R_0603_1608Metric, F.Cu at (95.2, 985.5)
- added R154: 499 kohm 0.1% 25ppm/C, Resistor_SMD:R_0603_1608Metric, F.Cu at (95.2, 989.3)
- added R155: 4.99 kohm 0.1% 25ppm/C, Resistor_SMD:R_0603_1608Metric, F.Cu at (95.2, 993.1)
- added R156: 499 kohm 0.1% 25ppm/C, Resistor_SMD:R_0603_1608Metric, F.Cu at (95.2, 997.0)
- added R157: 499 kohm 0.1% 25ppm/C, Resistor_SMD:R_0603_1608Metric, F.Cu at (95.2, 1000.8)
- added R158: 499 kohm 0.1% 25ppm/C, Resistor_SMD:R_0603_1608Metric, F.Cu at (95.2, 1004.6)
- added R159: 4.99 kohm 0.1% 25ppm/C, Resistor_SMD:R_0603_1608Metric, F.Cu at (95.2, 1008.4)
- added R160: 2.2 kohm 1% 100ppm/C, Resistor_SMD:R_0603_1608Metric, F.Cu at (95.2, 1012.2)
- added R161: 2.2 kohm 1% 100ppm/C, Resistor_SMD:R_0603_1608Metric, F.Cu at (95.2, 1016.0)
- added R162: 1.05 Mohm 0.1% 25ppm/K, Resistor_SMD:R_0805_2012Metric, F.Cu at (95.2, 1019.8)
- added R163: 95.3 kohm 0.1% 25ppm/K, Resistor_SMD:R_0603_1608Metric, F.Cu at (95.2, 1023.6)
- added R164: 287 kohm 0.1% 25ppm/K, Resistor_SMD:R_0603_1608Metric, F.Cu at (95.2, 1027.4)
- added R165: 44.2 kohm 0.1% 25ppm/K, Resistor_SMD:R_0603_1608Metric, F.Cu at (95.2, 1031.2)
- added R166: 499 kohm 0.1% 25ppm/C, Resistor_SMD:R_0603_1608Metric, F.Cu at (95.2, 1035.0)
- added R167: 499 kohm 0.1% 25ppm/C, Resistor_SMD:R_0603_1608Metric, F.Cu at (95.2, 1038.9)
- added R168: 499 kohm 0.1% 25ppm/C, Resistor_SMD:R_0603_1608Metric, F.Cu at (95.2, 1042.7)
- added R169: 4.99 kohm 0.1% 25ppm/C, Resistor_SMD:R_0603_1608Metric, F.Cu at (95.2, 1046.5)
- added R170: 10 kohm 0.1% 25ppm/K, Resistor_SMD:R_0603_1608Metric, F.Cu at (95.2, 1050.3)
- added R171: 10 kohm 0.1% 25ppm/K, Resistor_SMD:R_0603_1608Metric, F.Cu at (95.2, 1054.1)
- added R172: 10 kohm 0.1% 25ppm/K, Resistor_SMD:R_0603_1608Metric, F.Cu at (95.2, 1057.9)
- added R173: 10 kohm 0.1% 25ppm/K, Resistor_SMD:R_0603_1608Metric, F.Cu at (95.2, 1061.7)
- added R174: 200 ohm 1% 100ppm/K 1.5W CRCW2512-HP, Resistor_SMD:R_2512_6332Metric, F.Cu at (95.2, 1066.8)
- added R175: 200 ohm 1% 100ppm/K 1.5W CRCW2512-HP, Resistor_SMD:R_2512_6332Metric, F.Cu at (95.2, 1073.2)
- added R176: 499 kohm 0.1% 25ppm/K, Resistor_SMD:R_0603_1608Metric, F.Cu at (95.2, 1078.2)
- added R177: 499 kohm 0.1% 25ppm/K, Resistor_SMD:R_0603_1608Metric, F.Cu at (95.2, 1082.0)
- added R178: 499 kohm 0.1% 25ppm/K, Resistor_SMD:R_0603_1608Metric, F.Cu at (95.2, 1085.8)
- added R179: 4.99 kohm 0.1% 25ppm/K, Resistor_SMD:R_0603_1608Metric, F.Cu at (95.2, 1089.7)
- added R180: 100 kohm 1% 100ppm/K, Resistor_SMD:R_0603_1608Metric, F.Cu at (95.2, 1093.5)
- added R181: 1.2 kohm 0.1% 25ppm/K, Resistor_SMD:R_0603_1608Metric, F.Cu at (95.2, 1097.3)
- added R34: 10 kohm, Resistor_SMD:R_0603_1608Metric, F.Cu at (95.2, 651.5)
- added R35: 10 kohm, Resistor_SMD:R_0603_1608Metric, F.Cu at (95.2, 655.3)
- added R36: 100 ohm, Resistor_SMD:R_0603_1608Metric, F.Cu at (95.2, 659.1)
- added R37: 10 kohm, Resistor_SMD:R_0603_1608Metric, F.Cu at (95.2, 662.9)
- added R38: 10 kohm, Resistor_SMD:R_0603_1608Metric, F.Cu at (95.2, 666.8)
- added R39: 100 ohm, Resistor_SMD:R_0603_1608Metric, F.Cu at (95.2, 670.6)
- added R40: 10 kohm, Resistor_SMD:R_0603_1608Metric, F.Cu at (95.2, 674.4)
- added R41: 10 kohm, Resistor_SMD:R_0603_1608Metric, F.Cu at (95.2, 678.2)
- added R42: 100 ohm, Resistor_SMD:R_0603_1608Metric, F.Cu at (95.2, 682.0)
- added R43: 10 kohm, Resistor_SMD:R_0603_1608Metric, F.Cu at (95.2, 685.8)
- added R44: 10 kohm, Resistor_SMD:R_0603_1608Metric, F.Cu at (95.2, 689.6)
- added R45: 100 ohm, Resistor_SMD:R_0603_1608Metric, F.Cu at (95.2, 693.4)
- added R46: 10 kohm, Resistor_SMD:R_0603_1608Metric, F.Cu at (95.2, 697.2)
- added R47: 10 kohm, Resistor_SMD:R_0603_1608Metric, F.Cu at (95.2, 701.0)
- added R48: 10 kohm, Resistor_SMD:R_0603_1608Metric, F.Cu at (95.2, 704.9)
- added R49: 10 kohm, Resistor_SMD:R_0603_1608Metric, F.Cu at (95.2, 708.7)
- added R50: 10 kohm, Resistor_SMD:R_0603_1608Metric, F.Cu at (95.2, 712.5)
- added R55: 10 kohm, Resistor_SMD:R_0603_1608Metric, F.Cu at (95.2, 716.3)
- added R56: 16.9 kohm 0.1%, Resistor_SMD:R_0603_1608Metric, F.Cu at (95.2, 720.1)
- added R57: 10 kohm 0.1%, Resistor_SMD:R_0603_1608Metric, F.Cu at (95.2, 723.9)
- added R60: 30.1 kohm 0.1% 25ppm/K, Resistor_SMD:R_0603_1608Metric, F.Cu at (95.2, 727.7)
- added R61: 10 kohm 0.1%, Resistor_SMD:R_0603_1608Metric, F.Cu at (95.2, 731.5)
- added R62: 64.9 kohm 0.1%, Resistor_SMD:R_0603_1608Metric, F.Cu at (95.2, 735.3)
- added R63: 10 kohm 0.1%, Resistor_SMD:R_0603_1608Metric, F.Cu at (95.2, 739.1)
- added R64: 10 kohm, Resistor_SMD:R_0603_1608Metric, F.Cu at (95.2, 743.0)
- added R65: 10 kohm, Resistor_SMD:R_0603_1608Metric, F.Cu at (95.2, 746.8)
- added R66: 10 kohm, Resistor_SMD:R_0603_1608Metric, F.Cu at (95.2, 750.6)
- added R67: 10 kohm, Resistor_SMD:R_0603_1608Metric, F.Cu at (95.2, 754.4)
- added R68: 10 kohm, Resistor_SMD:R_0603_1608Metric, F.Cu at (95.2, 758.2)
- added R69: 10 kohm, Resistor_SMD:R_0603_1608Metric, F.Cu at (95.2, 762.0)
- added R70: 120 ohm, Resistor_SMD:R_0603_1608Metric, F.Cu at (95.2, 765.8)
- added R71: 10 kohm, Resistor_SMD:R_0603_1608Metric, F.Cu at (95.2, 769.6)
- added R72: 10 kohm, Resistor_SMD:R_0603_1608Metric, F.Cu at (95.2, 773.4)
- added R73: 1.05 Mohm 0.1% 25ppm/K, Resistor_SMD:R_0805_2012Metric, F.Cu at (95.2, 777.2)
- added R74: 68.1 kohm 0.1% 25ppm/K, Resistor_SMD:R_0603_1608Metric, F.Cu at (95.2, 781.0)
- added R75: 215 kohm 0.1% 25ppm/K, Resistor_SMD:R_0603_1608Metric, F.Cu at (95.2, 784.9)
- added R76: 44.2 kohm 0.1%, Resistor_SMD:R_0603_1608Metric, F.Cu at (95.2, 788.7)
- added R77: 1.05 Mohm 0.1% 25ppm/K, Resistor_SMD:R_0805_2012Metric, F.Cu at (95.2, 792.5)
- added R78: 68.1 kohm 0.1% 25ppm/K, Resistor_SMD:R_0603_1608Metric, F.Cu at (95.2, 796.3)
- added R79: 215 kohm 0.1% 25ppm/K, Resistor_SMD:R_0603_1608Metric, F.Cu at (95.2, 800.1)
- added R80: 44.2 kohm 0.1%, Resistor_SMD:R_0603_1608Metric, F.Cu at (95.2, 803.9)
- added R81: 1.05 Mohm 0.1% 25ppm/K, Resistor_SMD:R_0805_2012Metric, F.Cu at (95.2, 807.7)
- added R82: 68.1 kohm 0.1% 25ppm/K, Resistor_SMD:R_0603_1608Metric, F.Cu at (95.2, 811.5)
- added R83: 215 kohm 0.1% 25ppm/K, Resistor_SMD:R_0603_1608Metric, F.Cu at (95.2, 815.3)
- added R84: 26.7 kohm 0.1%, Resistor_SMD:R_0603_1608Metric, F.Cu at (95.2, 819.1)
- added U13: ADA4096-4ARUZ-R7, Package_SO:TSSOP-14_4.4x5mm_P0.65mm, F.Cu at (95.2, 1219.2)
- added U16: TPS389001DSER, PodSupervisor:DSE0006A, F.Cu at (95.2, 1225.5)
- added U18: TPS389001DSER, PodSupervisor:DSE0006A, F.Cu at (95.2, 1230.6)
- added U19: TPS389001DSER, PodSupervisor:DSE0006A, F.Cu at (95.2, 1235.7)
- added U20: MCP2518FDT-E/SL, Package_SO:SOIC-14_3.9x8.7mm_P1.27mm, F.Cu at (95.2, 1243.3)
- added U21: TJA1051T/3/1J, Package_SO:SOIC-8_3.9x4.9mm_P1.27mm, F.Cu at (95.2, 1252.2)
- added U22: SN74LVC1G132DBVR, Package_TO_SOT_SMD:SOT-23-5, F.Cu at (95.2, 1258.6)
- added U23: TPS26625DRCR, Package_SON:VSON-10-1EP_3x3mm_P0.5mm_EP1.65x2.4mm, F.Cu at (95.2, 1264.9)
- added U24: TPS26625DRCR, Package_SON:VSON-10-1EP_3x3mm_P0.5mm_EP1.65x2.4mm, F.Cu at (95.2, 1271.3)
- added U25: TPS26625DRCR, Package_SON:VSON-10-1EP_3x3mm_P0.5mm_EP1.65x2.4mm, F.Cu at (95.2, 1277.6)
- added U26: LM2903BQDRQ1, Package_SO:SOIC-8_3.9x4.9mm_P1.27mm, F.Cu at (95.2, 1285.2)
- added U27: ADS1119IPWR, Package_SO:TSSOP-16_4.4x5mm_P0.65mm, F.Cu at (95.2, 1292.9)
- added U28: ADS1119IPWR, Package_SO:TSSOP-16_4.4x5mm_P0.65mm, F.Cu at (95.2, 1300.5)
- added U29: ADS1119IPWR, Package_SO:TSSOP-16_4.4x5mm_P0.65mm, F.Cu at (95.2, 1308.1)
- added U30: TPS26625DRCR, Package_SON:VSON-10-1EP_3x3mm_P0.5mm_EP1.65x2.4mm, F.Cu at (95.2, 1315.7)
- added U31: TL431BQDBZR, Package_TO_SOT_SMD:SOT-23, F.Cu at (95.2, 1322.1)
- added Y1: X1E0003410031 20MHz 12pF, Crystal:Crystal_SMD_SeikoEpson_FA238-4Pin_3.2x2.5mm, F.Cu at (95.2, 1334.8)
- C47: value 1uF -> 10nF
- J1: value 776228-1 -> 1-776163-1; footprint ampseal:ampseal-23 -> PodConnector:AMPSEAL_35_1-776163-1
- R29: value 10k -> 100 kohm
- U4: value MCP3204-BI/SL -> MCP3208-BI/SL; footprint Package_SO:SOIC-14_3.9x8.7mm_P1.27mm -> Package_SO:SOIC-16_3.9x9.9mm_P1.27mm
- moved U100 1296.8 mm to (95.2, 1328.4), turned to 0 degrees
- moved U10 1175.2 mm to (95.2, 1197.6), turned to 0 degrees
- moved U7 1171.0 mm to (95.2, 1178.6), turned to 0 degrees
- moved U8 1163.0 mm to (95.2, 1186.2), turned to 0 degrees
- moved U12 1161.9 mm to (95.2, 1211.6), turned to 0 degrees
- moved U11 1159.3 mm to (95.2, 1204.0), turned to 0 degrees
- moved U9 1158.8 mm to (95.2, 1192.5)
- moved U5 1152.5 mm to (95.2, 1163.3)
- moved U4 1130.6 mm to (95.2, 1153.2), turned to 0 degrees
- moved U6 1128.8 mm to (95.2, 1170.9), turned to 0 degrees
- moved TP6 1114.1 mm to (95.2, 1126.5)
- moved U3 1110.6 mm to (95.2, 1137.9), turned to 0 degrees
- moved TP5 1105.7 mm to (95.2, 1121.4)
- moved TP4 1102.9 mm to (95.2, 1116.3)
- moved TP3 1100.0 mm to (95.2, 1111.2)
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Connections:
- J1 pad 17: unconnected-(J1-Pin_17-Pad17) -> /POD_AUX1_SIGNAL
- J1 pad 18: unconnected-(J1-Pin_18-Pad18) -> /POD_AUX2_SIGNAL
- J1 pad 19: unconnected-(J1-Pin_19-Pad19) -> /POD_AUX3_SIGNAL
- J1 pad 20: unconnected-(J1-Pin_20-Pad20) -> /POD_AUX4_SIGNAL
- J1 pad 21: unconnected-(J1-Pin_21-Pad21) -> /POD_5V_AUX
- J1 pad 22: unconnected-(J1-Pin_22-Pad22) -> /GND
- J1 pad 23: unconnected-(J1-Pin_23-Pad23) -> /POD_WHEEL_FRONT_SUPPLY
- U1 pad 12: unconnected-(U1-IO8-Pad12) -> /POWER_FAIL_N
- U1 pad 22: unconnected-(U1-IO14-Pad22) -> /DIAG_I2C_SDA
- U1 pad 23: unconnected-(U1-IO21-Pad23) -> /DIAG_I2C_SCL
- U1 pad 24: unconnected-(U1-IO47-Pad24) -> /SD_DAT3
- U1 pad 25: unconnected-(U1-IO48-Pad25) -> /SENSOR_FAULT_N
- U1 pad 28: unconnected-(U1-IO35-Pad28) -> /SD_CD
- U1 pad 31: unconnected-(U1-IO38-Pad31) -> /SD_CLK
- U1 pad 32: unconnected-(U1-IO39-Pad32) -> /SD_CMD
- U1 pad 33: unconnected-(U1-IO40-Pad33) -> /SD_DAT0
- U1 pad 34: unconnected-(U1-IO41-Pad34) -> /SD_DAT1
- U1 pad 35: unconnected-(U1-IO42-Pad35) -> /SD_DAT2
- U1 pad 38: unconnected-(U1-IO2-Pad38) -> /WHEEL_REAR_CAPTURE
- U1 pad 39: unconnected-(U1-IO1-Pad39) -> /WHEEL_FRONT_CAPTURE
- U1 pad 8: unconnected-(U1-IO15-Pad8) -> /TIRE_CAN_CS
- U1 pad 9: unconnected-(U1-IO16-Pad9) -> /TIRE_CAN_INT_N
- U4 pad 10: /SPI_MISO -> /ADC_CS
- U4 pad 11: /SPI_SCK -> /SPI_MOSI
- U4 pad 12: /GND -> /SPI_MISO
- U4 pad 13: /SENSOR_REF_2V5 -> /SPI_SCK
- U4 pad 14: /+3V3 -> /GND
- U4 pad 5: unconnected-(U4-NC-Pad5) -> /ADC_AIN4
- U4 pad 6: unconnected-(U4-NC-Pad6) -> /ADC_AIN5
- U4 pad 7: /GND -> /ADC_AIN6
- U4 pad 8: /ADC_CS -> /ADC_AIN7
- U4 pad 9: /SPI_MOSI -> /GND
Routing:
- net /+3V3: track 209.5 -> 0.00 mm, vias 14 -> 0
- net /GND: track 195.4 -> 0.00 mm, vias 42 -> 0
- net /PRE_6V3: track 144.4 -> 0.00 mm, vias 4 -> 0
- net /SETPOINT_5V: track 108.8 -> 0.00 mm, vias 2 -> 0
- net /POD_5V_SENSOR: track 83.2 -> 0.00 mm, vias 2 -> 0
- net /SPI_MISO: track 77.1 -> 0.00 mm, vias 6 -> 0
- net /SPI_SCK: track 73.7 -> 0.00 mm, vias 2 -> 0
- net /SPI_MOSI: track 66.7 -> 0.00 mm, vias 2 -> 0
- net /IMU_CS: track 64.5 -> 0.00 mm, vias 2 -> 0
- net /ADC_CS: track 62.9 -> 0.00 mm, vias 4 -> 0
- net /IMU_INT1: track 59.5 -> 0.00 mm
- net /+5V_CAN: track 55.1 -> 0.00 mm
- net /MCU_EN: track 45.1 -> 0.00 mm, vias 2 -> 0
- net /POD_REAR_BRAKE_SIGNAL: track 44.6 -> 0.00 mm, vias 2 -> 0
- net /POD_FRONT_FORK_SIGNAL: track 40.8 -> 0.00 mm
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- removed copper zone on In1.Cu, net /GND
- removed copper zone on In2.Cu, net /GND
Other:
- board text added: "ASM J1 0deg"
- board text added: "ASM J2 180deg"
- board text added: "ASM J3 90deg"
- board text added: "ASM U1 0deg"
- board text removed: "IMU_AXES X forward Y left Z up"
