File: telemetry-pod/telemetry-pod.kicad_pcb (KiCad board)
At the start: 4 copper layers, 90 x 65 mm, 309 parts, among them J1 1-776163-1, J2 732511150, J3 DM3AT-SF-PEJM5, Q1 DMP6023LE-13, U1 ESP32-S3-WROOM-1-N8, U10 TPS2553QDBVRQ1, U100 TJA1051T-3, U11 REF5050AIDR, U12 TPS7B4253QDDARQ1, U13 ADA4096-4ARUZ-R7, U16 TPS389001DSER, U18 TPS389001DSER, U19 TPS389001DSER, U2 LSM6DSO32TR, U20 MCP2518FDT-E/SL, U21 TJA1051T/3/1J, U22 SN74LVC1G132DBVR, U23 TPS26625DRCR, U24 TPS26625DRCR, U25 TPS26625DRCR, U26 LM2903BQDRQ1, U27 ADS1119IPWR, U28 ADS1119IPWR, U29 ADS1119IPWR, U3 NEO-M9N-00B, U30 TPS26625DRCR, U31 TL431BQDBZR, U4 MCP3208-BI/SL, U5 LMR36520ADDAR, U6 TPS7B4253QDDARQ1, U7 LMR36520ADDAR, U8 ADA4096-4ARUZ-R7, U9 OPA320AIDBVR, Y1 X1E0003410031 20MHz 12pF

Commit message: AGENTEE-484: supply decoupling repaired in the canonical source and regenerated through the production path -- +C130 (U4 1uF), C131 (U8), C132 (U9), C133 (U100 VIO) 100nF; rebinds C38/C41->U2, C43->U10, C44->U3, C18->U11 (U7 keeps 3x22uF per LMR36520 Table 8-1); U3.22 V_BCKP PENDING-510; 28/28 stages; sch cef8e4c7 / pcb 0b68a0ac (313 fp); ERC 0 old/new; correspondence 2 inherited findings only; coverage PASS 313/0/0; new retention emission-7d5b0d4d-agentee484
Co-Authored-By: Claude Opus 5.5 <noreply@anthropic.com>
Parts:
- added C130: 1 uF/16 V, Capacitor_SMD:C_0603_1608Metric, F.Cu at (95.2, 434.3)
- added C131: 100 nF/50 V X7R, Capacitor_SMD:C_0603_1608Metric, F.Cu at (95.2, 438.1)
- added C132: 100 nF/50 V X7R, Capacitor_SMD:C_0603_1608Metric, F.Cu at (95.2, 442.0)
- added C133: 100 nF/50 V X7R, Capacitor_SMD:C_0603_1608Metric, F.Cu at (95.2, 445.8)
- moved D1 15.2 mm to (95.2, 450.9)
- moved D100 15.2 mm to (95.2, 463.6)
- moved D101 15.2 mm to (95.2, 468.6)
- moved D103 15.2 mm to (95.2, 478.8)
- moved D104 15.2 mm to (95.2, 483.9)
- moved D105 15.2 mm to (95.2, 488.9)
- moved D2 15.2 mm to (95.2, 455.9)
- moved D3 15.2 mm to (95.2, 459.7)
- moved JP2 15.2 mm to (95.2, 499.1)
- moved JP3 15.2 mm to (95.2, 504.2)
- moved JP4 15.2 mm to (95.2, 509.3)
- moved JP5 15.2 mm to (95.2, 514.4)
- moved L3 15.2 mm to (95.2, 530.9)
- moved Q1 15.2 mm to (95.2, 538.5)
- moved R1 15.2 mm to (95.2, 546.1)
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
Commit message: AGENTEE-488: C133/C84 pin 2 -> /+5V_CAN (VIO-to-VCC), C18 -> C694521 22uF/25V 1210 (engineering margin); regenerated 28/28 on fresh stock; retention emission-7d5b0d4d-agentee488; ERC 0; correspondence 2 inherited only; board delta exactly 3; named-return relationships + unsatisfied-on-missing-return fix (9/9); validator PASS 313/0/0
Co-Authored-By: Claude Opus 5.5 <noreply@anthropic.com>
Parts:
- C18: value 1 uF/16 V -> 22 uF/25 V; footprint Capacitor_SMD:C_0603_1608Metric -> Capacitor_SMD:C_1210_3225Metric
- moved R163 2.54 mm to (95.2, 1041.4)
- moved R167 2.54 mm to (95.2, 1056.6)
- moved R171 2.54 mm to (95.2, 1071.9)
- moved R178 2.54 mm to (95.2, 1103.6)
- moved U10 2.54 mm to (95.2, 1215.4)
- moved U18 2.54 mm to (95.2, 1248.4)
- moved U25 2.54 mm to (95.2, 1295.4)
- moved U27 2.54 mm to (95.2, 1310.6)
- moved U29 2.54 mm to (95.2, 1325.9)
- moved L1 2.54 mm to (95.2, 522.0)
- moved L2 2.54 mm to (95.2, 528.3)
- moved R110 2.54 mm to (95.2, 845.8)
- moved R119 2.54 mm to (95.2, 885.2)
- moved R129 2.54 mm to (95.2, 927.1)
- moved R131 2.54 mm to (95.2, 934.7)
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Connections:
- C133 pad 2: /GND -> /+5V_CAN
- C84 pad 2: /GND -> /+5V_CAN

Commit message: AGENTEE-488c/491 coherent production (8ecee9c, native-admit, 15:08:50-15:23:17Z, all steps exit 0): new retention emission-7d5b0d4d-agentee491 (417 files) + --install (board fa7c2ca6, sch 21965aeb); retain --check OK; ERC 0; correspondence 2 inherited U3 findings; validator PASS 313/0/0; board delta vs cbfea9be exactly R74/R78/R82 68.1k->75k and R75/R79/R83 215k->208k (same fpid/nets), 0 geometry moves
Co-Authored-By: Claude Opus 5.5 <noreply@anthropic.com>
Parts:
- R74, R78, R82: value 68.1 kohm 0.1% 25ppm/K -> 75 kohm 0.1% 25ppm/K
- R75, R79, R83: value 215 kohm 0.1% 25ppm/K -> 208 kohm 0.1% 25ppm/K
