File: telemetry-pod/expansion/storage-candidate/telemetry-pod.kicad_sch (KiCad schematic)
At the start: 146 parts, among them J1 776163-1, J2 732511150, Q1 DMP6023LE-13, U1 ESP32-S3-WROOM-1-N8, U10 TPS2553QDBVRQ1, U100 TJA1051T-3, U11 REF5050AIDR, U12 TPS7B4253QDDARQ1, U13 ADA4096-4ARUZ-R7, U14 FEMDME008G-A8A39, U2 LSM6DSO32TR, U3 NEO-M9N-00B, U4 MCP3208-BI/SL, U5 LMR36520ADDAR, U6 TPS7B4253QDDARQ1, U7 LMR36520ADDAR, U8 ADA4096-4ARUZ-R7, U9 OPA320AIDBVR

Commit message: Add separate eMMC core supply to expanded pod candidate
Parts:
- added C68, C69, C70: 22 uF/25 V, Capacitor_SMD:C_1210_3225Metric, symbol Device:C
- added L4: 2.2 uH, PodStoragePower:SRP4020TA, symbol Device:L
- added U15: TPS62162QDSGRQ1, Package_SON:Texas_DSG0008A_WSON-8-1EP_2x2mm_P0.5mm_EP0.9x1.6mm, symbol Regulator_Switching:TPS62162DSG
Connections:
- net EMMC_VCCQ_3V3 is gone; now on net +3V3: C66.1, C67.1, R46.1, R47.1, R48.1, R49.1, R50.1, R51.1, R52.1, R53.1, R54.1, U14.C6 (VCCQ), U14.M4 (VCCQ), U14.N4 (VCCQ), U14.P3 (VCCQ), U14.P5 (VCCQ)
- net EMMC_VCC_3V3: now also C68.1, C69.1, L4.2, U15.6 (VOS)
- net GND: now also C68.2, C69.2, C70.2, U15.1 (PGND), U15.4 (AGND), U15.5 (FB), U15.9 (PAD)
- net PRE_6V3: now also C70.1, U15.2 (VIN), U15.3 (EN)
- new net EMMC_CORE_SW: L4.1, U15.7 (SW)
- no-connect marks 175 -> 176
Other:
- note added: "Separate eMMC core supply - supervisor pending"
- moved on the sheet: C63, C64, C65, C66, C67, R46, R47, R48, R49, R50, R51, R52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

Commit message: Add independently checked telemetry rail supervision candidate
Parts:
- added C71, C73, C75, C77: 22nF, Capacitor_SMD:C_0603_1608Metric, symbol Device:C
- added C72, C74, C76, C78: 100nF, Capacitor_SMD:C_0603_1608Metric, symbol Device:C
- added R56: 16.9 kohm 0.1%, Resistor_SMD:R_0603_1608Metric, symbol Device:R
- added R57, R59, R61, R63: 10 kohm 0.1%, Resistor_SMD:R_0603_1608Metric, symbol Device:R
- added R58: 15.2 kohm 0.1%, Resistor_SMD:R_0603_1608Metric, symbol Device:R
- added R60: 31.3 kohm 0.1%, Resistor_SMD:R_0603_1608Metric, symbol Device:R
- added R62: 64.9 kohm 0.1%, Resistor_SMD:R_0603_1608Metric, symbol Device:R
- added R64, R65: 10 kohm, Resistor_SMD:R_0603_1608Metric, symbol Device:R
- added U16, U17, U18, U19: TPS389001DSER, PodSupervisor:DSE0006A, symbol PodSupervisor:TPS389001DSE
- C47: value 1uF -> 10nF; AGENT_EE_Ratings {"ratings":{"Voltage":"16V"},"record_sha256":"cb4ab6fa1e85b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 -> (none); LCSC C76706 -> (none); Manufacturer TDK -> (none); PARAM_Datasheet {"schema":"agent-ee.datasheet-binding/1","sha256":"ff9b0a37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 -> (none); Partnumber CGA3E1X7R1C105KT0Y0N -> (none); Voltage 16V -> (none)
- R29: value 10k -> 100 kohm; AGENT_EE_Ratings {"ratings":{"Power":"100mW"},"record_sha256":"57d99da031e5d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 -> (none); LCSC C95204 -> (none); Manufacturer YAGEO -> (none); PARAM_Datasheet {"schema":"agent-ee.datasheet-binding/1","sha256":"0a729d14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 -> (none); Partnumber RT0603BRD0710KL -> (none); Power 100mW -> (none)
Connections:
- net +3V3: now also C72.1, C74.1, C76.1, C78.1, R56.1, R64.1, R65.1, U16.3 (MR), U16.4 (VDD), U17.3 (MR), U17.4 (VDD), U18.3 (MR), U18.4 (VDD), U19.3 (MR), U19.4 (VDD)
- net EMMC_VCC_3V3: now also R58.1
- net GND: now also C71.2, C72.2, C73.2, C74.2, C75.2, C76.2, C77.2, C78.2, R57.2, R59.2, R61.2, R63.2, U16.2 (GND), U17.2 (GND), U18.2 (GND), U19.2 (GND)
- net MCU_EN: now also U16.6 (RESET), U17.6 (RESET)
- net POD_12V_PROTECTED: now also R62.1
- net POD_5V_SENSOR: now also R60.1
- net POWER_FAIL_N: now reaches U1.12 (IO8)
- net POWER_FAIL_N: now also R65.2, U19.6 (RESET)
- net SENSOR_FAULT_N: now reaches U1.25 (IO48)
- net SENSOR_FAULT_N: now also R64.2, U18.6 (RESET)
- new net SUP_U16_CT: C71.1, U16.5 (CT)
- new net SUP_U16_SENSE: R56.2, R57.1, U16.1 (SENSE)
- new net SUP_U17_CT: C73.1, U17.5 (CT)
- new net SUP_U17_SENSE: R58.2, R59.1, U17.1 (SENSE)
- new net SUP_U18_CT: C75.1, U18.5 (CT)
- new net SUP_U18_SENSE: R60.2, R61.1, U18.1 (SENSE)
- new net SUP_U19_CT: C77.1, U19.5 (CT)
- new net SUP_U19_SENSE: R62.2, R63.1, U19.1 (SENSE)
- no-connect marks 176 -> 174
Other:
- note added: "Independent rail supervision - qualification pending"
- moved on the sheet: C100, C42, C45, C46, C47, C48, C49, C50, C51, C52, C53, C54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
