File: telemetry-pod/expansion/storage-microsd/project/telemetry-pod.kicad_sch (KiCad schematic)
At the start: 305 parts, among them J1 1-776163-1, J2 732511150, J3 DM3AT-SF-PEJM5, Q1 DMP6023LE-13, U1 ESP32-S3-WROOM-1-N8, U10 TPS2553QDBVRQ1, U100 TJA1051T-3, U11 REF5050AIDR, U12 TPS7B4253QDDARQ1, U13 ADA4096-4ARUZ-R7, U16 TPS389001DSER, U18 TPS389001DSER, U19 TPS389001DSER, U2 LSM6DSO32TR, U20 MCP2518FDT-E/SL, U21 TJA1051T/3/1J, U22 SN74LVC1G132DBVR, U23 TPS26625DRCR, U24 TPS26625DRCR, U25 TPS26625DRCR, U26 LM2903BQDRQ1, U27 ADS1119IPWR, U28 ADS1119IPWR, U29 ADS1119IPWR, U3 NEO-M9N-00B, U30 TPS26625DRCR, U31 TL431BQDBZR, U4 MCP3208-BI/SL, U5 LMR36520ADDAR, U6 TPS7B4253QDDARQ1, U7 LMR36520ADDAR, U8 ADA4096-4ARUZ-R7, U9 OPA320AIDBVR, Y1 X1E0003410031 20MHz 12pF

Commit message: AGENTEE-484 checkpoint 1: decoupling source repair (intent + layout: C130-C133 added, C38/C41/C43/C44/C18 rebound), storage-microsd re-emitted (ERC 0), requirements scope recompiled, build.py additions, 478 data on the 313 inventory
Co-Authored-By: Claude Opus 5.5 <noreply@anthropic.com>
Parts:
- added C130: 1 uF/16 V, Capacitor_SMD:C_0603_1608Metric, symbol Device:C
- added C131, C132, C133: 100 nF/50 V X7R, Capacitor_SMD:C_0603_1608Metric, symbol Device:C
Connections:
- net +3V3: now also C130.1, C131.1, C132.1, C133.1
- net GND: now also C130.2, C131.2, C132.2, C133.2
Other:
- moved on the sheet: C100, C11, C110, C111, C112, C114, C115, C116, C117, C118, C119, C12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

Commit message: AGENTEE-488 checkpoint: source (C133/C84 pin 2 -> /+5V_CAN, C18 -> C694521 22uF 1210), storage-microsd re-emitted (ERC 0), requirements recompiled, build.py rebindings
Co-Authored-By: Claude Opus 5.5 <noreply@anthropic.com>
Parts:
- C18: value 1 uF/16 V -> 22 uF/25 V; footprint Capacitor_SMD:C_0603_1608Metric -> Capacitor_SMD:C_1210_3225Metric; AGENT_EE_Ratings {"ratings":{"Voltage":"16V"},"record_sha256":"0317eeb5bb39b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 -> {"ratings":{"Voltage":"25V"},"record_sha256":"958f8b0776737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; LCSC C76706 -> C694521; Partnumber CGA3E1X7R1C105KT0Y0N -> CGA6P3X7R1E226MT000N; Voltage 16V -> 25V
Connections:
- net +5V_CAN: now also C133.2, C84.2
- net GND: no longer C133.2, C84.2
Other:
- moved on the sheet: C110, C111, C112, C114, C115, C116, C117, C118, C119, C120, C121, C122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

Commit message: AGENTEE-491 source-level: R74/R78/R82 -> 75k RT0603BRD0775KL (C723587), R75/R79/R83 -> 208k RT0603BRD07208KL (C861219), R73/R77/R81 unchanged; storage-microsd re-emitted (ERC 0; netlist delta exactly six value/part changes, no nets); requirements recompiled; read-only stock for the two ids (C861219 1901); sensor-power README corrections (agent-derived static 8.3 V screen, transients unqualified, Izze operating range); regeneration STOPPED: canonical records for the two new parts + the POD-ME-1 guard
Co-Authored-By: Claude Opus 5.5 <noreply@anthropic.com>
Parts:
- R74, R78, R82: value 68.1 kohm 0.1% 25ppm/K -> 75 kohm 0.1% 25ppm/K; LCSC C861521 -> C723587; PARAM_Datasheet {"schema":"agent-ee.datasheet-binding/1","sha256":"ecb56be7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 -> {"schema":"agent-ee.datasheet-binding/1","sha256":"7c8e6368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; Partnumber RT0603BRD0768K1L -> RT0603BRD0775KL
- R75, R79, R83: value 215 kohm 0.1% 25ppm/K -> 208 kohm 0.1% 25ppm/K; LCSC C861226 -> C861219; PARAM_Datasheet {"schema":"agent-ee.datasheet-binding/1","sha256":"90bf8b84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 -> {"schema":"agent-ee.datasheet-binding/1","sha256":"ffde22da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; Partnumber RT0603BRD07215KL -> RT0603BRD07208KL
Other:
- moved on the sheet: C110, C111, C112, C114, C115, C116, C117, C118, C119, C120, C121, C122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
